File: Schematic/External 40 Pin Header.kicad_sch (KiCad schematic)
At the start: 22 parts, among them J9 40 Pin Header

Commit message: Started to work on the BOM
Parts:
- removed R3, R4: 2k2, symbol Device:R
- removed TP26, TP27, TP28, TP29, TP30, TP31, TP32, TP33, TP34, TP35, TP36, TP37, TP38, TP39, TP40, TP41, TP42, TP43, TP44: TestPoint, symbol Connector:TestPoint
- J9: now not fitted; now left out of the parts list
