File: Schematic/GPS Sensor.kicad_sch (KiCad schematic)
At the start: 50 parts, among them J30 USB_C_Receptacle_USB2.0_14P, J31 EXT_GPS, J32 GPS_VCC, J33 GPS_RX, J34 GPS_TX, J35 SMA, U34 ZED-F9P-15B

Commit message: Started to work on the BOM
Parts:
- removed BT1: CR1220, symbol Device:Battery_Cell
- added BT1: BAT-HLD-007-SMT-TR, BAT-HLD-007-SMT-TR:BATHLD007SMTTR, symbol BAT-HLD-007-SMT-TR:BAT-HLD-007-SMT-TR
- added TP169, TP170: TestPoint, symbol Connector:TestPoint
- C212: renamed from C216; footprint (none) -> Capacitor_SMD:C_1206_3216Metric_Pad1.33x1.80mm_HandSolder; Link (none) -> https://mou.sr/4l54Mdx; Manufacturer Part Number (none) -> CL31A106KBHNNNE; Price per Unit (none) -> 0.11; Supplier (none) -> Mouser; Supplier Part Number (none) -> 187-CL31A106KBHNNNE; now left out of the parts list
- C213: renamed from C217; footprint (none) -> Capacitor_SMD:C_1206_3216Metric_Pad1.33x1.80mm_HandSolder; Link (none) -> https://mou.sr/4l54Mdx; Manufacturer Part Number (none) -> CL31A106KBHNNNE; Price per Unit (none) -> 0.11; Supplier (none) -> Mouser; Supplier Part Number (none) -> 187-CL31A106KBHNNNE; now left out of the parts list
- C214: renamed from C218; footprint (none) -> Capacitor_SMD:C_1206_3216Metric_Pad1.33x1.80mm_HandSolder; Link (none) -> https://mou.sr/4l54Mdx; Manufacturer Part Number (none) -> CL31A106KBHNNNE; Price per Unit (none) -> 0.11; Supplier (none) -> Mouser; Supplier Part Number (none) -> 187-CL31A106KBHNNNE; now left out of the parts list
- C215: renamed from C219; footprint (none) -> Capacitor_SMD:C_1206_3216Metric_Pad1.33x1.80mm_HandSolder; Link (none) -> https://mou.sr/41y0aEA; Manufacturer Part Number (none) -> CL31B105KBHNNNE; Price per Unit (none) -> 0.11; Supplier (none) -> Mouser; Supplier Part Number (none) -> 187-CL31B105KBHNNNE; now left out of the parts list
- C216: renamed from C220; footprint (none) -> Capacitor_SMD:C_1206_3216Metric_Pad1.33x1.80mm_HandSolder; Link (none) -> https://mou.sr/4n9ybmQ; Manufacturer Part Number (none) -> CL31B104KBCNNNC; Price per Unit (none) -> 0.11; Supplier (none) -> Mouser; Supplier Part Number (none) -> 187-CL31B104KBCNNNC; now left out of the parts list
- C217: renamed from C221; footprint (none) -> Capacitor_SMD:C_1206_3216Metric_Pad1.33x1.80mm_HandSolder; Link (none) -> https://mou.sr/4n9ybmQ; Manufacturer Part Number (none) -> CL31B104KBCNNNC; Price per Unit (none) -> 0.11; Supplier (none) -> Mouser; Supplier Part Number (none) -> 187-CL31B104KBCNNNC; now left out of the parts list
- C218: renamed from C222; footprint (none) -> Capacitor_SMD:C_1206_3216Metric_Pad1.33x1.80mm_HandSolder; Link (none) -> https://mou.sr/4n9ybmQ; Manufacturer Part Number (none) -> CL31B104KBCNNNC; Price per Unit (none) -> 0.11; Supplier (none) -> Mouser; Supplier Part Number (none) -> 187-CL31B104KBCNNNC; now left out of the parts list
- C219: renamed from C223; footprint (none) -> Capacitor_SMD:C_0603_1608Metric_Pad1.08x0.95mm_HandSolder; Link (none) -> https://mou.sr/4g6fuOy; Manufacturer Part Number (none) -> CL10B472KB8NFNC; Price per Unit (none) -> 0.10; Supplier (none) -> Mouser; Supplier Part Number (none) -> 187-CL10B472KB8NFNC; now left out of the parts list
- C220: renamed from C224; footprint (none) -> Capacitor_SMD:C_0603_1608Metric_Pad1.08x0.95mm_HandSolder; Link (none) -> https://mou.sr/42eP5Z4; Manufacturer Part Number (none) -> CL10C470JC81PNC; Price per Unit (none) -> 0.10; Supplier (none) -> Mouser; Supplier Part Number (none) -> 187-CL10C470JC81PNC; now left out of the parts list
- D48: renamed from D51; footprint ESD122DMYR:DIO_ESD122DMYR -> ESD122DMYR:ESD122DMYR; Link (none) -> https://mou.sr/46mVGTO; Manufacturer Part Number (none) -> ESD122DMYR; Price None -> (none); Price per Unit (none) -> 1.01; Supplier (none) -> Mouser; Supplier Part Number (none) -> 595-ESD122DMYR; now left out of the parts list
- D49: renamed from D52; footprint PCM_Diode_SMD_AKL:D_0805_2012Metric -> ASMM-CR03-BU802:LEDM3528X210N; Link (none) -> https://mou.sr/460BFB7; Manufacturer Part Number (none) -> ASMM-CR03-BU802; Price per Unit (none) -> 0.32; Supplier (none) -> Mouser; Supplier Part Number (none) -> 630-ASMM-CR03-BU802; now left out of the parts list
- D50: renamed from D53; footprint PCM_Diode_SMD_AKL:D_SOD-123 -> (none); now left out of the parts list
- D51: renamed from D54; footprint PCM_Diode_SMD_AKL:D_0805_2012Metric -> ASMM-CR03-BU802:LEDM3528X210N; Link (none) -> https://mou.sr/460BFB7; Manufacturer Part Number (none) -> ASMM-CR03-BU802; Price per Unit (none) -> 0.32; Supplier (none) -> Mouser; Supplier Part Number (none) -> 630-ASMM-CR03-BU802; now left out of the parts list
- D52: renamed from D55; footprint PCM_Diode_SMD_AKL:D_0805_2012Metric -> ASMM-CR03-BU802:LEDM3528X210N; Link (none) -> https://mou.sr/460BFB7; Manufacturer Part Number (none) -> ASMM-CR03-BU802; Price per Unit (none) -> 0.32; Supplier (none) -> Mouser; Supplier Part Number (none) -> 630-ASMM-CR03-BU802; now left out of the parts list
- D53: renamed from D56; footprint PCM_Diode_SMD_AKL:D_0805_2012Metric -> ASMM-CR03-BU802:LEDM3528X210N; Link (none) -> https://mou.sr/460BFB7; Manufacturer Part Number (none) -> ASMM-CR03-BU802; Price per Unit (none) -> 0.32; Supplier (none) -> Mouser; Supplier Part Number (none) -> 630-ASMM-CR03-BU802; now left out of the parts list
- J28: renamed from J30; now left out of the parts list
- J29: renamed from J31; now not fitted; now left out of the parts list
- J30: renamed from J32; now not fitted; now left out of the parts list
- J31: renamed from J33; now not fitted; now left out of the parts list
- J32: renamed from J34; now not fitted; now left out of the parts list
- J33: renamed from J35; now left out of the parts list
- L4: now left out of the parts list
- R173: renamed from R177; now left out of the parts list
- R174: renamed from R178; now left out of the parts list
- R175: renamed from R179; now left out of the parts list
- R176: renamed from R180; now left out of the parts list
- R177: renamed from R181; now left out of the parts list
- R178: renamed from R182; now left out of the parts list
- R179: renamed from R183; now left out of the parts list
- R180: renamed from R184; now left out of the parts list
- R181: renamed from R185; now left out of the parts list
- R182: renamed from R186; now left out of the parts list
- R183: renamed from R187; now left out of the parts list
- TP154: renamed from TP167; now not fitted; now left out of the parts list
- TP155: renamed from TP168; now not fitted; now left out of the parts list
- TP156: renamed from TP169; now not fitted; now left out of the parts list
- TP157: renamed from TP170; now not fitted; now left out of the parts list
- TP158: renamed from TP171; now not fitted; now left out of the parts list
- TP159: renamed from TP172; now not fitted; now left out of the parts list
- TP160: renamed from TP173; now not fitted; now left out of the parts list
- TP161: renamed from TP174; now not fitted; now left out of the parts list
- TP162: renamed from TP175; now not fitted; now left out of the parts list
- TP163: renamed from TP176; now not fitted; now left out of the parts list
- TP164: renamed from TP177; now not fitted; now left out of the parts list
- TP165: renamed from TP178; now not fitted; now left out of the parts list
- TP166: renamed from TP179; now not fitted; now left out of the parts list
- TP167: renamed from TP180; now not fitted; now left out of the parts list
- TP168: renamed from TP181; now not fitted; now left out of the parts list
- U32: renamed from U34; footprint RF_GPS:ublox_ZED -> (none); now left out of the parts list
Connections:
- net GND: now also BT1.3 (-)
- net GPS_RX: now also TP170.1
- net GPS_TX: now also TP169.1
- net V_BCKP: now also BT1.1 (+_1), BT1.2 (+_2)
Other:
- moved on the sheet: C218, C219, D50, R179
