File: Schematic/Charger FET Array.kicad_sch (KiCad schematic)
At the start: 31 parts, among them Q25 CSD19531Q5A, Q26 CSD19531Q5A, Q27 CSD19531Q5A, Q28 CSD19531Q5A

Commit message: Massive pivit, simplification
Parts:
- renumbered C123 to C116, C124 to C117, C125 to C118, C126 to C119, C127 to C120, C128 to C121, C129 to C122, C130 to C123, C131 to C124, C132 to C125, C133 to C126
