File: Schematic/USB-C Port.kicad_sch (KiCad schematic)
At the start: 16 parts, among them J14 USB_C_Receptacle_USB2.0_14P, U11 TVS2200DRV

Commit message: Started to work on the BOM
Parts:
- C56: renamed from C61; footprint (none) -> Capacitor_SMD:C_1206_3216Metric_Pad1.33x1.80mm_HandSolder; Link (none) -> https://mou.sr/45jYGQI; Manufacturer Part Number (none) -> CL31B475KBHNFNE; Price per Unit (none) -> 0.27; Supplier (none) -> Mouser; Supplier Part Number (none) -> 187-CL31B475KBHNFNE
- C57: renamed from C62; footprint (none) -> Capacitor_SMD:C_1206_3216Metric_Pad1.33x1.80mm_HandSolder; Link (none) -> https://mou.sr/45jYGQI; Manufacturer Part Number (none) -> CL31B475KBHNFNE; Price per Unit (none) -> 0.27; Supplier (none) -> Mouser; Supplier Part Number (none) -> 187-CL31B475KBHNFNE
- C58: renamed from C63; footprint (none) -> Capacitor_SMD:C_1206_3216Metric_Pad1.33x1.80mm_HandSolder; Link (none) -> https://mou.sr/4n9ybmQ; Manufacturer Part Number (none) -> CL31B104KBCNNNC; Price per Unit (none) -> 0.11; Supplier (none) -> Mouser; Supplier Part Number (none) -> 187-CL31B104KBCNNNC
- C59: renamed from C64; footprint (none) -> Capacitor_SMD:C_1206_3216Metric_Pad1.33x1.80mm_HandSolder; Link (none) -> https://mou.sr/3OC0xXF; Manufacturer Part Number (none) -> CL31B103KHFNFNE; Price per Unit (none) -> 0.13; Supplier (none) -> Mouser; Supplier Part Number (none) -> 187-CL31B103KHFNFNE
- C60: renamed from C65; footprint (none) -> Capacitor_SMD:C_1206_3216Metric_Pad1.33x1.80mm_HandSolder; Link (none) -> https://mou.sr/3OC0xXF; Manufacturer Part Number (none) -> CL31B103KHFNFNE; Price per Unit (none) -> 0.13; Supplier (none) -> Mouser; Supplier Part Number (none) -> 187-CL31B103KHFNFNE
- C61: renamed from C66; footprint (none) -> Capacitor_SMD:C_1206_3216Metric_Pad1.33x1.80mm_HandSolder; Link (none) -> https://mou.sr/3OC0xXF; Manufacturer Part Number (none) -> CL31B103KHFNFNE; Price per Unit (none) -> 0.13; Supplier (none) -> Mouser; Supplier Part Number (none) -> 187-CL31B103KHFNFNE
- C62: renamed from C67; footprint (none) -> Capacitor_SMD:C_1206_3216Metric_Pad1.33x1.80mm_HandSolder; Link (none) -> https://mou.sr/3OC0xXF; Manufacturer Part Number (none) -> CL31B103KHFNFNE; Price per Unit (none) -> 0.13; Supplier (none) -> Mouser; Supplier Part Number (none) -> 187-CL31B103KHFNFNE
- D39: renamed from D42; footprint ESD122DMYR:DIO_ESD122DMYR -> ESD122DMYR:ESD122DMYR; Link (none) -> https://mou.sr/46mVGTO; Manufacturer Part Number (none) -> ESD122DMYR; Price None -> (none); Price per Unit (none) -> 1.01; Supplier (none) -> Mouser; Supplier Part Number (none) -> 595-ESD122DMYR
- U9: renamed from U11; footprint Package_SON:WSON-6-1EP_2x2mm_P0.65mm_EP1x1.6mm -> (none)
- renumbered J14 to J12, TP99 to TP76, TP100 to TP77, TP101 to TP78, TP102 to TP79, TP103 to TP80

Commit message: Massive pivit, simplification
Parts:
- removed D39: ESD122DMYR, ESD122DMYR:ESD122DMYR, symbol ESD122:ESD122DMYR
- added D38, D44: 82306050029, 82306050029:WESURGE_0603134, symbol 82306050029:82306050029
- renumbered C56 to C49, C57 to C50, C58 to C51, C59 to C52, C60 to C53, C61 to C54, C62 to C55, FB10 to FB9, J12 to J10, TP76 to TP69, TP77 to TP70, TP78 to TP71, TP79 to TP72, TP80 to TP73, U9 to U8
Connections:
- net GND: now also D38.2 (A2), D44.2 (A2)
- net USB_C_N: now also D38.1 (A1)
- net USB_C_P: now also D44.1 (A1)
