File: Schematic/BMS Protection Board.kicad_sch (KiCad schematic)
At the start: 0 parts

Commit message: added sensors?
Other:
- sheet High Side Gate Driver ports: added BATT+; removed none
- note added: "BMS Protection Board for 8S Battery Pack In/Out: min voltage: 25.6 V, nominal voltage: 29.6 V, max voltage: 33.6 V Output: 50A continuous discharge current Min Each Cell set to 3.2V, Max Each Cell set to 4.2V"
- note removed: "BMS Protection Board for 8S Battery Pack In/Out: min voltage: 24.0 V, nominal voltage: 29.6 V, max voltage: 33.6 V Output: 30A continuous discharge current, 100A peak discharge current"
Changed lines of the file:
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@@
 	(generator_version "9.0")
 	(paper "A4")
-	(text "BMS Protection Board for 8S Battery Pack\nIn/Out: min voltage: 24.0 V, nominal voltage: 29.6 V, max voltage: 33.6 V\nOutput: 30A continuous discharge current, 100A peak discharge current"
+	(text "BMS Protection Board for 8S Battery Pack\nIn/Out: min voltage: 25.6 V, nominal voltage: 29.6 V, max voltage: 33.6 V\nOutput: 50A continuous discharge current\nMin Each Cell set to 3.2V, Max Each Cell set to 4.2V"
 		(exclude_from_sim no)
 		(at 22.352 184.658 0)
@@
 		(color 0 0 0 0)
 	)
+	(junction
+		(at 22.86 152.4)
+		(diameter 0)
+		(color 0 0 0 0)
+	)
 	(wire
 		(pts
@@
 	(wire
 		(pts
-			(xy 45.72 152.4) (xy 46.99 152.4)
+			(xy 20.32 152.4) (xy 22.86 152.4)
 		)
 		(stroke
@@
 	(wire
 		(pts
+			(xy 35.56 118.11) (xy 22.86 118.11)
+		)
+		(stroke
+			(width 0)
+			(type default)
+		)
+	)
+	(wire
+		(pts
 			(xy 203.2 88.9) (xy 243.84 88.9)
 		)
@@
 	(wire
 		(pts
-			(xy 16.51 118.11) (xy 16.51 86.36)
+			(xy 16.51 115.57) (xy 16.51 86.36)
 		)
 		(stroke
@@
 	(wire
 		(pts
+			(xy 22.86 152.4) (xy 46.99 152.4)
+		)
+		(stroke
+			(width 0)
+			(type default)
+		)
+	)
+	(wire
+		(pts
 			(xy 102.87 105.41) (xy 102.87 143.51)
 		)
@@
 	(wire
 		(pts
+			(xy 22.86 118.11) (xy 22.86 152.4)
+		)
+		(stroke
+			(width 0)
+			(type default)
+		)
+	)
+	(wire
+		(pts
 			(xy 270.51 121.92) (xy 283.21 121.92)
 		)
@@
 	(wire
 		(pts
-			(xy 16.51 118.11) (xy 35.56 118.11)
+			(xy 16.51 115.57) (xy 35.56 115.57)
 		)
 		(stroke
@@
 	)
 	(label "PACKDIV"
-		(at 25.4 118.11 0)
+		(at 25.4 115.57 0)
 		(effects
 			(font
@@
 	(hierarchical_label "BATT+"
 		(shape input)
-		(at 45.72 152.4 180)
+		(at 20.32 152.4 180)
 		(effects
 			(font
@@
 		)
 		(pin "PACKDIV" output
+			(at 35.56 115.57 180)
+			(effects
+				(font
+					(size 1.27 1.27)
+				)
+				(justify left)
+			)
+		)
+		(pin "BATT+" input
 			(at 35.56 118.11 180)
 			(effects
@@
 		)
 		(instances
-			(project "Project-Star"
+			(project "STAR"
 				(path "/fc8533bc-25dd-4c20-9b4c-ffebebd6739b/e8da5d81-614b-4fe5-84b3-4c351fab7114"
 					(page "8")
@@
 		)
 		(instances
-			(project "Project-Star"
+			(project "STAR"
 				(path "/fc8533bc-25dd-4c20-9b4c-ffebebd6739b/e8da5d81-614b-4fe5-84b3-4c351fab7114"
 					(page "3")
@@
 		)
 		(instances
-			(project "Project-Star"
+			(project "STAR"
 				(path "/fc8533bc-25dd-4c20-9b4c-ffebebd6739b/e8da5d81-614b-4fe5-84b3-4c351fab7114"
 					(page "4")
@@
 		)
 		(instances
-			(project "Project-Star"
+			(project "STAR"
 				(path "/fc8533bc-25dd-4c20-9b4c-ffebebd6739b/e8da5d81-614b-4fe5-84b3-4c351fab7114"
 					(page "9")
@@
 		)
 		(instances
-			(project "Project-Star"
+			(project "STAR"
 				(path "/fc8533bc-25dd-4c20-9b4c-ffebebd6739b/e8da5d81-614b-4fe5-84b3-4c351fab7114"
 					(page "11")
@@
 		)
 		(instances
-			(project "Project-Star"
+			(project "STAR"
 				(path "/fc8533bc-25dd-4c20-9b4c-ffebebd6739b/e8da5d81-614b-4fe5-84b3-4c351fab7114"
 					(page "7")
@@
 		)
 		(instances
-			(project "Project-Star"
+			(project "STAR"
 				(path "/fc8533bc-25dd-4c20-9b4c-ffebebd6739b/e8da5d81-614b-4fe5-84b3-4c351fab7114"
 					(page "6")
@@
 		)
 		(instances
-			(project "Project-Star"
+			(project "STAR"
 				(path "/fc8533bc-25dd-4c20-9b4c-ffebebd6739b/e8da5d81-614b-4fe5-84b3-4c351fab7114"
 					(page "10")
@@
 		)
 		(instances
-			(project "Project-Star"
+			(project "STAR"
 				(path "/fc8533bc-25dd-4c20-9b4c-ffebebd6739b/e8da5d81-614b-4fe5-84b3-4c351fab7114"
 					(page "5")

Commit message: Massive pivit, simplification
Parts:
- added C33, C34, C35, C36: 220n, Capacitor_SMD:C_0805_2012Metric_Pad1.18x1.45mm_HandSolder, symbol Device:C
- added C37, C38, C39, C40, C41, C48, C49, C56, C57, C59: 100n, Capacitor_SMD:C_1206_3216Metric_Pad1.33x1.80mm_HandSolder, symbol Device:C
- added C42, C47: 470p, Capacitor_SMD:C_0603_1608Metric_Pad1.08x0.95mm_HandSolder, symbol Device:C
- added C43, C45, C55, C58, C61: 1u, Capacitor_SMD:C_1206_3216Metric_Pad1.33x1.80mm_HandSolder, symbol Device:C
- added C44, C46: 10u, Capacitor_SMD:C_1206_3216Metric_Pad1.33x1.80mm_HandSolder, symbol Device:C
- added C50, C51: 4n7, Capacitor_SMD:C_0603_1608Metric_Pad1.08x0.95mm_HandSolder, symbol Device:C
- added C52, C62: 3n3, Capacitor_SMD:C_0603_1608Metric_Pad1.08x0.95mm_HandSolder, symbol Device:C
- added C53, C60: 10n, Capacitor_SMD:C_1206_3216Metric_Pad1.33x1.80mm_HandSolder, symbol Device:C
- added C54: 4u7, Capacitor_SMD:C_1206_3216Metric_Pad1.33x1.80mm_HandSolder, symbol Device:C
- added D10, D23, D8, D9: RED, ASMM-CR03-BU802:LEDM3528X210N, symbol PCM_SL_Devices:LED
- added D11, D12, D13, D29, D31: 5V6, DDZ5V6ASF-7:SODFL2512X75N, symbol Device:D_Zener_Filled
- added D14, D17: PTVS14VP1UP,115, PMEG3050EP115, symbol PTVS14VP1UP,115:PTVS14VP1UP,115
- added D15, D18: 1N4148W, 1N4148W:SODFL3816X120N, symbol PCM_Diode_AKL:1N4148W
- added D16, D22: 16V, MMSZ3V9T1G:SOD3716X135N, symbol Device:D_Zener_Filled
- added D19: V5N3202HM3/I, V5N3202HM3-I:DFN33A_VIS, symbol V5N3202HM3-I:V5N3202HM3_I
- added D20, D30, D32: 18V, MMSZ3V9T1G:SOD3716X135N, symbol Device:D_Zener_Filled
- added D21: 3V9, MMSZ3V9T1G:SOD3716X135N, symbol Device:D_Zener_Filled
- added D24, D25, D26, D27, D28: GREEN, ASMM-CR03-BU802:LEDM3528X210N, symbol PCM_SL_Devices:LED
- added E1: SparkGap, symbol Device:SparkGap
- added FB3, FB4, FB5, FB6: 220R, symbol Device:FerriteBead_Small
- added NT2: NetTie_2, symbol Device:NetTie_2
- added Q10, Q12, Q15: BSS123, symbol PCM_Transistor_MOSFET_AKL:BSS123
- added Q11, Q14, Q7: ZXMP10A13F, symbol PCM_Transistor_MOSFET_AKL:ZXMP10A13F
- added Q13: BCX56, symbol Transistor_BJT:BCX56
- added Q2, Q3, Q4: DMN2004K, symbol PCM_Transistor_MOSFET_AKL:DMN2004K
- added Q5, Q6, Q8, Q9: CSD19531Q5A, symbol Transistor_FET:CSD19531Q5A
- added R14, R15, R16, R22, R24, R25, R26, R29, R30, R31, R32, R47, R51: 1k, symbol Device:R
- added R17, R18, R19: 33R, symbol Device:R
- added R20, R21, R23, R28: 10k, symbol Device:R
- added R27, R40, R41, R46, R49: 10M, symbol Device:R
- added R33, R34, R39, R58, R60, R61, R62, R70, R76, R77: 100R, symbol Device:R
- added R35, R36, R37, R38: 2m, symbol Device:R
- added R42, R44, R52, R57, R59, R66, R74, R78: 100k, symbol Device:R
- added R43, R45: 4k7, symbol Device:R
- added R48, R63, R65: 1M, symbol Device:R
- added R50, R56, R79: 510k, symbol Device:R
- added R53, R54, R64, R71: 300k±0.1%, symbol Device:R
- added R55, R75: 10k±0.1%, symbol Device:R
- added R67, R68: 0R, symbol Device:R
- added R69: 220k, symbol Device:R
- added R72, R73, R80: 620R, symbol Device:R
- added SW6: SW_Push, symbol Switch:SW_Push
- added TH1: 10k NTC, symbol Device:Thermistor
- added TP19, TP20, TP21, TP22, TP23, TP24, TP25, TP26, TP27, TP28, TP29, TP30, TP31, TP32, TP33, TP34, TP35: TestPoint, symbol Connector:TestPoint
- added U10, U9: TPD1E05U06DYA, symbol Power_Protection:TPD1E05U06DYA
- added U6: BQ7692000PWR, Package_SO:TSSOP-20_4.4x6.5mm_P0.65mm, symbol Battery_Management:BQ76920PW
- added U7: BQ78350DBT-R1A, symbol Battery_Management:BQ78350DBT-R1
- added U8: BQ76200PW, symbol Battery_Management:BQ76200PW
Connections:
- net ALERT: now also R51.2, U7.2 (ALERT)
- net BAT: now also C43.2, C44.2, C62.1, R33.2, R71.2, R75.2, U6.10 (BAT), U6.9 (REGSRC), U7.7 (BAT)
- net BATT+: now also C38.1, D14.1 (A1), D16.2 (A), Q5.1 (S), Q5.2 (S), Q5.3 (S), Q6.1 (S), Q6.2 (S), Q6.3 (S), R27.2, R29.1, R30.1, R31.1, R32.1, R58.2
- net BATT-: now also D14.2 (A2), NT2.2, R34.1, R35.1, R36.1, R37.1, R38.1, TP25.1
- net C0: now also D13.2 (A), Q4.2 (S), R24.1
- net C1: now also D10.2, D12.2 (A), Q3.2 (S), R19.2, R22.1
- net C2: now also D11.2 (A), D9.2, Q2.2 (S), R18.2, R26.1
- net C3: now also C42.1, D15.2 (A), D30.1 (K), D8.2, Q14.2 (S), R17.2, R25.1, R28.1, R66.2, R67.2
- net CAP1: now also C45.2, R68.2, U6.7 (CAP1)
- net CHG: now also D16.1 (K), FB3.1, FB4.1, R27.1, R73.2, TP31.1
- net CHG_EN: now also U6.2 (CHG), U8.4 (CHG_EN)
- net CP_EN: now also R79.1, TP27.1, U7.15 (PWRM), U8.5 (CP_EN)
- net DSG: now also D22.1 (K), FB5.2, FB6.2, R46.2, R80.2, TP32.1
- net DSG_EN: now also U6.1 (DSG), U8.6 (DSG_EN)
- net PACK+: now also C40.2, C49.2, D17.1 (A1), D19.5, D19.6, D19.7, D19.8, D20.1 (K), D22.2 (A), E1.2, Q11.2 (S), Q8.1 (S), Q8.2 (S), Q8.3 (S), Q9.1 (S), Q9.2 (S), Q9.3 (S), R41.1, R46.1, R62.1
- net PACK-: now also C48.1, D17.2 (A2), D19.1, D19.2, D19.3, D19.4, E1.1, R35.2, R36.2, R37.2, R38.2, R39.1, TP26.1, U10.2 (GND), U9.2 (GND)
- net PACKDIV: now also R53.2, TP30.1, U8.10 (PACKDIV)
- net PCHG: now also Q5.5 (D), Q6.5 (D), Q7.1 (G), Q8.5 (D), Q9.5 (D), R40.1, R72.2, TP33.1
- net PCHG_EN: now also R56.1, TP28.1, U7.5 (~{PRECHG}), U8.8 (PCHG_EN)
- net PMON_EN: now also Q15.1 (G), R57.1, TP29.1, U7.12 (VEN), U8.7 (PMON_EN)
- net REGOUT: now also C46.2, C54.1, C55.1, C56.1, R43.2, R45.2, R47.1, R52.2, R56.2, R57.2, R59.2, R69.2, R79.2, U6.8 (REGOUT), U7.26 (VCC)
- net SCL: now also R45.1, U6.5 (SCL), U7.4 (SCL)
- net SDA: now also R43.1, U6.4 (SDA), U7.3 (SDA)
- net SMBC: now also R77.2, U9.1 (I/O)
- net SMBD: now also R76.2, U10.1 (I/O)
- net SRN: now also C39.2, C41.1, R39.2, TP24.1, U6.19 (SRN)
- net SRP: now also C37.2, C39.1, R34.2, TP23.1, U6.18 (SRP)
- net TS1: now also D18.1 (K)
- net VC0: now also C35.2, C36.1, R23.2, R24.2, TP22.1, U6.17 (VC0)
- net VC1: now also C34.2, C35.1, R21.2, R22.2, TP21.1, U6.16 (VC1)
- net VC2: now also C33.2, C34.1, R20.2, R26.2, TP20.1, U6.13 (VC4), U6.14 (VC3), U6.15 (VC2)
- net VC5: now also C33.1, R25.2, TP19.1, U6.12 (VC5)
- new net: Q2.3 (D), R15.2, R17.1
- new net: D27.1, U7.19 (LED4)
- new net: C58.1, C59.1, D24.2, D25.2, D26.2, D27.2, D28.2, Q13.3 (E), TP34.1
- new net: FB5.1, Q8.4 (G)
- new net: C48.2, C49.1
- new net: R60.1, U7.11 (SMBD)
- new net: D31.1 (K), R60.2, R65.2, R76.1
- new net: C38.2, C40.1
- new net: Q7.2 (S), R40.2
- new net: Q7.3 (D), R29.2, R30.2, R31.2, R32.2
- new net: FB4.2, Q6.4 (G)
- new net: R61.1, U7.13 (SMBC)
- new net: R69.1, SW6.1, TP35.1, U7.14 (~{DISP})
- new net: D24.1, U7.16 (LED1)
- new net: D25.1, U7.17 (LED2)
- new net: D26.1, U7.18 (LED3)
- new net: D28.1, U7.20 (LED5)
- new net: R59.1, U7.24 (~{MRST})
- new net: C57.1, U7.27 (RBI)
- new net: C52.1, R54.1, R55.2, U7.6 (VAUX)
- new net: D8.1, R15.1
- new net: Q13.1 (B), R68.1
- new net: Q13.2 (C), R67.1
- new net: D32.1 (K), R80.1, U8.12 (DSG)
- new net: FB6.1, Q9.4 (G)
- new net: Q15.3 (D), R78.2
- new net: R72.1, U8.14 (PCHG)
- new net: D30.2 (A), Q14.1 (G), R66.1, R74.1
- new net: R73.1, U8.16 (CHG)
- new net: C47.1, R50.1, R51.1, U6.20 (ALERT)
- new net: C50.1, C51.1, TH1.1, U6.6 (TS1)
- new net: Q10.1 (G), Q12.3 (D), R48.2, R49.1
- new net: C60.1, R62.2, R70.1, U8.11 (PACK)
- new net: D13.1 (K), Q4.1 (G), R23.1
- new net: Q4.3 (D), R14.2, R19.1
- new net: Q10.2 (S), R42.1, R44.1
- new net: Q10.3 (D), Q11.3 (D), R48.1
- new net: D23.2, R47.2
- new net: R74.2, R78.1
- new net: D10.1, R14.1
- new net: C42.2, D20.2 (A), Q11.1 (G), R41.2
- new net: D32.2 (A), R70.2
- new net: R53.1, R54.2
- new net: D29.1 (K), R61.2, R63.2, R77.1
- new net: D9.1, R16.1
- new net: Q3.3 (D), R16.2, R18.1
- new net: D18.2 (A), D21.1 (K), R42.2, R44.2
- new net: C61.1, U8.1 (VDDCP)
- new net: C53.1, C61.2, R58.1, U8.2 (BAT)
- new net: R64.2, R71.1
- new net: D15.1 (K), R28.2, R33.1
- new net: D11.1 (K), Q2.1 (G), R20.1
- new net: FB3.2, Q5.4 (G)
- new net: Q12.1 (G), R52.1
- new net: Q14.3 (D), R64.1
- new net: D12.1 (K), Q3.1 (G), R21.1
- new net GND: C36.2, C37.1, C41.2, C43.1, C44.1, C45.1, C46.1, C47.2, C50.2, C51.2, C52.2, C53.2, C54.2, C55.2, C56.2, C57.2, C58.2, C59.2, C60.2, C62.2, D21.2 (A), D23.1, D29.2 (A), D31.2 (A), NT2.1, Q12.2 (S), Q15.2 (S), R49.2, R50.2, R55.1, R63.1, R65.1, R75.1, SW6.2, TH1.2, U6.3 (VSS), U7.21 (GPIO_A), U7.22 (VSS), U7.23 (VSS), U7.25 (VSS), U7.28 (GPIO_B), U7.30 (SMBA), U7.8 (~{PRES}), U7.9 (~{KEYIN}), U8.9 (VSS)
- no-connect marks 0 -> 3
Other:
- removed sheet BMS Thermistors
- removed sheet Balancing - BMC (AFE)
- removed sheet Current Sense Filtering
- removed sheet Fuel Gauge
- removed sheet High Side Gate Driver
- removed sheet High Voltage REGSRC Supply
- removed sheet Pack Switching and Current Sensing
- removed sheet Passive Balancing Circuit
- removed sheet Wake Up
- note added: "*** REDO THE CALCULATIONS ***"
- note added: ">2W resistors"
- note added: "BMS Protection Board for 3S Battery Pack In/Out: min voltage: 9.6 V, nominal voltage: 11.1 V, max voltage: 12.6 V Output: 20A continuous discharge current Min Each Cell set to 3.2 V, Max Each Cell set to 4.2 V"
- note added: "Balancing & BMC (AFE)"
- note added: "Flash this with TI's software, will need to connec to computer with SMB to USB adapter, could use the expensive one from TI, but $$$"
- note added: "From slua810"
- note added: "From slusc16b"
- note added: "From slva729a VDDCP was picked"
- note added: "From slva729a with extra protection from tida-00792"
- note added: "From slvu925c"
- note added: "Fuel Gauge"
- note added: "High-Side Gate Driver"
- note added: "Pack Switching and Current Sensing"
- note added: "Thermistors"
- note added: "VC0-VSS (Vin max 3V6)"
- note added: "Wake-Up"
- note added: "from TIDA-00792"
- note added: "from TIDUCN1"
- note added: "system is on LED"
- note removed: "BMS Protection Board for 8S Battery Pack In/Out: min voltage: 25.6 V, nominal voltage: 29.6 V, max voltage: 33.6 V Output: 50A continuous discharge current Min Each Cell set to 3.2V, Max Each Cell set to 4.2V"

Commit message: now need 6V Line
Parts:
- added C10, C100, C101, C102, C103, C104, C105, C15, C16, C26, C28, C30, C31, C32, C39, C42, C43, C74, C87, C88, C89, C9, C90, C91, C93, C94, C97, C98, C99: 10u, symbol Device:C
- added C106, C107: 47n, symbol Device:C
- added C108, C56, C57: 4u7, symbol Device:C
- added C12, C22, C33, C37, C41, C44, C5, C58, C60, C76, C82, C83, C86, C92, C96: 100n, symbol Device:C
- added C34, C35: 330p, symbol Device:C
- added C45, C46, C6, C75: 1u, symbol Device:C
- added C47, C48, C49, C50: 10n, symbol Device:C
- added C77: 33p, symbol Device:C
- added C78, C79, C80, C81, C84, C85: 22u, symbol Device:C
- added C95: 1000p, symbol Device:C
- added D18, D19: 82306050029, 82306050029:WESURGE_0603134, symbol 82306050029:82306050029
- added D21: RED, ASMM-CR03-BU802:LEDM3528X210N, symbol PCM_SL_Devices:LED
- added FB5: 21R, symbol Device:FerriteBead_Small
- added J5, J6: Conn_01x04, symbol Connector_Generic:Conn_01x04
- added J7: USB_C_Receptacle_USB2.0_14P, symbol Connector:USB_C_Receptacle_USB2.0_14P
- added JP1, JP2: SolderJumper_2_Bridged, symbol Jumper:SolderJumper_2_Bridged
- added L1: SDR1806-2R2ML, SDR1806-2R2ML:SDR18062R2ML, symbol SDR1806-2R2ML:SDR1806-2R2ML
- added L2: VLS6045EX-1R0N, VLS6045, symbol VLS6045EX-1R0N:VLS6045EX-1R0N
- added NT3: NetTie_2, symbol Device:NetTie_2
- added R1, R18, R2, R3: 10k, symbol Device:R
- added R32, R33: 3k3, symbol Device:R
- added R34, R85, R91: 100k, symbol Device:R
- added R66: 220k, symbol Device:R
- added R67: 30k, symbol Device:R
- added R86: 100R, symbol Device:R
- added R87: 330R, symbol Device:R
- added R88: 10k5, symbol Device:R
- added R89: 4k7, symbol Device:R
- added R90: 137k, symbol Device:R
- added R92: 5k3, symbol Device:R
- added R94: 30k1, symbol Device:R
- added TH2: 10k NTC, symbol Device:Thermistor
- added TP20, TP21, TP22, TP23, TP24, TP25, TP26, TP27, TP28, TP29: TestPoint, symbol Connector:TestPoint
- added U1, U2, U22, U23, U24, U25, U26, U27, U3, U4, U5, U6: 1043, 1043:1043, symbol 1043:1043
- added U10: TVS2200DRV, symbol Power_Protection:TVS2200DRV
- added U12: TLV75533PDBV, Package_TO_SOT_SMD:SOT-23-5, symbol Regulator_Linear:TLV75533PDBV
- added U16: BQ25798RQMR, BQ25798RQMR:BQ25798RQMR, symbol BQ25798RQMR:BQ25798RQMR
- added U28: TPS566238PRQFR, TPS566238PRQFR:TPS566238PRQFR, symbol TPS566238PRQFR:TPS566238PRQFR
- added U7: CAT24C512WI-GT3, symbol CAT24C512WI:CAT24C512WI-GT3
- added U9: TPS25751DREFR, symbol TPS25751DREFR:TPS25751DREFR
- C1: renamed from C33; footprint Capacitor_SMD:C_0805_2012Metric_Pad1.18x1.45mm_HandSolder -> (none); Link https://mou.sr/42gipOV -> (none); Manufacturer Part Number CL21B224KBFNFNE -> (none); Price per Unit 0.10 -> (none); Supplier Mouser -> (none); Supplier Part Number 187-CL21B224KBFNFNE -> (none)
- C11: renamed from C39; footprint Capacitor_SMD:C_1206_3216Metric_Pad1.33x1.80mm_HandSolder -> (none); Link https://mou.sr/4n9ybmQ -> (none); Manufacturer Part Number CL31B104KBCNNNC -> (none); Price per Unit 0.11 -> (none); Supplier Mouser -> (none); Supplier Part Number 187-CL31B104KBCNNNC -> (none)
- C13: renamed from C40; footprint Capacitor_SMD:C_1206_3216Metric_Pad1.33x1.80mm_HandSolder -> (none); Link https://mou.sr/4n9ybmQ -> (none); Manufacturer Part Number CL31B104KBCNNNC -> (none); Price per Unit 0.11 -> (none); Supplier Mouser -> (none); Supplier Part Number 187-CL31B104KBCNNNC -> (none)
- C14: renamed from C41; footprint Capacitor_SMD:C_1206_3216Metric_Pad1.33x1.80mm_HandSolder -> (none); Link https://mou.sr/4n9ybmQ -> (none); Manufacturer Part Number CL31B104KBCNNNC -> (none); Price per Unit 0.11 -> (none); Supplier Mouser -> (none); Supplier Part Number 187-CL31B104KBCNNNC -> (none)
- C17: renamed from C42; footprint Capacitor_SMD:C_0603_1608Metric_Pad1.08x0.95mm_HandSolder -> (none); Link https://mou.sr/3UXYSz1 -> (none); Manufacturer Part Number CL10C471JB8NNND -> (none); Price per Unit 0.10 -> (none); Supplier Mouser -> (none); Supplier Part Number 187-CL10C471JB8NNND -> (none)
- C18: renamed from C43; footprint Capacitor_SMD:C_1206_3216Metric_Pad1.33x1.80mm_HandSolder -> (none); Link https://mou.sr/41y0aEA -> (none); Manufacturer Part Number CL31B105KBHNNNE -> (none); Price per Unit 0.11 -> (none); Supplier Mouser -> (none); Supplier Part Number 187-CL31B105KBHNNNE -> (none)
- C19: renamed from C44; footprint Capacitor_SMD:C_1206_3216Metric_Pad1.33x1.80mm_HandSolder -> (none); Link https://mou.sr/4l54Mdx -> (none); Manufacturer Part Number CL31A106KBHNNNE -> (none); Price per Unit 0.11 -> (none); Supplier Mouser -> (none); Supplier Part Number 187-CL31A106KBHNNNE -> (none)
- C2: renamed from C34; footprint Capacitor_SMD:C_0805_2012Metric_Pad1.18x1.45mm_HandSolder -> (none); Link https://mou.sr/42gipOV -> (none); Manufacturer Part Number CL21B224KBFNFNE -> (none); Price per Unit 0.10 -> (none); Supplier Mouser -> (none); Supplier Part Number 187-CL21B224KBFNFNE -> (none)
- C20: renamed from C45; footprint Capacitor_SMD:C_1206_3216Metric_Pad1.33x1.80mm_HandSolder -> (none); Link https://mou.sr/41y0aEA -> (none); Manufacturer Part Number CL31B105KBHNNNE -> (none); Price per Unit 0.11 -> (none); Supplier Mouser -> (none); Supplier Part Number 187-CL31B105KBHNNNE -> (none)
- C21: renamed from C46; footprint Capacitor_SMD:C_1206_3216Metric_Pad1.33x1.80mm_HandSolder -> (none); Link https://mou.sr/4l54Mdx -> (none); Manufacturer Part Number CL31A106KBHNNNE -> (none); Price per Unit 0.11 -> (none); Supplier Mouser -> (none); Supplier Part Number 187-CL31A106KBHNNNE -> (none)
- C23: renamed from C47; footprint Capacitor_SMD:C_0603_1608Metric_Pad1.08x0.95mm_HandSolder -> (none); Link https://mou.sr/3UXYSz1 -> (none); Manufacturer Part Number CL10C471JB8NNND -> (none); Price per Unit 0.10 -> (none); Supplier Mouser -> (none); Supplier Part Number 187-CL10C471JB8NNND -> (none)
- C24: renamed from C48; footprint Capacitor_SMD:C_1206_3216Metric_Pad1.33x1.80mm_HandSolder -> (none); Link https://mou.sr/4n9ybmQ -> (none); Manufacturer Part Number CL31B104KBCNNNC -> (none); Price per Unit 0.11 -> (none); Supplier Mouser -> (none); Supplier Part Number 187-CL31B104KBCNNNC -> (none)
- C25: renamed from C49; footprint Capacitor_SMD:C_1206_3216Metric_Pad1.33x1.80mm_HandSolder -> (none); Link https://mou.sr/4n9ybmQ -> (none); Manufacturer Part Number CL31B104KBCNNNC -> (none); Price per Unit 0.11 -> (none); Supplier Mouser -> (none); Supplier Part Number 187-CL31B104KBCNNNC -> (none)
- C27: renamed from C50; footprint Capacitor_SMD:C_0603_1608Metric_Pad1.08x0.95mm_HandSolder -> (none); Link https://mou.sr/4g6fuOy -> (none); Manufacturer Part Number CL10B472KB8NFNC -> (none); Price per Unit 0.10 -> (none); Supplier Mouser -> (none); Supplier Part Number 187-CL10B472KB8NFNC -> (none)
- C29: renamed from C51; footprint Capacitor_SMD:C_0603_1608Metric_Pad1.08x0.95mm_HandSolder -> (none); Link https://mou.sr/4g6fuOy -> (none); Manufacturer Part Number CL10B472KB8NFNC -> (none); Price per Unit 0.10 -> (none); Supplier Mouser -> (none); Supplier Part Number 187-CL10B472KB8NFNC -> (none)
- C3: renamed from C35; footprint Capacitor_SMD:C_0805_2012Metric_Pad1.18x1.45mm_HandSolder -> (none); Link https://mou.sr/42gipOV -> (none); Manufacturer Part Number CL21B224KBFNFNE -> (none); Price per Unit 0.10 -> (none); Supplier Mouser -> (none); Supplier Part Number 187-CL21B224KBFNFNE -> (none)
- C36: renamed from C62; footprint Capacitor_SMD:C_0603_1608Metric_Pad1.08x0.95mm_HandSolder -> (none); Link https://mou.sr/3VymwCd -> (none); Manufacturer Part Number CL10B332KB8NNNC -> (none); Price per Unit 0.10 -> (none); Supplier Mouser -> (none); Supplier Part Number 187-CL10B332KB8NNNC -> (none)
- C38: renamed from C53; footprint Capacitor_SMD:C_1206_3216Metric_Pad1.33x1.80mm_HandSolder -> (none); Link https://mou.sr/3OC0xXF -> (none); Manufacturer Part Number CL31B103KHFNFNE -> (none); Price per Unit 0.13 -> (none); Supplier Mouser -> (none); Supplier Part Number 187-CL31B103KHFNFNE -> (none)
- C4: renamed from C36; footprint Capacitor_SMD:C_0805_2012Metric_Pad1.18x1.45mm_HandSolder -> (none); Link https://mou.sr/42gipOV -> (none); Manufacturer Part Number CL21B224KBFNFNE -> (none); Price per Unit 0.10 -> (none); Supplier Mouser -> (none); Supplier Part Number 187-CL21B224KBFNFNE -> (none)
- C40: renamed from C52; footprint Capacitor_SMD:C_0603_1608Metric_Pad1.08x0.95mm_HandSolder -> (none); Link https://mou.sr/3VymwCd -> (none); Manufacturer Part Number CL10B332KB8NNNC -> (none); Price per Unit 0.10 -> (none); Supplier Mouser -> (none); Supplier Part Number 187-CL10B332KB8NNNC -> (none)
- C51: renamed from C60; footprint Capacitor_SMD:C_1206_3216Metric_Pad1.33x1.80mm_HandSolder -> (none); Link https://mou.sr/3OC0xXF -> (none); Manufacturer Part Number CL31B103KHFNFNE -> (none); Price per Unit 0.13 -> (none); Supplier Mouser -> (none); Supplier Part Number 187-CL31B103KHFNFNE -> (none)
- C52: renamed from C61; footprint Capacitor_SMD:C_1206_3216Metric_Pad1.33x1.80mm_HandSolder -> (none); Link https://mou.sr/41y0aEA -> (none); Manufacturer Part Number CL31B105KBHNNNE -> (none); Price per Unit 0.11 -> (none); Supplier Mouser -> (none); Supplier Part Number 187-CL31B105KBHNNNE -> (none)
- C53: renamed from C54; footprint Capacitor_SMD:C_1206_3216Metric_Pad1.33x1.80mm_HandSolder -> (none); Link https://mou.sr/45jYGQI -> (none); Manufacturer Part Number CL31B475KBHNFNE -> (none); Price per Unit 0.27 -> (none); Supplier Mouser -> (none); Supplier Part Number 187-CL31B475KBHNFNE -> (none)
- C54: renamed from C55; footprint Capacitor_SMD:C_1206_3216Metric_Pad1.33x1.80mm_HandSolder -> (none); Link https://mou.sr/41y0aEA -> (none); Manufacturer Part Number CL31B105KBHNNNE -> (none); Price per Unit 0.11 -> (none); Supplier Mouser -> (none); Supplier Part Number 187-CL31B105KBHNNNE -> (none)
- C55: renamed from C56; footprint Capacitor_SMD:C_1206_3216Metric_Pad1.33x1.80mm_HandSolder -> (none); Link https://mou.sr/4n9ybmQ -> (none); Manufacturer Part Number CL31B104KBCNNNC -> (none); Price per Unit 0.11 -> (none); Supplier Mouser -> (none); Supplier Part Number 187-CL31B104KBCNNNC -> (none)
- C59: renamed from C57; footprint Capacitor_SMD:C_1206_3216Metric_Pad1.33x1.80mm_HandSolder -> (none); Link https://mou.sr/4n9ybmQ -> (none); Manufacturer Part Number CL31B104KBCNNNC -> (none); Price per Unit 0.11 -> (none); Supplier Mouser -> (none); Supplier Part Number 187-CL31B104KBCNNNC -> (none)
- C61: renamed from C58; footprint Capacitor_SMD:C_1206_3216Metric_Pad1.33x1.80mm_HandSolder -> (none); Link https://mou.sr/41y0aEA -> (none); Manufacturer Part Number CL31B105KBHNNNE -> (none); Price per Unit 0.11 -> (none); Supplier Mouser -> (none); Supplier Part Number 187-CL31B105KBHNNNE -> (none)
- C62: renamed from C59; footprint Capacitor_SMD:C_1206_3216Metric_Pad1.33x1.80mm_HandSolder -> (none); Link https://mou.sr/4n9ybmQ -> (none); Manufacturer Part Number CL31B104KBCNNNC -> (none); Price per Unit 0.11 -> (none); Supplier Mouser -> (none); Supplier Part Number 187-CL31B104KBCNNNC -> (none)
- C7: renamed from C37; footprint Capacitor_SMD:C_1206_3216Metric_Pad1.33x1.80mm_HandSolder -> (none); Link https://mou.sr/4n9ybmQ -> (none); Manufacturer Part Number CL31B104KBCNNNC -> (none); Price per Unit 0.11 -> (none); Supplier Mouser -> (none); Supplier Part Number 187-CL31B104KBCNNNC -> (none)
- C8: renamed from C38; footprint Capacitor_SMD:C_1206_3216Metric_Pad1.33x1.80mm_HandSolder -> (none); Link https://mou.sr/4n9ybmQ -> (none); Manufacturer Part Number CL31B104KBCNNNC -> (none); Price per Unit 0.11 -> (none); Supplier Mouser -> (none); Supplier Part Number 187-CL31B104KBCNNNC -> (none)
- D10: renamed from D17; footprint PMEG3050EP115 -> PTVS14VP1UP,115:PMEG3050EP115
- D7: renamed from D14; footprint PMEG3050EP115 -> PTVS14VP1UP,115:PMEG3050EP115
- renumbered D8 to D1, D18 to D11, D19 to D12, D20 to D13, D21 to D14, D22 to D15, D23 to D16, D30 to D17, D9 to D2, D32 to D20, D24 to D22, D25 to D23, D26 to D24, D27 to D25, D28 to D26, D29 to D27, D31 to D28, D10 to D3, D11 to D4, D12 to D5, D13 to D6, D15 to D8, D16 to D9, FB3 to FB1, FB4 to FB2, FB5 to FB3, FB6 to FB4, NT2 to NT1, Q2 to Q1, Q11 to Q10, Q12 to Q11, Q14 to Q12, Q15 to Q13, Q13 to Q14, Q3 to Q2, Q4 to Q3, Q5 to Q4, Q6 to Q5, Q7 to Q6, Q8 to Q7, Q9 to Q8, Q10 to Q9, R20 to R10, R21 to R11, R22 to R12, R23 to R13, R24 to R14, R25 to R15, R26 to R16, R27 to R17, R28 to R19, R29 to R20, R30 to R21, R31 to R22, R32 to R23, R33 to R24, R34 to R25, R35 to R26, R36 to R27, R37 to R28, R38 to R29, R39 to R30, R40 to R31, R41 to R35, R42 to R36, R43 to R37, R44 to R38, R45 to R39, R14 to R4, R46 to R40, R47 to R41, R48 to R42, R49 to R43, R50 to R44, R51 to R45, R52 to R46, R64 to R47, R66 to R48, R71 to R49, R15 to R5, R53 to R50, R74 to R51, R75 to R52, R54 to R53, R58 to R54, R78 to R55, R55 to R56, R56 to R57, R57 to R58, R62 to R59, R16 to R6, R59 to R60, R70 to R61, R72 to R62, R73 to R63, R60 to R64, R61 to R65, R63 to R68, R65 to R69, R17 to R7, R80 to R70, R67 to R71, R68 to R72, R69 to R73, R76 to R74, R77 to R75, R79 to R76, R18 to R8, R19 to R9, SW6 to SW2, TP19 to TP12, TP20 to TP13, TP21 to TP14, TP22 to TP15, TP23 to TP16, TP24 to TP17, TP25 to TP18, TP26 to TP19, TP27 to TP30, TP28 to TP31, TP29 to TP32, TP30 to TP33, TP31 to TP34, TP32 to TP35, TP33 to TP36, TP34 to TP37, TP35 to TP38, U8 to U11, U7 to U13, U9 to U14, U10 to U15, U6 to U8
Connections:
- net C0 is gone; now on net BATT-: D6.2 (A), Q3.2 (S), R14.1
- net C3 is gone; now on net BATT+: C17.1, D1.2, D17.1 (K), D8.2 (A), Q12.2 (S), R15.1, R19.1, R48.2, R7.2, R71.2
- net BATT+: now also U1.1 (+), U22.1 (+), U25.1 (+), U4.1 (+)
- net BATT-: now also U24.2 (-), U27.2 (-), U3.2 (-), U6.2 (-)
- net C1: now also U2.2 (-), U23.2 (-), U24.1 (+), U26.2 (-), U27.1 (+), U3.1 (+), U5.2 (-), U6.1 (+)
- net C2: now also U1.2 (-), U2.1 (+), U22.2 (-), U23.1 (+), U25.2 (-), U26.1 (+), U4.2 (-), U5.1 (+)
- net GND: now also C10.2, C100.2, C101.2, C102.2, C103.2, C104.2, C105.2, C108.2, C12.2, C15.2, C16.2, C22.2, C26.2, C28.2, C30.2, C31.2, C32.2, C33.2, C34.2, C35.2, C37.2, C39.2, C41.2, C42.2, C43.2, C44.2, C45.2, C46.2, C47.1, C48.1, C49.1, C5.2, C50.1, C56.2, C57.2, C58.2, C6.2, C60.2, C74.2, C75.2, C78.2, C79.2, C80.2, C81.2, C82.2, C83.2, C84.2, C85.2, C86.2, C87.2, C88.2, C89.2, C9.2, C90.2, C91.2, C92.2, C93.2, C94.2, C96.2, C97.2, C98.2, C99.2, D18.2 (A2), D19.2 (A2), J5.1 (Pin_1), J6.1 (Pin_1), J7.A1 (GND), J7.A12 (GND), J7.B1 (GND), J7.B12 (GND), J7.S1 (SHIELD), NT3.1, R1.1, R18.1, R2.1, R3.1, R67.2, U10.1 (GND), U10.2 (GND), U10.3 (GND), U10.7 (GND), U12.2 (GND), U16.27 (GND), U28.4 (PGND), U7.4 (VSS), U9.10 (~{I2Ct_IRQ}), U9.11 (GND), U9.12 (GND), U9.13 (GPIO11), U9.14 (GND), U9.18 (~{I2Cc_IRQ}), U9.19 (GPIO3), U9.3 (ADCIN2), U9.31 (GND), U9.36 (GPIO7), U9.37 (GPIO6), U9.39 (GND), U9.5 (GPIO0), U9.6 (GPIO1), U9.7 (GPIO2)
- net PACK+: now also C83.1, C84.1, C85.1, C86.1, C87.1, C88.1, C89.1, C90.1, C91.1, C92.1, C93.1, C94.1, R86.2, U16.22 (BAT_1), U16.23 (BAT_2), U16.25 (SYS), U28.5 (VIN_1), U28.6 (VIN_2)
- net SCL renamed AFE_SCL
- net SDA renamed AFE_SDA
- new net: R1.2, U7.1 (A0)
- new net: R2.2, U7.2 (A1)
- new net: R3.2, U7.3 (A2)
- new net: R18.2, U7.7 (WP)
- new net: R86.1, U16.18 (BATP)
- new net: J6.2 (Pin_2), U9.9 (I2Ct_SCL)
- new net: J6.3 (Pin_3), U9.8 (I2Ct_SDA)
- new net: C47.2, C48.2, C49.2, C50.2, FB5.1, J7.A4 (VBUS), J7.A9 (VBUS), J7.B4 (VBUS), J7.B9 (VBUS), U10.4 (IN), U10.5 (IN), U10.6 (IN)
- new net: C75.1, R85.1, U28.1 (VCC)
- new net: C76.1, L1.2, U28.8 (SW)
- new net: C102.1, C103.1, C104.1, C105.1, U16.29 (PMID)
- new net: D21.2, R87.1
- new net: C108.1, R90.1, R92.1, U16.5 (REGN)
- new net: R90.2, R91.1, U16.17 (ILIM_HIZ)
- new net: C77.2, R66.2, R67.1, U28.2 (FB)
- new net: R85.2, U28.9 (PG)
- new net: R88.2, U16.20 (PROG)
- new net: JP1.1 (A), U16.6 (D+)
- new net: C76.2, U28.7 (BST)
- new net: JP2.1 (A), U16.7 (D-)
- new net ADCIN1: R34.2, TP24.1, U9.2 (ADCIN1)
- new net BQ25798_GNDA: C95.2, NT3.2, R88.1, R91.2, R94.2, TH2.2, U16.10 (ACDRV2), U16.11 (ACDRV1), U16.13 (~{CE})
- new net BTST1: C106.1, U16.4 (BTST1)
- new net BTST2: C107.1, U16.19 (BTST2)
- new net C_CC1: C34.1, J7.A5 (CC1), TP26.1, U9.28 (CC1)
- new net C_CC2: C35.1, J7.B5 (CC2), TP27.1, U9.29 (CC2)
- new net DRAIN: TP20.1, U9.15 (DRAIN), U9.30 (DRAIN), U9.40 (DRAIN)
- new net LDO_1V5: C15.1, C16.1, C22.1, U9.4 (LDO_1V5)
- new net LDO_3V3: C10.1, C12.1, C5.1, C6.1, C9.1, J6.4 (Pin_4), R32.2, R33.2, R34.1, R87.2, R89.2, U7.8 (VCC), U9.1 (LDO_3V3)
- new net P3V3: C41.1, C42.1, C43.1, C44.1, C45.1, C46.1, TP22.1, U12.5 (OUT), U9.38 (VIN_3V3)
- new net P5V0: C37.1, C39.1, C60.1, C74.1, C77.1, C78.1, C79.1, C80.1, C81.1, C82.1, L1.1, R66.1, TP23.1, U12.1 (IN), U12.3 (EN), U9.34 (PP5V), U9.35 (PP5V)
- new net PD_SCL: J5.2 (Pin_2), R33.1, U16.14 (SCL), U7.6 (SCL), U9.17 (I2Cc_SCL)
- new net PD_SDA: J5.3 (Pin_3), R32.1, U16.15 (SDA), U7.5 (SDA), U9.16 (I2Cc_SDA)
- new net PD_VAC: C100.1, C101.1, C26.1, C28.1, C30.1, C31.1, C32.1, C33.1, C96.1, C97.1, C98.1, C99.1, TP21.1, U16.2 (VBUS_1), U16.3 (VBUS_2), U16.31 (VAC1_2), U16.8 (VAC2), U16.9 (VAC1_1), U9.20 (PPHV), U9.21 (PPHV), U9.22 (PPHV)
- new net SDRV_1_2: C95.1, U16.24 (SDRV_1), U16.33 (SDRV_2)
- new net STAT_1_2: D21.1, R89.1, U16.1 (STAT_1), U16.30 (STAT_2)
- new net SW1: C106.2, L2.1, U16.28 (SW1)
- new net SW2: C107.2, L2.2, U16.26 (SW2)
- new net TS_1_2: R92.2, R94.1, TH2.1, U16.16 (TS_1), U16.32 (TS_2)
- new net USB_C_N: D18.1 (A1), J7.A7 (D-), J7.B7 (D-), JP2.2 (B), TP28.1, U9.27 (GPIO5/USB_N/LD2)
- new net USB_C_P: D19.1 (A1), J7.A6 (D+), J7.B6 (D+), JP1.2 (B), TP29.1, U9.26 (GPIO4/USB_P/LD1)
- new net VBUS: C56.1, C57.1, C58.1, FB5.2, TP25.1, U9.23 (VBUS_IN), U9.24 (VBUS_IN), U9.25 (VBUS_IN), U9.32 (VBUS), U9.33 (VBUS)
- no-connect marks 3 -> 7
Other:
- note added: ""can be used to directly program the TPS25751, and program the BQ25798 through the host microcontroller " ^^^^ for the I2Ct lines (pins 8, 9)"
- note added: "*** VERIFY THIS (esp the d+/-) ***"
- note added: "1010 ???? GND=0 so this: 1010 0000 -> 0x50 which is what we need for our PD controller"
- note added: "500mA 3V3"
- note added: "512Kb"
- note added: "5V/5A"
- note added: "ADCIN1 & ADCIN2 configured for "SafeMode" I2C Target is 0x20"
- note added: "BMS Protection Board for 3S4P Battery Pack In/Out: min voltage: 9.6 V, nominal voltage: 11.1 V, max voltage: 12.6 V Output: 25A continuous discharge current Min Each Cell set to 3.2 V, Max Each Cell set to 4.2 V"
- note added: "Flash this with the bin taken from TI's website. Use I2C to USB adapter. Flash this when the system is off (not powered), only flash/power this."
- note added: "Max Power Sourced = 45W, Sink Power = 60W"
- note added: "TPS25751DREFR will load from EEPROM"
- note added: "internal debugging"
- note added: "pins 15&30 tie to exposed pad 40 for internal fet"
- note removed: "BMS Protection Board for 3S Battery Pack In/Out: min voltage: 9.6 V, nominal voltage: 11.1 V, max voltage: 12.6 V Output: 20A continuous discharge current Min Each Cell set to 3.2 V, Max Each Cell set to 4.2 V"
- moved on the sheet: C1, C11, C13, C14, C17, C18, C19, C2, C20, C21, C23, C24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
