File: Schematic/STAR.kicad_pcb (KiCad board)
At the start: 2 copper layers, 12 parts, among them Q11 CSD19531Q5A, Q13 CSD19531Q5A, Q14 CSD19531Q5A, Q15 BCX56, Q17 BSS84, Q20 BSS138, Q9 CSD19531Q5A, U1 BQ7693006DBTR, U2 BQ76200PW, U3 BQ78350DBT-R1A, U4 TPD1E05U06DYA, U5 TPD1E05U06DYA

Commit message: Started to work on the BOM
Parts:
- removed Q11, Q13, Q14, Q9: CSD19531Q5A, Package_TO_SOT_SMD:TDSON-8-1
- removed Q15: BCX56, Package_TO_SOT_SMD:SOT-89-3
- removed Q17: BSS84, Package_TO_SOT_SMD:SOT-23
- removed Q20: BSS138, Package_TO_SOT_SMD:SOT-23
- removed U1: BQ7693006DBTR, Package_SO:TSSOP-30_4.4x7.8mm_P0.5mm
- removed U3: BQ78350DBT-R1A, Package_SO:TSSOP-30_4.4x7.8mm_P0.5mm
- removed U4, U5: TPD1E05U06DYA, Diode_SMD:D_SOD-523
- added C1: 4u7, Capacitor_SMD:C_1206_3216Metric_Pad1.33x1.80mm_HandSolder, F.Cu at (195.3, 112.2)
- added C10: 100n, Capacitor_SMD:C_1206_3216Metric_Pad1.33x1.80mm_HandSolder, F.Cu at (158.2, 92.4)
- added C100: 4u7, Capacitor_SMD:C_1206_3216Metric_Pad1.33x1.80mm_HandSolder, F.Cu at (108.6, 77.0)
- added C101: 4u7, Capacitor_SMD:C_1206_3216Metric_Pad1.33x1.80mm_HandSolder, F.Cu at (108.6, 80.3)
- added C102: 1u, Capacitor_SMD:C_1206_3216Metric_Pad1.33x1.80mm_HandSolder, F.Cu at (114.6, 56.9)
- added C103: 1u, Capacitor_SMD:C_1206_3216Metric_Pad1.33x1.80mm_HandSolder, F.Cu at (114.6, 60.2)
- added C104: 1u, Capacitor_SMD:C_1206_3216Metric_Pad1.33x1.80mm_HandSolder, F.Cu at (114.6, 63.6)
- added C105: 100n, Capacitor_SMD:C_1206_3216Metric_Pad1.33x1.80mm_HandSolder, F.Cu at (114.6, 66.9)
- added C106: 100n, Capacitor_SMD:C_1206_3216Metric_Pad1.33x1.80mm_HandSolder, F.Cu at (114.6, 70.3)
- added C107: 1u, Capacitor_SMD:C_1206_3216Metric_Pad1.33x1.80mm_HandSolder, F.Cu at (114.6, 73.6)
- added C108: 100n, Capacitor_SMD:C_1206_3216Metric_Pad1.33x1.80mm_HandSolder, F.Cu at (114.6, 77.0)
- added C109: 56u, AHA0810560M040R:CAPAE830X1100M, F.Cu at (141.2, 26.3)
- added C11: 10u, Capacitor_SMD:C_1206_3216Metric_Pad1.33x1.80mm_HandSolder, F.Cu at (158.2, 95.7)
- added C110: 56u, AHA0810560M040R:CAPAE830X1100M, F.Cu at (141.2, 37.9)
- added C111: 56u, AHA0810560M040R:CAPAE830X1100M, F.Cu at (141.2, 49.4)
- added C112: 56u, AHA0810560M040R:CAPAE830X1100M, F.Cu at (155.5, 26.3)
- added C113: 56u, AHA0810560M040R:CAPAE830X1100M, F.Cu at (155.5, 37.9)
- added C114: 56u, AHA0810560M040R:CAPAE830X1100M, F.Cu at (155.5, 49.4)
- added C115: 10u, Capacitor_SMD:C_1206_3216Metric_Pad1.33x1.80mm_HandSolder, F.Cu at (114.6, 80.3)
- added C116: 10u, Capacitor_SMD:C_1206_3216Metric_Pad1.33x1.80mm_HandSolder, F.Cu at (120.6, 56.9)
- added C117: 4u7, Capacitor_SMD:C_1206_3216Metric_Pad1.33x1.80mm_HandSolder, F.Cu at (120.6, 60.2)
- added C118: 4u7, Capacitor_SMD:C_1206_3216Metric_Pad1.33x1.80mm_HandSolder, F.Cu at (120.6, 63.6)
- added C119: 1u, Capacitor_SMD:C_1206_3216Metric_Pad1.33x1.80mm_HandSolder, F.Cu at (120.6, 66.9)
- added C12: 100n, Capacitor_SMD:C_1206_3216Metric_Pad1.33x1.80mm_HandSolder, F.Cu at (158.2, 99.1)
- added C120: 1u, Capacitor_SMD:C_1206_3216Metric_Pad1.33x1.80mm_HandSolder, F.Cu at (120.6, 70.3)
- added C121: 100n, Capacitor_SMD:C_1206_3216Metric_Pad1.33x1.80mm_HandSolder, F.Cu at (120.6, 73.6)
- added C122: 100n, Capacitor_SMD:C_1206_3216Metric_Pad1.33x1.80mm_HandSolder, F.Cu at (120.6, 77.0)
- added C123: 4u7, Capacitor_SMD:C_1206_3216Metric_Pad1.33x1.80mm_HandSolder, F.Cu at (202.9, 85.7)
- added C124: 100n, Capacitor_SMD:C_1206_3216Metric_Pad1.33x1.80mm_HandSolder, F.Cu at (202.9, 89.0)
- added C125: 100n, Capacitor_SMD:C_1206_3216Metric_Pad1.33x1.80mm_HandSolder, F.Cu at (202.9, 92.4)
- added C126: 100n, Capacitor_SMD:C_1206_3216Metric_Pad1.33x1.80mm_HandSolder, F.Cu at (202.9, 95.7)
- added C127: 470n, Capacitor_SMD:C_0805_2012Metric_Pad1.18x1.45mm_HandSolder, F.Cu at (208.3, 85.5)
- added C128: 100n, Capacitor_SMD:C_1206_3216Metric_Pad1.33x1.80mm_HandSolder, F.Cu at (202.9, 99.1)
- added C129: 33p, Capacitor_SMD:C_0603_1608Metric_Pad1.08x0.95mm_HandSolder, F.Cu at (208.0, 91.3)
- added C13: 220n, Capacitor_SMD:C_0805_2012Metric_Pad1.18x1.45mm_HandSolder, F.Cu at (171.9, 85.5)
- added C130: 33p, Capacitor_SMD:C_0603_1608Metric_Pad1.08x0.95mm_HandSolder, F.Cu at (208.0, 93.8)
- added C131: 100n, Capacitor_SMD:C_1206_3216Metric_Pad1.33x1.80mm_HandSolder, F.Cu at (202.9, 102.4)
- added C132: 470n, Capacitor_SMD:C_0805_2012Metric_Pad1.18x1.45mm_HandSolder, F.Cu at (208.3, 88.5)
- added C133: 100n, Capacitor_SMD:C_1206_3216Metric_Pad1.33x1.80mm_HandSolder, F.Cu at (202.9, 105.8)
- added C134: 56u, AHA0810560M040R:CAPAE830X1100M, F.Cu at (90.5, 26.3)
- added C135: 56u, AHA0810560M040R:CAPAE830X1100M, F.Cu at (90.5, 37.9)
- added C136: 56u, AHA0810560M040R:CAPAE830X1100M, F.Cu at (90.5, 49.4)
- added C137: 56u, AHA0810560M040R:CAPAE830X1100M, F.Cu at (90.5, 61.0)
- added C138: 220n, Capacitor_SMD:C_0805_2012Metric_Pad1.18x1.45mm_HandSolder, F.Cu at (100.0, 38.8)
- added C139: 220n, Capacitor_SMD:C_0805_2012Metric_Pad1.18x1.45mm_HandSolder, F.Cu at (100.0, 41.8)
- added C14: 220n, Capacitor_SMD:C_0805_2012Metric_Pad1.18x1.45mm_HandSolder, F.Cu at (171.9, 88.5)
- added C140: 470p, Capacitor_SMD:C_0603_1608Metric_Pad1.08x0.95mm_HandSolder, F.Cu at (99.8, 50.6)
- added C141: 82n, Capacitor_SMD:C_1206_3216Metric_Pad1.33x1.80mm_HandSolder, F.Cu at (100.6, 22.2)
- added C142: 56p, Capacitor_SMD:C_0603_1608Metric_Pad1.08x0.95mm_HandSolder, F.Cu at (99.8, 53.1)
- added C143: 10n, Capacitor_SMD:C_1206_3216Metric_Pad1.33x1.80mm_HandSolder, F.Cu at (100.6, 25.6)
- added C144: 100n, Capacitor_SMD:C_1206_3216Metric_Pad1.33x1.80mm_HandSolder, F.Cu at (100.6, 28.9)
- added C145: 10u, Capacitor_SMD:C_1206_3216Metric_Pad1.33x1.80mm_HandSolder, F.Cu at (100.6, 32.3)
- added C146: 2u2, Capacitor_SMD:C_1206_3216Metric_Pad1.33x1.80mm_HandSolder, F.Cu at (100.6, 35.6)
- added C147: 220n, Capacitor_SMD:C_0805_2012Metric_Pad1.18x1.45mm_HandSolder, F.Cu at (100.0, 44.8)
- added C148: 4n7, Capacitor_SMD:C_0603_1608Metric_Pad1.08x0.95mm_HandSolder, F.Cu at (99.8, 55.6)
- added C149: 100p, Capacitor_SMD:C_0603_1608Metric_Pad1.08x0.95mm_HandSolder, F.Cu at (99.8, 58.1)
- added C15: 220n, Capacitor_SMD:C_0805_2012Metric_Pad1.18x1.45mm_HandSolder, F.Cu at (171.9, 91.5)
- added C150: 56u, AHA0810560M040R:CAPAE830X1100M, F.Cu at (90.5, 72.5)
- added C151: 56u, AHA0810560M040R:CAPAE830X1100M, F.Cu at (90.5, 84.1)
- added C152: 56u, AHA0810560M040R:CAPAE830X1100M, F.Cu at (90.5, 95.6)
- added C153: 220n, Capacitor_SMD:C_0805_2012Metric_Pad1.18x1.45mm_HandSolder, F.Cu at (100.0, 47.8)
- added C154: 56u, AHA0810560M040R:CAPAE830X1100M, F.Cu at (171.7, 26.3)
- added C155: 56u, AHA0810560M040R:CAPAE830X1100M, F.Cu at (171.7, 37.9)
- added C156: 56u, AHA0810560M040R:CAPAE830X1100M, F.Cu at (171.7, 49.4)
- added C157: 56u, AHA0810560M040R:CAPAE830X1100M, F.Cu at (171.7, 61.0)
- added C158: 56u, AHA0810560M040R:CAPAE830X1100M, F.Cu at (171.7, 72.5)
- added C159: 220n, Capacitor_SMD:C_0805_2012Metric_Pad1.18x1.45mm_HandSolder, F.Cu at (195.5, 42.2)
- added C16: 220n, Capacitor_SMD:C_0805_2012Metric_Pad1.18x1.45mm_HandSolder, F.Cu at (171.9, 94.5)
- added C160: 220n, Capacitor_SMD:C_0805_2012Metric_Pad1.18x1.45mm_HandSolder, F.Cu at (195.5, 45.2)
- added C161: 470p, Capacitor_SMD:C_0603_1608Metric_Pad1.08x0.95mm_HandSolder, F.Cu at (195.3, 54.0)
- added C162: 100n, Capacitor_SMD:C_1206_3216Metric_Pad1.33x1.80mm_HandSolder, F.Cu at (196.1, 22.2)
- added C163: 62p, Capacitor_SMD:C_0603_1608Metric_Pad1.08x0.95mm_HandSolder, F.Cu at (195.3, 56.5)
- added C164: 1u, Capacitor_SMD:C_1206_3216Metric_Pad1.33x1.80mm_HandSolder, F.Cu at (196.1, 25.6)
- added C165: 10n, Capacitor_SMD:C_1206_3216Metric_Pad1.33x1.80mm_HandSolder, F.Cu at (196.1, 28.9)
- added C166: 100n, Capacitor_SMD:C_1206_3216Metric_Pad1.33x1.80mm_HandSolder, F.Cu at (196.1, 32.3)
- added C167: 2u2, Capacitor_SMD:C_1206_3216Metric_Pad1.33x1.80mm_HandSolder, F.Cu at (196.1, 35.6)
- added C168: 220n, Capacitor_SMD:C_0805_2012Metric_Pad1.18x1.45mm_HandSolder, F.Cu at (195.5, 48.2)
- added C169: 4n7, Capacitor_SMD:C_0603_1608Metric_Pad1.08x0.95mm_HandSolder, F.Cu at (195.3, 59.0)
- added C17: 220n, Capacitor_SMD:C_0805_2012Metric_Pad1.18x1.45mm_HandSolder, F.Cu at (171.9, 97.5)
- added C170: 100p, Capacitor_SMD:C_0603_1608Metric_Pad1.08x0.95mm_HandSolder, F.Cu at (195.3, 61.5)
- added C171: 56u, AHA0810560M040R:CAPAE830X1100M, F.Cu at (186.0, 26.3)
- added C172: 56u, AHA0810560M040R:CAPAE830X1100M, F.Cu at (186.0, 37.9)
- added C173: 56u, AHA0810560M040R:CAPAE830X1100M, F.Cu at (186.0, 49.4)
- added C174: 56u, AHA0810560M040R:CAPAE830X1100M, F.Cu at (186.0, 61.0)
- added C175: 56u, AHA0810560M040R:CAPAE830X1100M, F.Cu at (186.0, 72.5)
- added C176: 220n, Capacitor_SMD:C_0805_2012Metric_Pad1.18x1.45mm_HandSolder, F.Cu at (195.5, 51.2)
- added C177: 1u, Capacitor_SMD:C_1206_3216Metric_Pad1.33x1.80mm_HandSolder, F.Cu at (166.2, 124.3)
- added C178: 100n, Capacitor_SMD:C_1206_3216Metric_Pad1.33x1.80mm_HandSolder, F.Cu at (166.2, 127.7)
- added C179: 1u, Capacitor_SMD:C_1206_3216Metric_Pad1.33x1.80mm_HandSolder, F.Cu at (166.2, 131.0)
- added C18: 220n, Capacitor_SMD:C_0805_2012Metric_Pad1.18x1.45mm_HandSolder, F.Cu at (176.7, 85.5)
- added C180: 100n, Capacitor_SMD:C_1206_3216Metric_Pad1.33x1.80mm_HandSolder, F.Cu at (166.2, 134.4)
- added C181: 1u, Capacitor_SMD:C_1206_3216Metric_Pad1.33x1.80mm_HandSolder, F.Cu at (166.2, 137.7)
- added C182: 100n, Capacitor_SMD:C_1206_3216Metric_Pad1.33x1.80mm_HandSolder, F.Cu at (166.2, 141.1)
- added C183: 1u, Capacitor_SMD:C_1206_3216Metric_Pad1.33x1.80mm_HandSolder, F.Cu at (166.2, 144.4)
- added C184: 100n, Capacitor_SMD:C_1206_3216Metric_Pad1.33x1.80mm_HandSolder, F.Cu at (166.2, 147.8)
- added C185: 56u, AHA0810560M040R:CAPAE830X1100M, F.Cu at (90.5, 109.2)
- added C186: 220n, Capacitor_SMD:C_0805_2012Metric_Pad1.18x1.45mm_HandSolder, F.Cu at (98.1, 116.5)
- added C187: 100n, Capacitor_SMD:C_1206_3216Metric_Pad1.33x1.80mm_HandSolder, F.Cu at (92.7, 116.6)
- added C188: 56u, AHA0810560M040R:CAPAE830X1100M, F.Cu at (90.5, 127.3)
- added C189: 220n, Capacitor_SMD:C_0805_2012Metric_Pad1.18x1.45mm_HandSolder, F.Cu at (98.1, 134.6)
- added C19: 220n, Capacitor_SMD:C_0805_2012Metric_Pad1.18x1.45mm_HandSolder, F.Cu at (176.7, 88.5)
- added C190: 100n, Capacitor_SMD:C_1206_3216Metric_Pad1.33x1.80mm_HandSolder, F.Cu at (92.7, 134.7)
- added C191: 56u, AHA0810560M040R:CAPAE830X1100M, F.Cu at (90.5, 145.4)
- added C192: 220n, Capacitor_SMD:C_0805_2012Metric_Pad1.18x1.45mm_HandSolder, F.Cu at (98.1, 152.7)
- added C193: 100n, Capacitor_SMD:C_1206_3216Metric_Pad1.33x1.80mm_HandSolder, F.Cu at (92.7, 152.8)
- added C194: 56u, AHA0810560M040R:CAPAE830X1100M, F.Cu at (199.4, 141.7)
- added C195: 220n, Capacitor_SMD:C_0805_2012Metric_Pad1.18x1.45mm_HandSolder, F.Cu at (207.0, 149.0)
- added C196: 100n, Capacitor_SMD:C_1206_3216Metric_Pad1.33x1.80mm_HandSolder, F.Cu at (201.6, 149.2)
- added C197: 100p, Capacitor_SMD:C_0603_1608Metric_Pad1.08x0.95mm_HandSolder, F.Cu at (205.6, 128.9)
- added C198: 100n, Capacitor_SMD:C_1206_3216Metric_Pad1.33x1.80mm_HandSolder, F.Cu at (206.4, 126.0)
- added C199: 100p, Capacitor_SMD:C_0603_1608Metric_Pad1.08x0.95mm_HandSolder, F.Cu at (205.6, 131.4)
- added C2: 4u7, Capacitor_SMD:C_1206_3216Metric_Pad1.33x1.80mm_HandSolder, F.Cu at (195.3, 115.5)
- added C20: 220n, Capacitor_SMD:C_0805_2012Metric_Pad1.18x1.45mm_HandSolder, F.Cu at (176.7, 91.5)
- added C200: 100n, Capacitor_SMD:C_1206_3216Metric_Pad1.33x1.80mm_HandSolder, F.Cu at (141.0, 146.0)
- added C201: 100n, Capacitor_SMD:C_1206_3216Metric_Pad1.33x1.80mm_HandSolder, F.Cu at (141.0, 149.3)
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Connections:
- net /BMS Protection Board/PACKDIV renamed /SPI_SDI
- net Net-(D37-K) renamed /I2C_SDA
- net Net-(U2-PACK) renamed /SPI_SDO
- U2 pad 1: Net-(U2-VDDCP) -> GND
- U2 pad 13: unconnected-(U2-NC-Pad13) -> /MCU/USB_C_N
- U2 pad 14: Net-(U2-PCHG) -> /MCU/USB_C_P
- U2 pad 15: unconnected-(U2-NC-Pad15) -> /MCU/IO_RST
- U2 pad 16: Net-(U2-CHG) -> unconnected-(U2-IO46-Pad16)
- U2 pad 2: Net-(U2-BAT) -> /SENSOR_P3V3
- U2 pad 3: unconnected-(U2-NC-Pad3) -> /MCU/ESP32/RST
- U2 pad 4: /BMS Protection Board/CHG_EN -> /MOTOR_EN_DATA
- U2 pad 5: /BMS Protection Board/CP_EN -> /MOTOR_PH_DATA
- U2 pad 6: /BMS Protection Board/DSG_EN -> /MCU/ESP32/IO6
- U2 pad 7: /BMS Protection Board/PMON_EN -> /I2C_SCL
- U2 pad 8: /BMS Protection Board/PCHG_EN -> /MOTORx_nFAULT
- U2 pad 9: GND -> /SPI_SCLK

Commit message: Massive pivit, simplification
Parts:
- removed C1, C100, C101, C117, C118, C123, C206, C98, C99: 4u7, Capacitor_SMD:C_1206_3216Metric_Pad1.33x1.80mm_HandSolder
- removed C102, C103, C104, C107, C119, C120, C164, C177, C179, C181, C183, C23, C25, C83, C84, C85, C86, C9: 1u, Capacitor_SMD:C_1206_3216Metric_Pad1.33x1.80mm_HandSolder
- removed C105, C106, C108, C121, C122, C124, C125, C126, C128, C131, C133, C144, C162, C166, C178, C180, C182, C184, C187, C190, C193, C196, C198, C200, C201, C202, C203, C204, C207, C28, C29, C30, C31, C32, C74, C77, C79, C82, C87, C88, C89: 100n, Capacitor_SMD:C_1206_3216Metric_Pad1.33x1.80mm_HandSolder
- removed C109, C110, C111, C112, C113, C114, C134, C135, C136, C137, C150, C151, C152, C154, C155, C156, C157, C158, C171, C172, C173, C174, C175, C185, C188, C191, C194, C90, C91, C92, C93, C94, C95: 56u, AHA0810560M040R:CAPAE830X1100M
- removed C115, C116, C145, C24, C26, C78, C80, C81, C96, C97: 10u, Capacitor_SMD:C_1206_3216Metric_Pad1.33x1.80mm_HandSolder
- removed C127, C132, C205: 470n, Capacitor_SMD:C_0805_2012Metric_Pad1.18x1.45mm_HandSolder
- removed C129, C130: 33p, Capacitor_SMD:C_0603_1608Metric_Pad1.08x0.95mm_HandSolder
- removed C13, C138, C139, C14, C147, C15, C153, C159, C160, C168, C17, C176, C186, C189, C19, C192, C195, C20, C21, C22: 220n, Capacitor_SMD:C_0805_2012Metric_Pad1.18x1.45mm_HandSolder
- removed C140, C161, C27: 470p, Capacitor_SMD:C_0603_1608Metric_Pad1.08x0.95mm_HandSolder
- removed C141: 82n, Capacitor_SMD:C_1206_3216Metric_Pad1.33x1.80mm_HandSolder
- removed C142: 56p, Capacitor_SMD:C_0603_1608Metric_Pad1.08x0.95mm_HandSolder
- removed C143, C165: 10n, Capacitor_SMD:C_1206_3216Metric_Pad1.33x1.80mm_HandSolder
- removed C146, C167, L3: 2u2, Capacitor_SMD:C_1206_3216Metric_Pad1.33x1.80mm_HandSolder
- removed C148, C169: 4n7, Capacitor_SMD:C_0603_1608Metric_Pad1.08x0.95mm_HandSolder
- removed C149, C170, C197, C199: 100p, Capacitor_SMD:C_0603_1608Metric_Pad1.08x0.95mm_HandSolder
- removed C163: 62p, Capacitor_SMD:C_0603_1608Metric_Pad1.08x0.95mm_HandSolder
- removed C75, C76: 330p, Capacitor_SMD:C_0603_1608Metric_Pad1.08x0.95mm_HandSolder
- removed D35: GREEN, ASMM-CR03-BU802:LEDM3528X210N
- removed D36, D37: 5V6, DDZ5V6ASF-7:SODFL2512X75N
- removed D38: 18V, MMSZ3V9T1G:SOD3716X135N
- removed D39: ESD122DMYR, ESD122DMYR:ESD122DMYR
- removed D40: 9V1, MMSZ3V9T1G:SOD3716X135N
- removed D41, D55: V5N3202HM3/I, V5N3202HM3-I:DFN33A_VIS
- removed D43, D44, D45, D46: RED, ASMM-CR03-BU802:LEDM3528X210N
- removed U2: ESP32-S3-WROOM-2, RF_Module:ESP32-S3-WROOM-2
- added Q1: PDTC114ET,215, PDTC114ET,215:SOT95P230X110-3N, F.Cu at (137.8, 73.7)
- added SW3: SW_MEC_5E, T6VJ11GQR:T6VJ11GQR, F.Cu at (117.5, 60.8)
- added SW4: SW_MEC_5E, T6VJ11GQR:T6VJ11GQR, F.Cu at (117.5, 70.0)
- added SW5: SW_MEC_5E, T6VJ11GQR:T6VJ11GQR, F.Cu at (117.5, 79.2)
- added U1: MAX809TEUR+T, MAX809TEUR+T:SOT95P237X112-3N, F.Cu at (120.5, 86.2)
- added U5: STM32H743VIT6, Package_QFP:LQFP-100_14x14mm_P0.5mm, F.Cu at (132.6, 85.5)
- added U6: BQ7692000PWR, Package_SO:TSSOP-20_4.4x6.5mm_P0.65mm, F.Cu at (178.1, 90.4)
- C11, C41, C64, C66, C71, C72, C73: value 10u -> 100n
- C12: value 100n -> 470n; footprint Capacitor_SMD:C_1206_3216Metric_Pad1.33x1.80mm_HandSolder -> Capacitor_SMD:C_0805_2012Metric_Pad1.18x1.45mm_HandSolder
- C16: value 220n -> 4u7; footprint Capacitor_SMD:C_0805_2012Metric_Pad1.18x1.45mm_HandSolder -> Capacitor_SMD:C_1206_3216Metric_Pad1.33x1.80mm_HandSolder
- C18: value 220n -> 100n; footprint Capacitor_SMD:C_0805_2012Metric_Pad1.18x1.45mm_HandSolder -> Capacitor_SMD:C_1206_3216Metric_Pad1.33x1.80mm_HandSolder
- C3: value 100n -> 4u7
- C33, C34: value 100n -> 220n; footprint Capacitor_SMD:C_1206_3216Metric_Pad1.33x1.80mm_HandSolder -> Capacitor_SMD:C_0805_2012Metric_Pad1.18x1.45mm_HandSolder
- C35: value 470p -> 220n; footprint Capacitor_SMD:C_0603_1608Metric_Pad1.08x0.95mm_HandSolder -> Capacitor_SMD:C_0805_2012Metric_Pad1.18x1.45mm_HandSolder
- C36: value 4n7 -> 220n; footprint Capacitor_SMD:C_0603_1608Metric_Pad1.08x0.95mm_HandSolder -> Capacitor_SMD:C_0805_2012Metric_Pad1.18x1.45mm_HandSolder
- C37, C39, C40: value 4n7 -> 100n; footprint Capacitor_SMD:C_0603_1608Metric_Pad1.08x0.95mm_HandSolder -> Capacitor_SMD:C_1206_3216Metric_Pad1.33x1.80mm_HandSolder
- C38, C48: value 1u -> 100n
- C4, C59: value 10n -> 100n
- C42: value 10u -> 470p; footprint Capacitor_SMD:C_1206_3216Metric_Pad1.33x1.80mm_HandSolder -> Capacitor_SMD:C_0603_1608Metric_Pad1.08x0.95mm_HandSolder
- C44: value 1u -> 10u
- C45: value 3n3 -> 1u; footprint Capacitor_SMD:C_0603_1608Metric_Pad1.08x0.95mm_HandSolder -> Capacitor_SMD:C_1206_3216Metric_Pad1.33x1.80mm_HandSolder
- C46: value 3n3 -> 10u; footprint Capacitor_SMD:C_0603_1608Metric_Pad1.08x0.95mm_HandSolder -> Capacitor_SMD:C_1206_3216Metric_Pad1.33x1.80mm_HandSolder
- C47: value 4u7 -> 470p; footprint Capacitor_SMD:C_1206_3216Metric_Pad1.33x1.80mm_HandSolder -> Capacitor_SMD:C_0603_1608Metric_Pad1.08x0.95mm_HandSolder
- C50: value 100n -> 4n7; footprint Capacitor_SMD:C_1206_3216Metric_Pad1.33x1.80mm_HandSolder -> Capacitor_SMD:C_0603_1608Metric_Pad1.08x0.95mm_HandSolder
- C51: value 1u -> 4n7; footprint Capacitor_SMD:C_1206_3216Metric_Pad1.33x1.80mm_HandSolder -> Capacitor_SMD:C_0603_1608Metric_Pad1.08x0.95mm_HandSolder
- C52: value 100n -> 3n3; footprint Capacitor_SMD:C_1206_3216Metric_Pad1.33x1.80mm_HandSolder -> Capacitor_SMD:C_0603_1608Metric_Pad1.08x0.95mm_HandSolder
- C54: value 10n -> 4u7
- C56, C57: value 4u7 -> 100n
- C58, C65: value 100n -> 1u
- C61: value 10n -> 1u
- C62: value 10n -> 3n3; footprint Capacitor_SMD:C_1206_3216Metric_Pad1.33x1.80mm_HandSolder -> Capacitor_SMD:C_0603_1608Metric_Pad1.08x0.95mm_HandSolder
- C63: value 10u -> 1u
- C67: value 10u -> 56u; footprint Capacitor_SMD:C_1206_3216Metric_Pad1.33x1.80mm_HandSolder -> AHA0810560M040R:CAPAE830X1100M
- C68: value 100n -> 56u; footprint Capacitor_SMD:C_1206_3216Metric_Pad1.33x1.80mm_HandSolder -> AHA0810560M040R:CAPAE830X1100M
- C69, C70: value 10u -> 220n; footprint Capacitor_SMD:C_1206_3216Metric_Pad1.33x1.80mm_HandSolder -> Capacitor_SMD:C_0805_2012Metric_Pad1.18x1.45mm_HandSolder
- C8: value 100n -> 10n
- D1: value ESD122DMYR -> 82306050029; footprint ESD122DMYR:ESD122DMYR -> 82306050029:WESURGE_0603134
- D10: value 5V6 -> RED; footprint DDZ5V6ASF-7:SODFL2512X75N -> ASMM-CR03-BU802:LEDM3528X210N
- D14, D17: value 5V6 -> PTVS14VP1UP,115; footprint DDZ5V6ASF-7:SODFL2512X75N -> PTVS14VP1UP,115:PMEG3050EP115
- D15: value 5V6 -> 1N4148W; footprint DDZ5V6ASF-7:SODFL2512X75N -> 1N4148W:SODFL3816X120N
- D16: value 5V6 -> 16V; footprint DDZ5V6ASF-7:SODFL2512X75N -> MMSZ3V9T1G:SOD3716X135N
- D18: value RED -> 1N4148W; footprint ASMM-CR03-BU802:LEDM3528X210N -> 1N4148W:SODFL3816X120N
- D19: value 1N4148W -> V5N3202HM3/I; footprint 1N4148W:SODFL3816X120N -> V5N3202HM3-I:DFN33A_VIS
- D2, D3, D4, D7: value RED -> 82306050029; footprint ASMM-CR03-BU802:LEDM3528X210N -> 82306050029:WESURGE_0603134
- D20: value 1N4148W -> 18V; footprint 1N4148W:SODFL3816X120N -> MMSZ3V9T1G:SOD3716X135N
- D21: value PTVS40VS1UTR -> 3V9; footprint PTVS40VS1UTR,115:SOD123W -> MMSZ3V9T1G:SOD3716X135N
- D23: value PTVS40VS1UTR -> RED; footprint PTVS40VS1UTR,115:SOD123W -> ASMM-CR03-BU802:LEDM3528X210N
- D24: value V5N3202HM3/I -> GREEN; footprint V5N3202HM3-I:DFN33A_VIS -> ASMM-CR03-BU802:LEDM3528X210N
- D25: value 16V -> GREEN; footprint MMSZ3V9T1G:SOD3716X135N -> ASMM-CR03-BU802:LEDM3528X210N
- D26: value 1N4148W -> GREEN; footprint 1N4148W:SODFL3816X120N -> ASMM-CR03-BU802:LEDM3528X210N
- D27: value 18V -> GREEN; footprint MMSZ3V9T1G:SOD3716X135N -> ASMM-CR03-BU802:LEDM3528X210N
- D28: value 3V9 -> GREEN; footprint MMSZ3V9T1G:SOD3716X135N -> ASMM-CR03-BU802:LEDM3528X210N
- D29: value 1N4148W -> 5V6; footprint 1N4148W:SODFL3816X120N -> DDZ5V6ASF-7:SODFL2512X75N
- D31: value GREEN -> 5V6; footprint ASMM-CR03-BU802:LEDM3528X210N -> DDZ5V6ASF-7:SODFL2512X75N
- D32: value GREEN -> 18V; footprint ASMM-CR03-BU802:LEDM3528X210N -> MMSZ3V9T1G:SOD3716X135N
- D33, D34: value GREEN -> RED
- D5: value RED -> BLUE
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Connections:
- net /C4 renamed Net-(D6-Pad2)
- net Net-(U5-LED3) renamed /Motor Control Board/MOTOR2_nFAULT
- net Net-(U5-LED4) renamed /Motor Control Board/MOTOR1_PH_IN2
- C10 pad 1: /SENSOR_P3V3 -> /P5V0
- C11 pad 1: /SENSOR_P3V3 -> /MCU/MCU_VBUS
- C16 pad 1: /BMS Protection Board/VC5 -> /MCU_P3V3
- C16 pad 2: /BMS Protection Board/VC5X -> GND
- C18 pad 1: /BMS Protection Board/VC3 -> /MCU_P3V3
- C18 pad 2: /BMS Protection Board/VC2 -> GND
- C2 pad 2: /MCU_VBUS -> /MCU/MCU_VBUS
- C3 pad 2: /MCU_VBUS -> /MCU/MCU_VBUS
- C33 pad 1: Net-(C33-Pad1) -> /BMS Protection Board/VC5
- C33 pad 2: /PACK+ -> /BMS Protection Board/VC2
- C34 pad 1: /PACK- -> /BMS Protection Board/VC2
- C34 pad 2: Net-(C33-Pad1) -> /BMS Protection Board/VC1
- C35 pad 1: /C8 -> /BMS Protection Board/VC1
- C35 pad 2: Net-(D27-A) -> /BMS Protection Board/VC0
- C36 pad 1: /BMS Protection Board/TS1 -> /BMS Protection Board/VC0
- C37 pad 1: /BMS Protection Board/TS1 -> GND
- C37 pad 2: GND -> /BMS Protection Board/SRP
- C38 pad 1: /BMS Protection Board/TS2 -> /BATT+
- C38 pad 2: /BMS Protection Board/VCX5 -> Net-(C38-Pad2)
- C39 pad 1: /BMS Protection Board/TS2 -> /BMS Protection Board/SRP
- C39 pad 2: /BMS Protection Board/VCX5 -> /BMS Protection Board/SRN
- C4 pad 1: Net-(C4-Pad1) -> GND
- C4 pad 2: GND -> /MCU/MCU_VBUS
- C40 pad 1: /BMS Protection Board/TS2 -> Net-(C38-Pad2)
- C40 pad 2: /BMS Protection Board/VCX5 -> /PACK+
- C41 pad 1: /BMS Protection Board/VCX5 -> /BMS Protection Board/SRN
- C41 pad 2: /BMS Protection Board/BAT -> GND
- C42 pad 1: GND -> /BMS Protection Board/C3
- C42 pad 2: /BMS Protection Board/VCX5 -> Net-(D20-A)
- C43 pad 2: /BMS Protection Board/REGSRC -> /BMS Protection Board/BAT
- C44 pad 2: Net-(Q21-D) -> /BMS Protection Board/BAT
- C45 pad 1: Net-(U5-VAUX) -> GND
- C45 pad 2: GND -> /BMS Protection Board/CAP1
- C46 pad 1: /BMS Protection Board/Fuel Gauge/BAT -> GND
- C46 pad 2: GND -> /BMS Protection Board/REGOUT
- C47 pad 1: /BMS Protection Board/REGOUT -> Net-(U6-ALERT)
- C48 pad 1: /BMS Protection Board/REGOUT -> /PACK-
- C48 pad 2: GND -> Net-(C48-Pad2)
- C49 pad 1: /BMS Protection Board/REGOUT -> Net-(C48-Pad2)
- C49 pad 2: GND -> /PACK+
- C5 pad 1: Net-(C4-Pad1) -> Net-(C5-Pad1)
- C50 pad 1: Net-(U5-RBI) -> Net-(U6-TS1)
- C51 pad 1: Net-(Q24-E) -> Net-(U6-TS1)
- C52 pad 1: Net-(Q24-E) -> Net-(U7-VAUX)
- C54 pad 1: Net-(U8-PACK) -> /BMS Protection Board/REGOUT
- C55 pad 1: Net-(U8-VDDCP) -> /BMS Protection Board/REGOUT
- C55 pad 2: Net-(U8-BAT) -> GND
- C56 pad 1: GND -> /BMS Protection Board/REGOUT
- C56 pad 2: /USB-C Power Delivery/VBUS -> GND
- C57 pad 1: GND -> Net-(U7-RBI)
- C57 pad 2: /USB-C Power Delivery/VBUS -> GND
- C58 pad 1: GND -> Net-(Q13-E)
- C58 pad 2: /USB-C Power Delivery/VBUS -> GND
- C59 pad 1: Net-(C59-Pad1) -> Net-(Q13-E)
- C6 pad 1: Net-(C4-Pad1) -> Net-(C5-Pad1)
- C60 pad 1: Net-(C59-Pad1) -> Net-(U8-PACK)
- C61 pad 1: Net-(C59-Pad1) -> Net-(U8-VDDCP)
- C61 pad 2: GND -> Net-(U8-BAT)
- C62 pad 1: Net-(C59-Pad1) -> /BMS Protection Board/BAT
- C63 pad 1: /LDO_3V3 -> /P5V0
- C63 pad 2: GND -> /Motor Control Board/Optical Encoder Headers/ENC_GND
- C64 pad 1: /LDO_3V3 -> /P5V0
- C64 pad 2: GND -> /Motor Control Board/Optical Encoder Headers/ENC_GND
- C65 pad 1: /LDO_3V3 -> /P5V0
- C65 pad 2: GND -> /Motor Control Board/Optical Encoder Headers/ENC_GND
- C66 pad 1: /USB-C Power Delivery/USB-C PD Controller/LDO_1V5 -> /P5V0
- C66 pad 2: GND -> /Motor Control Board/Optical Encoder Headers/ENC_GND
- C67 pad 1: /USB-C Power Delivery/USB-C PD Controller/LDO_1V5 -> /Motor Control Board/P6V0
- C68 pad 1: /USB-C Power Delivery/USB-C PD Controller/LDO_1V5 -> /Motor Control Board/P6V0
- C69 pad 1: /USB-C Power Delivery/PPHV -> /Motor Control Board/P6V0
- C7 pad 1: Net-(C4-Pad1) -> Net-(C5-Pad1)
- C70 pad 1: /USB-C Power Delivery/PPHV -> /Motor Control Board/P6V0
- C71 pad 1: /USB-C Power Delivery/PPHV -> /Motor Control Board/P6V0
- C72 pad 1: /USB-C Power Delivery/PPHV -> /Motor Control Board/P6V0
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
Commit message: now need 6V Line
Parts:
- removed the D21 at (147.0, 67.1)
- removed D31: 5V6, DDZ5V6ASF-7:SODFL2512X75N
- removed D32: 18V, MMSZ3V9T1G:SOD3716X135N
- removed D33, D34: RED, ASMM-CR03-BU802:LEDM3528X210N
- removed Q1: PDTC114ET,215, PDTC114ET,215:SOT95P230X110-3N
- removed SW3, SW4, SW5: SW_MEC_5E, T6VJ11GQR:T6VJ11GQR
- added C1: 220n, Capacitor_SMD:C_0805_2012Metric_Pad1.18x1.45mm_HandSolder, F.Cu at (291.8, 191.2)
- added C13: 100n, Capacitor_SMD:C_1206_3216Metric_Pad1.33x1.80mm_HandSolder, F.Cu at (277.4, 167.7)
- added C14: 100n, Capacitor_SMD:C_1206_3216Metric_Pad1.33x1.80mm_HandSolder, F.Cu at (277.4, 171.1)
- added C15: 10u, Capacitor_SMD:C_1206_3216Metric_Pad1.33x1.80mm_HandSolder, F.Cu at (277.4, 174.4)
- added C17: 470p, Capacitor_SMD:C_0603_1608Metric_Pad1.08x0.95mm_HandSolder, F.Cu at (282.8, 177.3)
- added C19: 10u, Capacitor_SMD:C_1206_3216Metric_Pad1.33x1.80mm_HandSolder, F.Cu at (283.5, 147.6)
- added C20: 1u, Capacitor_SMD:C_1206_3216Metric_Pad1.33x1.80mm_HandSolder, F.Cu at (283.5, 151.0)
- added C21: 10u, Capacitor_SMD:C_1206_3216Metric_Pad1.33x1.80mm_HandSolder, F.Cu at (283.5, 154.3)
- added C22: 100n, Capacitor_SMD:C_1206_3216Metric_Pad1.33x1.80mm_HandSolder, F.Cu at (283.5, 157.7)
- added C23: 470p, Capacitor_SMD:C_0603_1608Metric_Pad1.08x0.95mm_HandSolder, F.Cu at (282.8, 179.8)
- added C24: 100n, Capacitor_SMD:C_1206_3216Metric_Pad1.33x1.80mm_HandSolder, F.Cu at (283.5, 161.0)
- added C25: 100n, Capacitor_SMD:C_1206_3216Metric_Pad1.33x1.80mm_HandSolder, F.Cu at (283.5, 164.4)
- added C26: 10u, Capacitor_SMD:C_1206_3216Metric_Pad1.33x1.80mm_HandSolder, F.Cu at (283.5, 167.7)
- added C27: 4n7, Capacitor_SMD:C_0603_1608Metric_Pad1.08x0.95mm_HandSolder, F.Cu at (282.8, 182.4)
- added C28: 10u, Capacitor_SMD:C_1206_3216Metric_Pad1.33x1.80mm_HandSolder, F.Cu at (283.5, 171.1)
- added C29: 4n7, Capacitor_SMD:C_0603_1608Metric_Pad1.08x0.95mm_HandSolder, F.Cu at (282.8, 184.9)
- added C30: 10u, Capacitor_SMD:C_1206_3216Metric_Pad1.33x1.80mm_HandSolder, F.Cu at (283.5, 174.4)
- added C31: 10u, Capacitor_SMD:C_1206_3216Metric_Pad1.33x1.80mm_HandSolder, F.Cu at (289.5, 140.9)
- added C32: 10u, Capacitor_SMD:C_1206_3216Metric_Pad1.33x1.80mm_HandSolder, F.Cu at (289.5, 144.3)
- added C74: 10u, Capacitor_SMD:C_1206_3216Metric_Pad1.33x1.80mm_HandSolder, F.Cu at (277.9, 240.4)
- added C75: 1u, Capacitor_SMD:C_1206_3216Metric_Pad1.33x1.80mm_HandSolder, F.Cu at (277.9, 243.8)
- added C76: 100n, Capacitor_SMD:C_1206_3216Metric_Pad1.33x1.80mm_HandSolder, F.Cu at (277.9, 247.2)
- added C77: 33p, Capacitor_SMD:C_1206_3216Metric_Pad1.33x1.80mm_HandSolder, F.Cu at (277.9, 250.5)
- added C78: 22u, Capacitor_SMD:C_1206_3216Metric_Pad1.33x1.80mm_HandSolder, F.Cu at (283.9, 240.4)
- added C79: 22u, Capacitor_SMD:C_1206_3216Metric_Pad1.33x1.80mm_HandSolder, F.Cu at (283.9, 243.8)
- added C80: 22u, Capacitor_SMD:C_1206_3216Metric_Pad1.33x1.80mm_HandSolder, F.Cu at (283.9, 247.2)
- added C81: 22u, Capacitor_SMD:C_1206_3216Metric_Pad1.33x1.80mm_HandSolder, F.Cu at (283.9, 250.5)
- added C82: 100n, Capacitor_SMD:C_1206_3216Metric_Pad1.33x1.80mm_HandSolder, F.Cu at (289.9, 240.4)
- added C83: 100n, Capacitor_SMD:C_1206_3216Metric_Pad1.33x1.80mm_HandSolder, F.Cu at (289.9, 243.8)
- added C84: 22u, Capacitor_SMD:C_1206_3216Metric_Pad1.33x1.80mm_HandSolder, F.Cu at (289.9, 247.2)
- added C85: 22u, Capacitor_SMD:C_1206_3216Metric_Pad1.33x1.80mm_HandSolder, F.Cu at (289.9, 250.5)
- added C9: 10u, Capacitor_SMD:C_1206_3216Metric_Pad1.33x1.80mm_HandSolder, F.Cu at (277.4, 154.3)
- added D21: 9V1, MMSZ3V9T1G:SOD3716X135N, F.Cu at (277.5, 204.6)
- added D21: RED, ASMM-CR03-BU802:LEDM3528X210N, F.Cu at (302.5, 215.5)
- added IC1: TPS566238PRQFR, TPS566238PRQFR:TPS566238PRQFR, F.Cu at (287.6, 216.5)
- added L1: SDR1806-2R2ML, SDR1806-2R2ML:SDR18062R2ML, F.Cu at (285.8, 230.2)
- added L2: VLS6045EX-1R0N, VLS6045EX-1R0N:VLS6045, F.Cu at (306.9, 229.5)
- added U12: TLV75533PDBV, Package_TO_SOT_SMD:SOT-23-5, F.Cu at (282.6, 217.3)
- added U16: BQ25798RQMR, BQ25798RQMR:BQ25798RQMR, F.Cu at (287.3, 210.5)
- added U2: 1043, 1043:1043, F.Cu at (270.5, 175.4)
- added U22: 1043, 1043:1043, F.Cu at (402.5, 150.8)
- added U23: 1043, 1043:1043, F.Cu at (402.5, 174.9)
- added U24: 1043, 1043:1043, F.Cu at (402.5, 199.0)
- added U25: 1043, 1043:1043, F.Cu at (402.5, 223.1)
- added U26: 1043, 1043:1043, F.Cu at (402.5, 247.3)
- added U27: 1043, 1043:1043, F.Cu at (402.5, 271.4)
- added U28: TPS566238PRQFR, TPS566238PRQFR:TPS566238PRQFR, F.Cu at (295.7, 241.2)
- added U3: 1043, 1043:1043, F.Cu at (270.5, 199.5)
- added U4: 1043, 1043:1043, F.Cu at (270.5, 223.6)
- added U8: BQ7692000PWR, Package_SO:TSSOP-20_4.4x6.5mm_P0.65mm, F.Cu at (279.2, 210.8)
- C10, C39: value 100n -> 10u
- C12: value 470n -> 100n; footprint Capacitor_SMD:C_0805_2012Metric_Pad1.18x1.45mm_HandSolder -> Capacitor_SMD:C_1206_3216Metric_Pad1.33x1.80mm_HandSolder
- C16: value 4u7 -> 10u
- C18: value 100n -> 1u
- C2, C3: value 4u7 -> 220n; footprint Capacitor_SMD:C_1206_3216Metric_Pad1.33x1.80mm_HandSolder -> Capacitor_SMD:C_0805_2012Metric_Pad1.18x1.45mm_HandSolder
- C33: value 220n -> 100n; footprint Capacitor_SMD:C_0805_2012Metric_Pad1.18x1.45mm_HandSolder -> Capacitor_SMD:C_1206_3216Metric_Pad1.33x1.80mm_HandSolder
- C34, C35: value 220n -> 330p; footprint Capacitor_SMD:C_0805_2012Metric_Pad1.18x1.45mm_HandSolder -> Capacitor_SMD:C_0603_1608Metric_Pad1.08x0.95mm_HandSolder
- C36: value 220n -> 3n3; footprint Capacitor_SMD:C_0805_2012Metric_Pad1.18x1.45mm_HandSolder -> Capacitor_SMD:C_0603_1608Metric_Pad1.08x0.95mm_HandSolder
- C38, C48, C49: value 100n -> 10n
- C4: value 100n -> 220n; footprint Capacitor_SMD:C_1206_3216Metric_Pad1.33x1.80mm_HandSolder -> Capacitor_SMD:C_0805_2012Metric_Pad1.18x1.45mm_HandSolder
- C40: value 100n -> 3n3; footprint Capacitor_SMD:C_1206_3216Metric_Pad1.33x1.80mm_HandSolder -> Capacitor_SMD:C_0603_1608Metric_Pad1.08x0.95mm_HandSolder
- C42: value 470p -> 10u; footprint Capacitor_SMD:C_0603_1608Metric_Pad1.08x0.95mm_HandSolder -> Capacitor_SMD:C_1206_3216Metric_Pad1.33x1.80mm_HandSolder
- C43: value 1u -> 10u
- C44: value 10u -> 100n
- C46: value 10u -> 1u
- C47: value 470p -> 10n; footprint Capacitor_SMD:C_0603_1608Metric_Pad1.08x0.95mm_HandSolder -> Capacitor_SMD:C_1206_3216Metric_Pad1.33x1.80mm_HandSolder
- C5, C60, C7, C8: value 10n -> 100n
- C50, C51: value 4n7 -> 10n; footprint Capacitor_SMD:C_0603_1608Metric_Pad1.08x0.95mm_HandSolder -> Capacitor_SMD:C_1206_3216Metric_Pad1.33x1.80mm_HandSolder
- C52: value 3n3 -> 1u; footprint Capacitor_SMD:C_0603_1608Metric_Pad1.08x0.95mm_HandSolder -> Capacitor_SMD:C_1206_3216Metric_Pad1.33x1.80mm_HandSolder
- C53: value 10n -> 4u7
- C54: value 4u7 -> 1u
- C55, C58: value 1u -> 100n
- C56, C57: value 100n -> 4u7
- C6: value 10n -> 1u
- C62: value 3n3 -> 100n; footprint Capacitor_SMD:C_0603_1608Metric_Pad1.08x0.95mm_HandSolder -> Capacitor_SMD:C_1206_3216Metric_Pad1.33x1.80mm_HandSolder
- D1, D2, D3: value 82306050029 -> RED; footprint 82306050029:WESURGE_0603134 -> ASMM-CR03-BU802:LEDM3528X210N
- D10: value RED -> PTVS14VP1UP,115; footprint ASMM-CR03-BU802:LEDM3528X210N -> PTVS14VP1UP,115:PMEG3050EP115
- D11: value 5V6 -> 1N4148W; footprint DDZ5V6ASF-7:SODFL2512X75N -> 1N4148W:SODFL3816X120N
- D12: value 5V6 -> V5N3202HM3/I; footprint DDZ5V6ASF-7:SODFL2512X75N -> V5N3202HM3-I:DFN33A_VIS
- D13: value 5V6 -> 18V; footprint DDZ5V6ASF-7:SODFL2512X75N -> MMSZ3V9T1G:SOD3716X135N
- D14: value PTVS14VP1UP,115 -> 3V9; footprint PTVS14VP1UP,115:PMEG3050EP115 -> MMSZ3V9T1G:SOD3716X135N
- D15: value 1N4148W -> 16V; footprint 1N4148W:SODFL3816X120N -> MMSZ3V9T1G:SOD3716X135N
- D16: value 16V -> RED; footprint MMSZ3V9T1G:SOD3716X135N -> ASMM-CR03-BU802:LEDM3528X210N
- D17: value PTVS14VP1UP,115 -> 18V; footprint PTVS14VP1UP,115:PMEG3050EP115 -> MMSZ3V9T1G:SOD3716X135N
- D18: value 1N4148W -> 82306050029; footprint 1N4148W:SODFL3816X120N -> 82306050029:WESURGE_0603134
- D19: value V5N3202HM3/I -> 82306050029; footprint V5N3202HM3-I:DFN33A_VIS -> 82306050029:WESURGE_0603134
- D22: value 16V -> GREEN; footprint MMSZ3V9T1G:SOD3716X135N -> ASMM-CR03-BU802:LEDM3528X210N
- D23: value RED -> GREEN
- D27, D28: value GREEN -> 5V6; footprint ASMM-CR03-BU802:LEDM3528X210N -> DDZ5V6ASF-7:SODFL2512X75N
- D29: value 5V6 -> RED; footprint DDZ5V6ASF-7:SODFL2512X75N -> ASMM-CR03-BU802:LEDM3528X210N
- D30: value 18V -> RED; footprint MMSZ3V9T1G:SOD3716X135N -> ASMM-CR03-BU802:LEDM3528X210N
- D4: value 82306050029 -> 5V6; footprint 82306050029:WESURGE_0603134 -> DDZ5V6ASF-7:SODFL2512X75N
- D5: value BLUE -> 5V6; footprint ASMM-CR03-BU802:LEDM3528X210N -> DDZ5V6ASF-7:SODFL2512X75N
- D6: value RED -> 5V6; footprint ASMM-CR03-BU802:LEDM3528X210N -> DDZ5V6ASF-7:SODFL2512X75N
- D7: value 82306050029 -> PTVS14VP1UP,115; footprint 82306050029:WESURGE_0603134 -> PTVS14VP1UP,115:PMEG3050EP115
- D8: value RED -> 1N4148W; footprint ASMM-CR03-BU802:LEDM3528X210N -> 1N4148W:SODFL3816X120N
- D9: value RED -> 16V; footprint ASMM-CR03-BU802:LEDM3528X210N -> MMSZ3V9T1G:SOD3716X135N
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Connections:
- net /MCU/USB_C_N renamed Net-(D2-Pad1)
- net /MCU/USB_C_P renamed Net-(D3-Pad1)
- C10 pad 1: /P5V0 -> /BMS Protection Board/LDO_3V3
- C11 pad 1: /MCU/MCU_VBUS -> /BMS Protection Board/SRP
- C11 pad 2: GND -> /BMS Protection Board/SRN
- C12 pad 1: Net-(U3-OUT) -> /BMS Protection Board/LDO_3V3
- C16 pad 1: /MCU_P3V3 -> /BMS Protection Board/LDO_1V5
- C18 pad 1: /MCU_P3V3 -> GND
- C18 pad 2: GND -> /BMS Protection Board/BAT
- C2 pad 1: GND -> /BMS Protection Board/VC2
- C2 pad 2: /MCU/MCU_VBUS -> /BMS Protection Board/VC1
- C3 pad 1: GND -> /BMS Protection Board/VC1
- C3 pad 2: /MCU/MCU_VBUS -> /BMS Protection Board/VC0
- C33 pad 1: /BMS Protection Board/VC5 -> /BMS Protection Board/PD_VAC
- C33 pad 2: /BMS Protection Board/VC2 -> GND
- C34 pad 1: /BMS Protection Board/VC2 -> /BMS Protection Board/C_CC1
- C34 pad 2: /BMS Protection Board/VC1 -> GND
- C35 pad 1: /BMS Protection Board/VC1 -> /BMS Protection Board/C_CC2
- C35 pad 2: /BMS Protection Board/VC0 -> GND
- C36 pad 1: /BMS Protection Board/VC0 -> /BMS Protection Board/BAT
- C37 pad 1: GND -> /BMS Protection Board/P5V0
- C37 pad 2: /BMS Protection Board/SRP -> GND
- C38 pad 1: /BATT+ -> Net-(U11-BAT)
- C38 pad 2: Net-(C38-Pad2) -> GND
- C39 pad 1: /BMS Protection Board/SRP -> /BMS Protection Board/P5V0
- C39 pad 2: /BMS Protection Board/SRN -> GND
- C4 pad 1: GND -> /BMS Protection Board/VC0
- C4 pad 2: /MCU/MCU_VBUS -> GND
- C40 pad 1: Net-(C38-Pad2) -> Net-(U13-VAUX)
- C40 pad 2: /PACK+ -> GND
- C41 pad 1: /BMS Protection Board/SRN -> /BMS Protection Board/P3V3
- C42 pad 1: /BMS Protection Board/C3 -> /BMS Protection Board/P3V3
- C42 pad 2: Net-(D20-A) -> GND
- C43 pad 1: GND -> /BMS Protection Board/P3V3
- C43 pad 2: /BMS Protection Board/BAT -> GND
- C44 pad 1: GND -> /BMS Protection Board/P3V3
- C44 pad 2: /BMS Protection Board/BAT -> GND
- C45 pad 1: GND -> /BMS Protection Board/P3V3
- C45 pad 2: /BMS Protection Board/CAP1 -> GND
- C46 pad 1: GND -> /BMS Protection Board/P3V3
- C46 pad 2: /BMS Protection Board/REGOUT -> GND
- C47 pad 1: Net-(U6-ALERT) -> GND
- C47 pad 2: GND -> Net-(C47-Pad2)
- C48 pad 1: /PACK- -> GND
- C48 pad 2: Net-(C48-Pad2) -> Net-(C47-Pad2)
- C49 pad 1: Net-(C48-Pad2) -> GND
- C49 pad 2: /PACK+ -> Net-(C47-Pad2)
- C5 pad 1: Net-(C5-Pad1) -> /BMS Protection Board/LDO_3V3
- C50 pad 1: Net-(U6-TS1) -> GND
- C50 pad 2: GND -> Net-(C47-Pad2)
- C51 pad 1: Net-(U6-TS1) -> Net-(U11-PACK)
- C52 pad 2: GND -> Net-(U11-BAT)
- C53 pad 1: Net-(U8-BAT) -> /BMS Protection Board/REGOUT
- C56 pad 1: /BMS Protection Board/REGOUT -> /BMS Protection Board/VBUS
- C57 pad 1: Net-(U7-RBI) -> /BMS Protection Board/VBUS
- C58 pad 1: Net-(Q13-E) -> /BMS Protection Board/VBUS
- C59 pad 1: Net-(Q13-E) -> Net-(U13-RBI)
- C6 pad 1: Net-(C5-Pad1) -> /BMS Protection Board/LDO_3V3
- C60 pad 1: Net-(U8-PACK) -> /BMS Protection Board/P5V0
- C61 pad 1: Net-(U8-VDDCP) -> Net-(Q14-E)
- C61 pad 2: Net-(U8-BAT) -> GND
- C62 pad 1: /BMS Protection Board/BAT -> Net-(Q14-E)
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
Commit message: Added 6V Line
Parts:
- removed C1, C2, C3, C4, C69, C70: 220n, Capacitor_SMD:C_0805_2012Metric_Pad1.18x1.45mm_HandSolder
- removed C10, C15, C16, C19, C21, C26, C28, C30, C31, C32, C39, C42, C43, C74, C9: 10u, Capacitor_SMD:C_1206_3216Metric_Pad1.33x1.80mm_HandSolder
- removed C11, C12, C13, C14, C22, C24, C25, C33, C37, C41, C44, C5, C55, C58, C59, C60, C62, C64, C66, C7, C71, C72, C73, C76, C8, C82, C83: 100n, Capacitor_SMD:C_1206_3216Metric_Pad1.33x1.80mm_HandSolder
- removed C17, C23: 470p, Capacitor_SMD:C_0603_1608Metric_Pad1.08x0.95mm_HandSolder
- removed C18, C20, C45, C46, C52, C54, C6, C61, C63, C65, C75: 1u, Capacitor_SMD:C_1206_3216Metric_Pad1.33x1.80mm_HandSolder
- removed C27, C29: 4n7, Capacitor_SMD:C_0603_1608Metric_Pad1.08x0.95mm_HandSolder
- removed C34, C35: 330p, Capacitor_SMD:C_0603_1608Metric_Pad1.08x0.95mm_HandSolder
- removed C36, C40: 3n3, Capacitor_SMD:C_0603_1608Metric_Pad1.08x0.95mm_HandSolder
- removed C38, C47, C48, C49, C50, C51: 10n, Capacitor_SMD:C_1206_3216Metric_Pad1.33x1.80mm_HandSolder
- removed C53, C56, C57: 4u7, Capacitor_SMD:C_1206_3216Metric_Pad1.33x1.80mm_HandSolder
- removed C67, C68: 56u, AHA0810560M040R:CAPAE830X1100M
- removed C77: 33p, Capacitor_SMD:C_1206_3216Metric_Pad1.33x1.80mm_HandSolder
- removed C78, C79, C80, C81, C84, C85: 22u, Capacitor_SMD:C_1206_3216Metric_Pad1.33x1.80mm_HandSolder
- removed the D21 at (277.5, 204.6)
- removed the D21 at (302.5, 215.5)
- removed IC1: TPS566238PRQFR, TPS566238PRQFR:TPS566238PRQFR
- added D21: RED, ASMM-CR03-BU802:LEDM3528X210N, F.Cu at (298.8, 67.5)
- added L3: SLC1480-441MLD, SLC1480-441MLD:SLC1480441MLD, F.Cu at (321.5, 81.9)
- added U29: TPS40305DRCT, TPS40305DRCT:TPS40305DRCT, F.Cu at (335.9, 61.4)
- L1: value SDR1806-2R2ML -> PA4343.222NLT; footprint SDR1806-2R2ML:SDR18062R2ML -> PA4343.222NLT:INDPM135125X650N
- moved U28 206.1 mm to (216.5, 51.0)
- moved U25 190.9 mm to (499.1, 58.5)
- moved U27 190.9 mm to (499.1, 106.7)
- moved U26 190.9 mm to (499.1, 82.6)
- moved D12 179.1 mm to (211.3, 51.0)
- moved U4 177.4 mm to (204.2, 59.1)
- moved U6 177.4 mm to (204.2, 107.4)
- moved U5 177.4 mm to (204.2, 83.2)
- moved L1 149.6 mm to (301.8, 81.5)
- moved D22 134.0 mm to (305.1, 49.3)
- moved D23 134.0 mm to (305.1, 53.9)
- moved D13 129.9 mm to (292.5, 53.6)
- moved D15 129.9 mm to (292.5, 62.4)
- moved D20 129.9 mm to (292.5, 71.2)
- moved D14 129.9 mm to (292.5, 58.0)
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Connections:
- net /BMS Protection Board/PACK+ renamed /PACK+
- net /Motor Control Board/MOTOR1_PH_IN2 renamed /MOTOR1_nFAULT
- net /Motor Control Board/MOTOR2_nFAULT renamed /MOTOR2_nFAULT
- L1 pad 1: /BMS Protection Board/P5V0 -> /P5V0
- U12 pad 1: /BMS Protection Board/P5V0 -> /P5V0
- U12 pad 3: /BMS Protection Board/P5V0 -> /P5V0

Commit message: bom progress
Parts:
- removed U22, U23, U24, U25, U26, U27: 1043, 1043:1043
- added J1: 796739-2, 796739-2:7967392, F.Cu at (283.5, 147.4)
- added J14: Conn_02x20_Odd_Even, 7-534206-0:SHDR40W69P254_2X20_5080X503X813P, F.Cu at (279.2, 84.4)
- added J15: Conn_02x20_Odd_Even, Connector_PinHeader_2.54mm:PinHeader_2x20_P2.54mm_Vertical, F.Cu at (279.5, 88.7)
- added J3: Conn_01x04, Connector_PinHeader_2.54mm:PinHeader_1x04_P2.54mm_Vertical, F.Cu at (279.5, 159.1)
- added J4: SMB, Connector_PinHeader_2.54mm:PinHeader_1x04_P2.54mm_Vertical, F.Cu at (284.1, 159.1)
- added U18: DRV8243SQDGQRQ1 (S-Variant), DRV8243SQDGQRQ1:SOP50P490X110-29N, F.Cu at (264.4, 193.8)
- added U19: DRV8243SQDGQRQ1 (S-Variant), DRV8243SQDGQRQ1:SOP50P490X110-29N, F.Cu at (271.8, 193.8)
- added U20: LS7366R-S, LS7366R_S:SOIC127P600X175-14N, F.Cu at (281.8, 176.1)
- added U21: LS7366R-S, LS7366R_S:SOIC127P600X175-14N, F.Cu at (290.6, 176.1)
- added Y1: ASV-30.000MHZ-E-T, ASV-30.000MHZ-E-T:ASV25000MHZEJT, F.Cu at (282.2, 185.9)
- moved D29 155.7 mm to (280.3, 194.8)
- moved D30 155.7 mm to (280.3, 199.3)
- moved D12 141.2 mm to (261.7, 182.9)
- moved U28 141.2 mm to (266.9, 182.8)
- moved U4 116.6 mm to (254.7, 164.2)
- moved U6 116.6 mm to (254.7, 212.5)
- moved U5 116.6 mm to (254.7, 188.4)
- moved U29 84.6 mm to (320.5, 144.5)
- moved U8 74.7 mm to (263.3, 170.2)
- moved D8 71.9 mm to (267.0, 175.8)
- moved D11 71.9 mm to (267.0, 178.8)
- moved D18 71.9 mm to (261.4, 175.8)
- moved D19 71.9 mm to (261.4, 178.8)
- moved D1 69.8 mm to (261.7, 108.5)
- moved D2 69.8 mm to (261.7, 113.0)
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Connections:
- D1 pad 2: /BATT+ -> /C3
- D17 pad 1: /BATT+ -> /C3
- D6 pad 2: /BATT- -> /C0
- D8 pad 2: /BATT+ -> /C3
- U1 pad 1: /BATT+ -> /C3
- U3 pad 2: /BATT- -> /C0
- U4 pad 1: /BATT+ -> /C3
- U6 pad 2: /BATT- -> /C0
