File: Schematic/STAR_BUCK_BOOST_CHARGER.kicad_pcb (KiCad board)
At the start: 2 copper layers, 40 parts, among them J1 Conn_01x02, J2 1017491, J3 1017491, J4 1017491, U1 BQ25798RQMR

Commit message: started to work on the high side gate driver PCB
Parts:
- added C24: 22u, T527T226M025ATE100:CAPPM3528X120N, F.Cu at (94.6, 79.3)
- added C25: 22u, T527T226M025ATE100:CAPPM3528X120N, F.Cu at (94.6, 83.9)
- added C26: 22u, T527T226M025ATE100:CAPPM3528X120N, F.Cu at (94.6, 88.4)
- moved J3 78.1 mm to (89.1, 22.9)
- moved J2 78.1 mm to (74.3, 22.9)
- moved J4 78.1 mm to (104.0, 22.9)
- moved TH1 60.5 mm to (104.3, 93.8)
- moved NT1 60.5 mm to (103.6, 95.8)
- moved C1 48.5 mm to (79.4, 78.5)
- moved C18 48.5 mm to (89.0, 78.5)
- moved C21 48.5 mm to (89.0, 84.6)
- moved C22 48.5 mm to (89.0, 87.6)
- moved C9 48.5 mm to (79.4, 93.6)
- moved C20 48.5 mm to (89.0, 81.6)
- moved C10 48.5 mm to (84.2, 78.5)
- moved C11 48.5 mm to (84.2, 81.6)
- moved C12 48.5 mm to (84.2, 84.6)
- moved C13 48.5 mm to (84.2, 87.6)
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Connections:
- net /5V_BUCK_SYS renamed /P5V0_BUCK_SYS
- net /BUCK_BOOST_PACK+ renamed /AFE_PACK+
- R5 pad 2: /LDO_3V3 -> /USB_C_LDO_3V3
- R6 pad 1: /LDO_3V3 -> /USB_C_LDO_3V3
