File: Schematic/STAR_FUEL_GUAGE.kicad_sch (KiCad schematic)
At the start: 50 parts, among them J1 6120XX21621_61200821621, J2 BMS_I2C, J3 Conn_01x02, J4 Conn_01x02, J5 6120XX21621_61200621621, J6 6120XX21621_61200621621, J7 SMB, Q1 ZXMP10A13FTA, Q2 BSS123, Q3 MMBT3904, U1 BQ78350DBT-R1A, U2 PCA9306D,118

Commit message: Fuel Gauge Version 1.0.0
Other:
- note added: "AFE"
- note added: "Gate Driver"
- note added: "MCU"
- moved on the sheet: J6
