File: Schematic/STAR_MCU.kicad_sch (KiCad schematic)
At the start: 34 parts, among them J11 HC-SR04, J12 HC-SR04, J13 HC-SR04, J14 HC-SR04, J15 HC-SR04, J16 HC-SR04, J17 HC-SR04, J18 Conn_02x20_Odd_Even, J19 USB4216-03-A, U11 BMI323, U12 ESP32-S3-WROOM-1-N16, U13 74HC139D,653

Commit message: splitting this up into smaller pcbs
Parts:
- renumbered C111 to C100, C112 to C101, C113 to C102, C114 to C103, C115 to C104, C116 to C105, C106 to C95, C107 to C96, C108 to C97, C109 to C98, C110 to C99
Other:
- note added: "NEED TO ADD HEADERS FOR POWER AND TO THE OTHER BOARDS"
- moved on the sheet: C100, C101, C102, C103, C104, C105, C95, C96, C97, C98, C99, D25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

Commit message: updated schematic
Parts:
- added J10, J3, J6: 6120XX21621_61200621621, 61200621621:61200621621, symbol 61200621621:6120XX21621_61200621621
- added J4, J7, J8: 6120XX21621_61200821621, 61200821621:61200821621, symbol 61200821621:6120XX21621_61200821621
Connections:
- net ENCODER1_OUTPUT1: now also J7.2
- net ENCODER1_OUTPUT2: now also J7.4
- net ENCODER2_OUTPUT1: now also J7.6
- net ENCODER2_OUTPUT2: now also J7.8
- net GND: now also J10.5, J10.6, J3.5, J3.6, J6.1, J6.6
- net MOTOR1_EN_IN1: now also J8.1
- net MOTOR1_IPROPI: now also J4.2
- net MOTOR1_PH_IN2: now also J8.2
- net MOTOR1_nCS: now also J3.1; no longer U13.4 (1~{Y0})
- net MOTOR1_nFAULT: now also J4.1
- net MOTOR2_EN_IN1: now also J8.3
- net MOTOR2_IPROPI: now also J4.4
- net MOTOR2_PH_IN2: now also J8.4
- net MOTOR2_nCS: now also J3.2; no longer U13.5 (1~{Y1})
- net MOTOR2_nFAULT: now also J4.3
- net MOTOR3_EN_IN1: now also J8.5
- net MOTOR3_IPROPI: now also J4.6
- net MOTOR3_PH_IN2: now also J8.6
- net MOTOR3_nCS: now also J3.4; no longer U13.6 (1~{Y2})
- net MOTOR3_nFAULT: now also J4.5
- net MOTOR4_EN_IN1: now also J8.7
- net MOTOR4_IPROPI: now also J4.8
- net MOTOR4_PH_IN2: now also J8.8
- net MOTOR4_nCS: now also J3.3; no longer U13.7 (1~{Y3})
- net MOTOR4_nFAULT: now also J4.7
- net SPI_SCLK: now also J10.2; no longer U12.29 (IO36)
- net P3V3 renamed MCU_P3V3
- net MCU_P3V3: now also J10.1, J6.3, J6.5
- net SMBC renamed MCU_SMBC
- net MCU_SMBC: now also J6.2
- net SMBD renamed MCU_SMBD
- net MCU_SMBD: now also J6.4
- net SPI3_SM_CS renamed SPI3_PM_CS
- net SPI3_SM_MISO renamed SPI3_PM_CIPO
- net SPI3_SM_MOSI renamed SPI3_PM_COPI
- net SPI3_SM_SCLK renamed SPI3_PM_SCLK
- net SPI_SDI renamed SPI_CIPO
- net SPI_CIPO: now also J10.4
- net SPI_SDO renamed SPI_COPI
- net SPI_COPI: now also J10.3
- new net MOTOR1_TERMINAL1: J7.1
- new net MOTOR1_TERMINAL2: J7.3
- new net MOTOR2_TERMINAL1: J7.5
- new net MOTOR2_TERMINAL2: J7.7
- new net SPI2_CM_SCLK: U12.29 (IO36)
- new net SPI2_MOTOR1_nCS: U13.4 (1~{Y0})
- new net SPI2_MOTOR2_nCS: U13.5 (1~{Y1})
- new net SPI2_MOTOR3_nCS: U13.6 (1~{Y2})
- new net SPI2_MOTOR4_nCS: U13.7 (1~{Y3})
Other:
- note added: "3,sda 5,scl 8,txd 10,rxd 19,copi 21,cipo 23,sclk 24,ce0 26,ce1"
- note added: "SPI2 will act as a "controller""
- note added: "SPI3 will act as a "peripheral""
- note removed: "3,sda 5,scl 8,txd 10,rxd 19,mosi 21,miso 23,sclk 24,ce0 26,ce1"
- note removed: "NEED TO ADD HEADERS FOR POWER AND TO THE OTHER BOARDS"
- note removed: "SPI2 will act as a "master""
- note removed: "SPI3 will act as a "slave""

Commit message: cookin
Parts:
- removed C100, C97: 1u, Capacitor_SMD:C_0603_1608Metric_Pad1.08x0.95mm_HandSolder, symbol Device:C
- removed C95, C96, C98, C99: 100n, Capacitor_SMD:C_0603_1608Metric_Pad1.08x0.95mm_HandSolder, symbol Device:C
- removed J10, J3: 6120XX21621_61200621621, 61200621621:61200621621, symbol 61200621621:6120XX21621_61200621621
- removed U11: BMI323, BMI323:BMI323, symbol BMI323:BMI323
- added J1, J5: 6120XX21621_61200821621, 61200821621:61200821621, symbol 61200821621:6120XX21621_61200821621
- added J2: 6120XX21621_61200621621, 61200621621:61200621621, symbol 61200621621:6120XX21621_61200621621
- added J3: Conn_01x09, 4ms_Connector:Pins_1x09_2.54mm_TH, symbol PCM_4ms_Connector:Conn_01x09
- added J9: Conn_01x04, 4ms_Connector:Pins_1x04_2.54mm_TH_SWD, symbol PCM_4ms_Connector:Conn_01x04
- added U1: SN74HC153DR, SOIC127P600X175-16N, symbol SN74HC153DR:SN74HC153DR
Connections:
- net GND: now also J1.2, J1.4, J1.6, J1.8, J2.2, J2.4, J2.6, J3.2 (Pin_2), J5.8, J9.2 (Pin_2), U1.1 (1~{G}), U1.15 (2~{G}), U1.8 (GND)
- net PI_SCL: now also J9.3 (Pin_3)
- net PI_SDA: now also J9.4 (Pin_4)
- net ENCODER1_OUTPUT1 renamed MOTOR_DRIVER_ENCODER1_OUTPUT_B
- net MOTOR_DRIVER_ENCODER1_OUTPUT_B: now also U1.10 (2C0); no longer U12.33 (IO40)
- net ENCODER1_OUTPUT2 renamed MOTOR_DRIVER_ENCODER2_OUTPUT_B
- net MOTOR_DRIVER_ENCODER2_OUTPUT_B: now also U1.11 (2C1); no longer U12.34 (IO41)
- net ENCODER2_OUTPUT1 renamed MOTOR_DRIVER_ENCODER3_OUTPUT_B
- net MOTOR_DRIVER_ENCODER3_OUTPUT_B: now also U1.12 (2C2); no longer U12.35 (IO42)
- net ENCODER2_OUTPUT2 renamed MOTOR_DRIVER_ENCODER4_OUTPUT_B
- net MOTOR_DRIVER_ENCODER4_OUTPUT_B: now also U1.13 (2C3); no longer U12.24 (IO47)
- net IMU_INT1 renamed IMU_RST
- net IMU_RST: now also J3.4 (Pin_4)
- net IMU_INT2 renamed IMU_INT
- net IMU_INT: now also J3.5 (Pin_5)
- net MCU_P3V3 renamed FUEL_GUAGE_P3V3
- net FUEL_GUAGE_P3V3: now also J1.1, J1.3, J1.5, J1.7, J2.1, J2.3, J2.5, J3.1 (Pin_1), J9.1 (Pin_1), U1.16 (VCC)
- net MOTOR1_EN_IN1 renamed MOTOR_DRIVER_MOTOR1_EN_IN1
- net MOTOR1_IPROPI renamed MOTOR_DRIVER_MOTOR1_IPROPI
- net MOTOR1_PH_IN2 renamed MOTOR_DRIVER_MOTOR1_PH_IN2
- net MOTOR1_TERMINAL1 renamed MOTOR_DRIVER_ENCODER1_OUTPUT_A
- net MOTOR_DRIVER_ENCODER1_OUTPUT_A: now also U1.6 (1C0)
- net MOTOR1_TERMINAL2 renamed MOTOR_DRIVER_ENCODER2_OUTPUT_A
- net MOTOR_DRIVER_ENCODER2_OUTPUT_A: now also U1.5 (1C1)
- net MOTOR1_nFAULT renamed MOTOR_DRIVER_MOTOR1_nFAULT
- net MOTOR2_EN_IN1 renamed MOTOR_DRIVER_MOTOR2_EN_IN1
- net MOTOR2_IPROPI renamed MOTOR_DRIVER_MOTOR2_IPROPI
- net MOTOR2_PH_IN2 renamed MOTOR_DRIVER_MOTOR2_PH_IN2
- net MOTOR2_TERMINAL1 renamed MOTOR_DRIVER_ENCODER3_OUTPUT_A
- net MOTOR_DRIVER_ENCODER3_OUTPUT_A: now also U1.4 (1C2)
- net MOTOR2_TERMINAL2 renamed MOTOR_DRIVER_ENCODER4_OUTPUT_A
- net MOTOR_DRIVER_ENCODER4_OUTPUT_A: now also U1.3 (1C3)
- net MOTOR2_nFAULT renamed MOTOR_DRIVER_MOTOR2_nFAULT
- net MOTOR3_EN_IN1 renamed MOTOR_DRIVER_MOTOR3_EN_IN1
- net MOTOR3_IPROPI renamed MOTOR_DRIVER_MOTOR3_IPROPI
- net MOTOR3_PH_IN2 renamed MOTOR_DRIVER_MOTOR3_PH_IN2
- net MOTOR3_nFAULT renamed MOTOR_DRIVER_MOTOR3_nFAULT
- net MOTOR4_EN_IN1 renamed MOTOR_DRIVER_MOTOR4_EN_IN1
- net MOTOR4_IPROPI renamed MOTOR_DRIVER_MOTOR4_IPROPI
- net MOTOR4_PH_IN2 renamed MOTOR_DRIVER_MOTOR4_PH_IN2
- net MOTOR4_nFAULT renamed MOTOR_DRIVER_MOTOR4_nFAULT
- net SPI2_CM_SCLK renamed MOTOR_DRIVER_SPI2_CM_SCLK
- net MOTOR_DRIVER_SPI2_CM_SCLK: now also J5.4
- net SPI2_MOTOR1_nCS renamed MOTOR_DRIVER_SPI2_MOTOR1_nCS
- net MOTOR_DRIVER_SPI2_MOTOR1_nCS: now also J5.1
- net SPI2_MOTOR2_nCS renamed MOTOR_DRIVER_SPI2_MOTOR2_nCS
- net MOTOR_DRIVER_SPI2_MOTOR2_nCS: now also J5.3
- net SPI2_MOTOR3_nCS renamed MOTOR_DRIVER_SPI2_MOTOR3_nCS
- net MOTOR_DRIVER_SPI2_MOTOR3_nCS: now also J5.5
- net SPI2_MOTOR4_nCS renamed MOTOR_DRIVER_SPI2_MOTOR4_nCS
- net MOTOR_DRIVER_SPI2_MOTOR4_nCS: now also J5.7
- net SPI3_PM_CIPO renamed ESP_PI_SPI3_PM_CIPO
- net SPI3_PM_COPI renamed ESP_PI_SPI3_PM_COPI
- net SPI3_PM_CS renamed ESP_PI_SPI3_PM_CS
- net SPI3_PM_SCLK renamed ESP_PI_SPI3_PM_SCLK
- net SPI_CIPO renamed MOTOR_DRIVER_SPI2_CM_COPI
- net MOTOR_DRIVER_SPI2_CM_COPI: now also J5.2
- net SPI_COPI renamed MOTOR_DRIVER_SPI2_CM_CIPO
- net MOTOR_DRIVER_SPI2_CM_CIPO: now also J5.6
- new net MOTOR_ENCODER_OUT0: U1.9 (2Y), U12.35 (IO42)
- new net MOTOR_ENCODER_OUT1: U1.7 (1Y), U12.24 (IO47)
- new net MOTOR_ENCODER_SEL0: U1.14 (A), U12.33 (IO40)
- new net MOTOR_ENCODER_SEL1: U1.2 (B), U12.34 (IO41)
- no-connect marks 22 -> 23
Other:
- note added: "By default pins are high, when selected they go low"
- note added: "IMU"
- note added: "Motor Driver"
- note added: "TODO: ADD LIDAR HEADER"
- note added: "i2c_addr ps2 ps1 bl_ind"
- note added: "io48 is unused, we can use if we need"
- note added: "nboot"
- note removed: "addr: 0x68"
- note removed: "pin is just unused, could use if we want (IO48)"
- moved on the sheet: C101, C102, C103, C104, C105, D25, D26, J11, J12, J13, J14, J15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

Commit message: mcu
Parts:
- added J10: S5B-XH-A, S5B-XH-A:JST_S5B-XH-A, symbol S5B-XH-A:S5B-XH-A
- added J20: 6120XX21621_61200621621, 61200621621:61200621621, symbol 61200621621:6120XX21621_61200621621
Connections:
- net GND: now also J10.2, J20.2, J20.4, J20.6
- net ESP_RXD_PI_TXD: no longer names the net of U12.36 (RXD0)
- net ESP_RXD_PI_TXD: no longer J18.8 (Pin_8)
- net ESP_TXD_PI_RXD: no longer names the net of U12.37 (TXD0)
- net ESP_TXD_PI_RXD: no longer J18.10 (Pin_10)
- net FUEL_GUAGE_P3V3 renamed MOTOR_DRIVER_P3V3
- net MCU_SMBC renamed FUEL_GUAGE_SMBC_SCL
- net MCU_SMBD renamed FUEL_GUAGE_SMBD_SDA
- new net LiDAR_RX_PI5_TX: J10.3, J18.8 (Pin_8)
- new net LiDAR_TX_PI5_RX: J10.4, J18.10 (Pin_10)
- new net P5V0_BUCK: J10.5, J20.1, J20.3, J20.5
- no-connect marks 23 -> 26
Other:
- note added: "3V3 Buck"
- note added: "5V0 Buck"
- note added: "Fuel Guage"
- note added: "LiDAR"
- note added: "SONAR"
- note added: "these are unused, we can use if we need"
- note removed: "TODO: ADD LIDAR HEADER"

Commit message: Fixed ur shit
Other:
- note added: "Fuel Gauge"
- note removed: "Fuel Guage"
Changed lines of the file:
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@@
 		)
 	)
-	(text "Fuel Guage"
+	(text "Fuel Gauge"
 		(exclude_from_sim no)
 		(at 310.134 242.062 0)

Commit message: fixed muc
Parts:
- added J12: Conn_01x04, 4ms_Connector:Pins_1x04_2.54mm_TH_SWD, symbol PCM_4ms_Connector:Conn_01x04
- added R8: 10k, Resistor_SMD:R_0603_1608Metric_Pad0.98x0.95mm_HandSolder, symbol Device:R
- added U1: DS18B20+, DS18B20, symbol DS188B20+:DS18B20+
- renumbered C101 to C1, C102 to C2, C103 to C3, C104 to C4, C105 to C5, D25 to D1, D26 to D2, J11 to J1, J9 to J10, J2 to J11, J5 to J13, J7 to J14, J4 to J15, J8 to J16, J19 to J17, J6 to J18, J1 to J19, J12 to J2, J10 to J20, J20 to J21, J13 to J3, J14 to J4, J15 to J5, J16 to J6, J17 to J7, J18 to J8, J3 to J9, R75 to R1, R76 to R2, R77 to R3, R78 to R4, R79 to R5, R80 to R6, R81 to R7, S3 to S1, S4 to S2, U12 to U2, U13 to U3, U1 to U4
Connections:
- net GND: now also J12.2 (Pin_2), U1.1 (GND)
- net MOTOR_DRIVER_P3V3: now also J12.1 (Pin_1), R8.2, U1.3 (VDD)
- net PI_SCL: now also J12.3 (Pin_3)
- net PI_SDA: now also J12.4 (Pin_4)
- net TEMPERATURE_SENSOR: now reaches U2.25 (IO48)
- net TEMPERATURE_SENSOR: now also R8.1, U1.2 (DQ)
- no-connect marks 26 -> 25
Other:
- note added: "Stereo Cameras"
- note added: "Temperature Sensor"
- note removed: "io48 is unused, we can use if we need"
- moved on the sheet: J10, J9

Commit message: regular updates
Parts:
- J8: now in the parts list
Changed lines of the file:
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@@
 		(unit 1)
 		(exclude_from_sim no)
-		(in_bom no)
+		(in_bom yes)
 		(on_board yes)
 		(dnp no)

Commit message: Worked on FBD
Other:
- note added: "There are 2 headers because: BNO055 + BMP280"
Changed lines of the file:
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@@
 	(paper "A3")
 	(rectangle
-		(start 74.93 119.38)
+		(start 72.39 119.38)
 		(end 121.92 166.37)
 		(stroke
@@
 		(effects
 			(font
+				(size 1.27 1.27)
+			)
+		)
+	)
+	(text "There are 2 headers because: BNO055 + BMP280"
+		(exclude_from_sim no)
+		(at 97.028 121.158 0)
+		(effects
+			(font
