File: Schematic/STAR_FUEL_GAUGE.kicad_sch (KiCad schematic)
At the start: 50 parts, among them J1 6120XX21621_61200821621, J2 BMS_I2C, J3 Conn_01x02, J4 Conn_01x02, J5 6120XX21621_61200621621, J6 6120XX21621_61200621621, J7 SMB, Q1 ZXMP10A13FTA, Q2 BSS123, Q3 MMBT3904, U1 BQ78350DBT-R1A, U2 PCA9306D,118

Commit message: fuel gauge
Parts:
- added MP1, MP2, MP3, MP4: M3 Via, MountingHole:MountingHole_3.2mm_M3_Pad_Via, symbol Mechanical:MountingHole_Pad
Connections:
- net GND: now also MP1.1, MP2.1, MP3.1, MP4.1
Other:
- note added: "AFE"
- note added: "Gate Driver"
- note added: "MCU"
- company: (none) -> Locked Inc.
- title: (none) -> Fuel Gauge
- moved on the sheet: J1, J5, J6, R8

Commit message: fuel guage bom
fueal guage bom
Parts:
- J1: DigiKey Link (none) -> https://www.digikey.com/short/0fn8mfq4; DigiKey Part Number (none) -> 732-5395-ND; DigiKey Price per Unit (none) -> 0.97; Manufactaurer Part Number (none) -> 61200821621; Mouser Link (none) -> https://mou.sr/4rK5D6r; Mouser Part Number (none) -> 710-61200821621; Mouser Price per Unit (none) -> 1.08
- J2: DigiKey Link (none) -> https://www.digikey.com/short/w0z5733v; DigiKey Part Number (none) -> 2057-PH1-04-UA-ND; DigiKey Price per Unit (none) -> 0.10; Manufactaurer Part Number (none) -> PH1-04-UA; Mouser Link (none) -> https://mou.sr/3KIjcCG; Mouser Part Number (none) -> 737-PH1-04-UA; Mouser Price per Unit (none) -> 0.10
- J3, J4: DigiKey Link (none) -> https://www.digikey.com/short/n3b99f8m; DigiKey Part Number (none) -> 952-2262-ND; DigiKey Price per Unit (none) -> 0.10; Manufactaurer Part Number (none) -> M20-9990246; Mouser Link (none) -> https://mou.sr/3MtirxW; Mouser Part Number (none) -> 855-M20-9990246; Mouser Price per Unit (none) -> 0.10
- J5, J6: DigiKey Link (none) -> https://www.digikey.com/short/bdv8v937; DigiKey Part Number (none) -> 732-5394-ND; DigiKey Price per Unit (none) -> 0.43; Manufactaurer Part Number (none) -> 61200621621; Mouser Link (none) -> https://mou.sr/3XISxZx; Mouser Part Number (none) -> 710-61200621621; Mouser Price per Unit (none) -> 0.47
- J7: DigiKey Link (none) -> https://www.digikey.com/short/0fn8mfq4; DigiKey Part Number (none) -> 732-3040-1-ND; DigiKey Price per Unit (none) -> 0.73; Manufactaurer Part Number (none) -> 82306050029; Mouser Link (none) -> https://mou.sr/4nmVvNY; Mouser Part Number (none) -> 710-82306050029; Mouser Price per Unit (none) -> 0.73
