File: schematic/STAR_AFE.kicad_sch (KiCad schematic)
At the start: 89 parts, among them J1 1017495, J2 Conn_01x02, J3 694106301002, J4 6120XX21621_61200821621, J5 6120XX21621_61200821621, J6 1017491, J7 1017491, Q1 DMN2004K-7, Q2 DMN2004K-7, Q3 DMN2004K-7, Q4 CSD19531Q5AT, Q5 CSD19531Q5AT, Q6 ZXMP10A13FTA, Q7 CSD19531Q5AT, Q8 CSD19531Q5AT, Q9 FDD4141, U1 BQ7692000PWR

Commit message: Normalize KiCad symbol library structure
- Remove ul_ prefixes from Ultra Librarian exports (10 directories renamed, 2 duplicates deleted)
- Flatten directory structure (remove KiCad/KiCADv6 subdirectories from 93 components)
- Replace date-stamped filenames with part numbers (3 files renamed)
- Standardize separators: comma to hyphen (7 directories renamed)
- Update library table references (sym-lib-table: 84 entries, fp-lib-table: 85 entries)
- Update all schematic and PCB references (10 schematics + 10 PCBs)

Total changes:
- 100 component directories normalized to flat structure
- All library references updated and validated
- No ul_ prefixes, KiCad subdirs, date-stamped files, or commas in names remain
Parts:
- D10, D8: footprint PTVS14VP1UP,115:PMEG3050EP115 -> PTVS14VP1UP-115:PMEG3050EP115; symbol PTVS14VP1UP,115:PTVS14VP1UP,115 -> PTVS14VP1UP-115:PTVS14VP1UP,115
Connections:
- net BATT-: no longer D8.2 (A2)
- net PACK-: no longer D10.2 (A2)
- net at C15.2, C9.2, D11.5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: no longer D10.1 (A1)
- net at C6.1, F1.2, F1.4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: no longer D8.1 (A1)
Changed lines of the file:
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@@
 	)
 	(symbol
-		(lib_id "PTVS14VP1UP,115:PTVS14VP1UP,115")
+		(lib_id "PTVS14VP1UP-115:PTVS14VP1UP,115")
 		(at 218.44 200.66 90)
 		(unit 1)
@@
 			)
 		)
-		(property "Footprint" "PTVS14VP1UP,115:PMEG3050EP115"
+		(property "Footprint" "PTVS14VP1UP-115:PMEG3050EP115"
 			(at 312.09 190.5 0)
 			(effects
@@
 	)
 	(symbol
-		(lib_id "PTVS14VP1UP,115:PTVS14VP1UP,115")
+		(lib_id "PTVS14VP1UP-115:PTVS14VP1UP,115")
 		(at 156.21 200.66 90)
 		(unit 1)
@@
 			)
 		)
-		(property "Footprint" "PTVS14VP1UP,115:PMEG3050EP115"
+		(property "Footprint" "PTVS14VP1UP-115:PMEG3050EP115"
 			(at 249.86 190.5 0)
 			(effects

Commit message: Update AFE schematic: fix PTVS14VP1UP symbol reference
- Changed lib_id from PTVS14VP1UP,115 to PTVS14VP1UP-115
- Matches updated symbol name in library file
- Fixes schematic not opening issue
Parts:
- D10, D8: value PTVS14VP1UP,115 -> PTVS14VP1UP-115; symbol PTVS14VP1UP-115:PTVS14VP1UP,115 -> PTVS14VP1UP-115:PTVS14VP1UP-115; Manufactaurer Part Number PTVS14VP1UP,115 -> PTVS14VP1UP-115
Connections:
- net BATT-: now also D8.2 (A2)
- net PACK-: now also D10.2 (A2)
- net at C15.2, C9.2, D11.5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: now also D10.1 (A1)
- net at C6.1, F1.2, F1.4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: now also D8.1 (A1)
Changed lines of the file:
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@@
 	)
 	(symbol
-		(lib_id "PTVS14VP1UP-115:PTVS14VP1UP,115")
+		(lib_id "PTVS14VP1UP-115:PTVS14VP1UP-115")
 		(at 218.44 200.66 90)
 		(unit 1)
@@
 			)
 		)
-		(property "Value" "PTVS14VP1UP,115"
+		(property "Value" "PTVS14VP1UP-115"
 			(at 218.44 195.326 90)
 			(effects
@@
 			)
 		)
-		(property "Manufactaurer Part Number" "PTVS14VP1UP,115"
+		(property "Manufactaurer Part Number" "PTVS14VP1UP-115"
 			(at 218.44 200.66 90)
 			(effects
@@
 	)
 	(symbol
-		(lib_id "PTVS14VP1UP-115:PTVS14VP1UP,115")
+		(lib_id "PTVS14VP1UP-115:PTVS14VP1UP-115")
 		(at 156.21 200.66 90)
 		(unit 1)
@@
 			)
 		)
-		(property "Value" "PTVS14VP1UP,115"
+		(property "Value" "PTVS14VP1UP-115"
 			(at 156.21 195.326 90)
 			(effects
@@
 			)
 		)
-		(property "Manufactaurer Part Number" "PTVS14VP1UP,115"
+		(property "Manufactaurer Part Number" "PTVS14VP1UP-115"
 			(at 156.21 200.66 90)
 			(effects

Commit message: Fix typo: Manufactaurer → Manufacturer Part Number
- Corrected property name in all schematic, PCB, and project files
- Fixed 29 files across all board designs
Parts:
- C1, C2, C3, C4: Manufactaurer Part Number CL10B224KB8NNNC -> (none); Manufacturer Part Number (none) -> CL10B224KB8NNNC
- C10, C14, C15, C5, C6, C8, C9: Manufactaurer Part Number CC0603JRX7R9BB104 -> (none); Manufacturer Part Number (none) -> CC0603JRX7R9BB104
- C11, C13: Manufactaurer Part Number GRM21BR61H106KE43L -> (none); Manufacturer Part Number (none) -> GRM21BR61H106KE43L
- C12, C7: Manufactaurer Part Number 963-UMK107AB7105KA-T -> (none); Manufacturer Part Number (none) -> 963-UMK107AB7105KA-T
- C16: Manufactaurer Part Number VJ0603Y471KXAPW1BC -> (none); Manufacturer Part Number (none) -> VJ0603Y471KXAPW1BC
- C17, C18: Manufactaurer Part Number CGA3E2X7R1H472K080AA -> (none); Manufacturer Part Number (none) -> CGA3E2X7R1H472K080AA
- D1, D2, D3: Manufactaurer Part Number SML-D12Y1WT86 -> (none); Manufacturer Part Number (none) -> SML-D12Y1WT86
- D10, D8: Manufactaurer Part Number PTVS14VP1UP-115 -> (none); Manufacturer Part Number (none) -> PTVS14VP1UP-115
- D11: Manufactaurer Part Number V5N3202HM3/I -> (none); Manufacturer Part Number (none) -> V5N3202HM3/I
- D12: Manufactaurer Part Number 150060RS75000 -> (none); Manufacturer Part Number (none) -> 150060RS75000
- D4, D5, D6: Manufactaurer Part Number DDZ9690-7 -> (none); Manufacturer Part Number (none) -> DDZ9690-7
- D7: Manufactaurer Part Number 1N4148W -> (none); Manufacturer Part Number (none) -> 1N4148W
- D9: Manufactaurer Part Number MMSZ5226C-E3-08 -> (none); Manufacturer Part Number (none) -> MMSZ5226C-E3-08
- F1, F2: Manufactaurer Part Number 3568 -> (none); Manufacturer Part Number (none) -> 3568
- FB1, FB2, FB3, FB4: Manufactaurer Part Number BBPY00201209221Y00 -> (none); Manufacturer Part Number (none) -> BBPY00201209221Y00
- J1: Manufactaurer Part Number 1017495 -> (none); Manufacturer Part Number (none) -> 1017495
- J2: Manufactaurer Part Number M20-9990246 -> (none); Manufacturer Part Number (none) -> M20-9990246
- J3: Manufactaurer Part Number 694106301002 -> (none); Manufacturer Part Number (none) -> 694106301002
- J4, J5: Manufactaurer Part Number 61200821621 -> (none); Manufacturer Part Number (none) -> 61200821621
- J6, J7: Manufactaurer Part Number 1017491 -> (none); Manufacturer Part Number (none) -> 1017491
- Q1, Q2, Q3: Manufactaurer Part Number DMN2004K-7 -> (none); Manufacturer Part Number (none) -> DMN2004K-7
- Q4, Q5, Q7, Q8: Manufactaurer Part Number CSD19531Q5AT -> (none); Manufacturer Part Number (none) -> CSD19531Q5AT
- Q6: Manufactaurer Part Number ZXMP10A13FTA -> (none); Manufacturer Part Number (none) -> ZXMP10A13FTA
- Q9: Manufactaurer Part Number FDD4141 -> (none); Manufacturer Part Number (none) -> FDD4141
- R1, R15, R18, R2, R20, R3: Manufactaurer Part Number CRCW0603100RJNEA -> (none); Manufacturer Part Number (none) -> CRCW0603100RJNEA
- R10, R11, R13, R17, R26, R8: Manufactaurer Part Number AC0603JR-131KL -> (none); Manufacturer Part Number (none) -> AC0603JR-131KL
- R12, R14, R22, R24, R7, R9: Manufactaurer Part Number RT0603BRE0710KL -> (none); Manufacturer Part Number (none) -> RT0603BRE0710KL
- R16, R21, R23: Manufactaurer Part Number RK73H1JTTD1005F -> (none); Manufacturer Part Number (none) -> RK73H1JTTD1005F
- R19: Manufactaurer Part Number WSK1216L2000FEA -> (none); Manufacturer Part Number (none) -> WSK1216L2000FEA
- R25: Manufactaurer Part Number CRCW0603510KJNEA -> (none); Manufacturer Part Number (none) -> CRCW0603510KJNEA
- R27: Manufactaurer Part Number RT0603BRD0724RL -> (none); Manufacturer Part Number (none) -> RT0603BRD0724RL
- R28: Manufactaurer Part Number RC0603DR-073K01L -> (none); Manufacturer Part Number (none) -> RC0603DR-073K01L
- R4, R5, R6: Manufactaurer Part Number CRCW060333R0FKEAC -> (none); Manufacturer Part Number (none) -> CRCW060333R0FKEAC
- S1: Manufactaurer Part Number SKRPACE010 -> (none); Manufacturer Part Number (none) -> SKRPACE010
- TH1: Manufactaurer Part Number NTCGS163JX103DT7 -> (none); Manufacturer Part Number (none) -> NTCGS163JX103DT7
- U1: Manufactaurer Part Number BQ7692000PWR -> (none); Manufacturer Part Number (none) -> BQ7692000PWR
