File: schematic/STAR_FUEL_GAUGE.kicad_sch (KiCad schematic)
At the start: 54 parts, among them J1 6120XX21621_61200821621, J2 BMS_I2C, J3 Conn_01x02, J4 Conn_01x02, J5 6120XX21621_61200621621, J6 6120XX21621_61200621621, J7 SMB, Q1 ZXMP10A13FTA, Q2 BSS123, Q3 MMBT3904, U1 BQ78350DBT-R1A, U2 PCA9306D,118

Commit message: Fix typo: Manufactaurer → Manufacturer Part Number
- Corrected property name in all schematic, PCB, and project files
- Fixed 29 files across all board designs
Parts:
- C1, C2: Manufactaurer Part Number GCM188R71H332KA37D -> (none); Manufacturer Part Number (none) -> GCM188R71H332KA37D
- C3: Manufactaurer Part Number GRT21BR61H475KE13K -> (none); Manufacturer Part Number (none) -> GRT21BR61H475KE13K
- C4, C7: Manufactaurer Part Number 963-UMK107AB7105KA-T -> (none); Manufacturer Part Number (none) -> 963-UMK107AB7105KA-T
- C5, C6, C8: Manufactaurer Part Number CC0603JRX7R9BB104 -> (none); Manufacturer Part Number (none) -> CC0603JRX7R9BB104
- D1, D2, D3, D4, D5: Manufactaurer Part Number SML-D12M1WT86 -> (none); Manufacturer Part Number (none) -> SML-D12M1WT86
- D6, D7: Manufactaurer Part Number DDZ9690-7 -> (none); Manufacturer Part Number (none) -> DDZ9690-7
- D8, D9, J7: Manufactaurer Part Number 82306050029 -> (none); Manufacturer Part Number (none) -> 82306050029
- J1: Manufactaurer Part Number 61200821621 -> (none); Manufacturer Part Number (none) -> 61200821621
- J2: Manufactaurer Part Number PH1-04-UA -> (none); Manufacturer Part Number (none) -> PH1-04-UA
- J3, J4: Manufactaurer Part Number M20-9990246 -> (none); Manufacturer Part Number (none) -> M20-9990246
- J5, J6: Manufactaurer Part Number 61200621621 -> (none); Manufacturer Part Number (none) -> 61200621621
- Q1: Manufactaurer Part Number ZXMP10A13FTA -> (none); Manufacturer Part Number (none) -> ZXMP10A13FTA
- Q2: Manufactaurer Part Number BSS123 -> (none); Manufacturer Part Number (none) -> BSS123
- Q3: Manufactaurer Part Number MMBT3904 -> (none); Manufacturer Part Number (none) -> MMBT3904
- R1, R2, R4: Manufactaurer Part Number ERA-3AEB304V -> (none); Manufacturer Part Number (none) -> ERA-3AEB304V
- R10, R3, R6, R9: Manufactaurer Part Number AC0603JR-07100KL -> (none); Manufacturer Part Number (none) -> AC0603JR-07100KL
- R11, R12, R15, R16: Manufactaurer Part Number CRCW0603100RJNEA -> (none); Manufacturer Part Number (none) -> CRCW0603100RJNEA
- R13, R14: Manufactaurer Part Number AC0603FR-071ML -> (none); Manufacturer Part Number (none) -> AC0603FR-071ML
- R17: Manufactaurer Part Number CRCW0603220KFKEA -> (none); Manufacturer Part Number (none) -> CRCW0603220KFKEA
- R18, R8: Manufactaurer Part Number CRCW0603510KJNEA -> (none); Manufacturer Part Number (none) -> CRCW0603510KJNEA
- R19, R20, R7: Manufactaurer Part Number RT0603BRE0710KL -> (none); Manufacturer Part Number (none) -> RT0603BRE0710KL
- R5: Manufactaurer Part Number RT0603BRD0724K9L -> (none); Manufacturer Part Number (none) -> RT0603BRD0724K9L
- S1: Manufactaurer Part Number SKRPACE010 -> (none); Manufacturer Part Number (none) -> SKRPACE010
- U1: Manufactaurer Part Number BQ78350DBT-R1A -> (none); Manufacturer Part Number (none) -> BQ78350DBT-R1A
- U2: Manufactaurer Part Number PCA9306D,118 -> (none); Manufacturer Part Number (none) -> PCA9306D,118
Changed lines of the file:
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@@
 			)
 		)
-		(property "Manufactaurer Part Number" "GCM188R71H332KA37D"
+		(property "Manufacturer Part Number" "GCM188R71H332KA37D"
 			(at 74.93 123.19 0)
 			(effects
@@
 			)
 		)
-		(property "Manufactaurer Part Number" "PH1-04-UA"
+		(property "Manufacturer Part Number" "PH1-04-UA"
 			(at 152.4 144.78 0)
 			(effects
@@
 			)
 		)
-		(property "Manufactaurer Part Number" " SML-D12M1WT86 "
+		(property "Manufacturer Part Number" " SML-D12M1WT86 "
 			(at 205.74 132.08 0)
 			(effects
@@
 			)
 		)
-		(property "Manufactaurer Part Number" "963-UMK107AB7105KA-T"
+		(property "Manufacturer Part Number" "963-UMK107AB7105KA-T"
 			(at 189.23 109.22 90)
 			(effects
@@
 			)
 		)
-		(property "Manufactaurer Part Number" "CRCW0603100RJNEA"
+		(property "Manufacturer Part Number" "CRCW0603100RJNEA"
 			(at 200.66 147.32 90)
 			(effects
@@
 			)
 		)
-		(property "Manufactaurer Part Number" " DDZ9690-7"
+		(property "Manufacturer Part Number" " DDZ9690-7"
 			(at 234.95 154.94 90)
 			(effects
@@
 			)
 		)
-		(property "Manufactaurer Part Number" "RT0603BRE0710KL"
+		(property "Manufacturer Part Number" "RT0603BRE0710KL"
 			(at 102.87 144.78 0)
 			(effects
@@
 			)
 		)
-		(property "Manufactaurer Part Number" " SML-D12M1WT86 "
+		(property "Manufacturer Part Number" " SML-D12M1WT86 "
 			(at 205.74 134.62 0)
 			(effects
@@
 			)
 		)
-		(property "Manufactaurer Part Number" "BSS123"
+		(property "Manufacturer Part Number" "BSS123"
 			(at 113.03 111.76 0)
 			(effects
@@
 			)
 		)
-		(property "Manufactaurer Part Number" "82306050029"
+		(property "Manufacturer Part Number" "82306050029"
 			(at 267.97 176.53 0)
 			(effects
@@
 			)
 		)
-		(property "Manufactaurer Part Number" "ERA-3AEB304V "
+		(property "Manufacturer Part Number" "ERA-3AEB304V "
 			(at 81.28 137.16 90)
 			(effects
@@
 			)
 		)
-		(property "Manufactaurer Part Number" "CRCW0603100RJNEA"
+		(property "Manufacturer Part Number" "CRCW0603100RJNEA"
 			(at 200.66 149.86 90)
 			(effects
@@
 			)
 		)
-		(property "Manufactaurer Part Number" "M20-9990246"
+		(property "Manufacturer Part Number" "M20-9990246"
 			(at 307.34 125.73 0)
 			(effects
@@
 			)
 		)
-		(property "Manufactaurer Part Number" " DDZ9690-7"
+		(property "Manufacturer Part Number" " DDZ9690-7"
 			(at 228.6 154.94 90)
 			(effects
@@
 			)
 		)
-		(property "Manufactaurer Part Number" "PCA9306D,118"
+		(property "Manufacturer Part Number" "PCA9306D,118"
 			(at 363.22 125.73 0)
 			(effects
@@
 			)
 		)
-		(property "Manufactaurer Part Number" "RT0603BRE0710KL"
+		(property "Manufacturer Part Number" "RT0603BRE0710KL"
 			(at 313.69 114.3 0)
 			(effects
@@
 			)
 		)
-		(property "Manufactaurer Part Number" "61200621621"
+		(property "Manufacturer Part Number" "61200621621"
 			(at 209.55 226.06 90)
 			(effects
@@
 			)
 		)
-		(property "Manufactaurer Part Number" "AC0603FR-071ML"
+		(property "Manufacturer Part Number" "AC0603FR-071ML"
 			(at 219.71 154.94 0)
 			(effects
@@
 			)
 		)
-		(property "Manufactaurer Part Number" "ZXMP10A13FTA"
+		(property "Manufacturer Part Number" "ZXMP10A13FTA"
 			(at 50.8 105.41 0)
 			(effects
@@
 			)
 		)
-		(property "Manufactaurer Part Number" "GCM188R71H332KA37D"
+		(property "Manufacturer Part Number" "GCM188R71H332KA37D"
 			(at 95.25 143.51 0)
 			(effects
@@
 			)
 		)
-		(property "Manufactaurer Part Number" "ERA-3AEB304V "
+		(property "Manufacturer Part Number" "ERA-3AEB304V "
 			(at 59.69 116.84 90)
 			(effects
@@
 			)
 		)
-		(property "Manufactaurer Part Number" "82306050029"
+		(property "Manufacturer Part Number" "82306050029"
 			(at 289.56 176.53 0)
 			(effects
@@
 			)
 		)
-		(property "Manufactaurer Part Number" "GRT21BR61H475KE13K"
+		(property "Manufacturer Part Number" "GRT21BR61H475KE13K"
 			(at 189.23 104.14 90)
 			(effects
@@
 			)
 		)
-		(property "Manufactaurer Part Number" "AC0603JR-07100KL"
+		(property "Manufacturer Part Number" "AC0603JR-07100KL"
 			(at 101.6 105.41 90)
 			(effects
@@
 			)
 		)
-		(property "Manufactaurer Part Number" "963-UMK107AB7105KA-T"
+		(property "Manufacturer Part Number" "963-UMK107AB7105KA-T"
 			(at 222.25 118.11 90)
 			(effects
@@
 			)
 		)
-		(property "Manufactaurer Part Number" "M20-9990246"
+		(property "Manufacturer Part Number" "M20-9990246"
 			(at 326.39 125.73 0)
 			(effects
@@
 			)
 		)
-		(property "Manufactaurer Part Number" "CC0603JRX7R9BB104"
+		(property "Manufacturer Part Number" "CC0603JRX7R9BB104"
 			(at 189.23 114.3 90)
 			(effects
@@
 			)
 		)
-		(property "Manufactaurer Part Number" "CRCW0603510KJNEA"
+		(property "Manufacturer Part Number" "CRCW0603510KJNEA"
 			(at 144.78 143.51 0)
 			(effects
@@
 			)
 		)
-		(property "Manufactaurer Part Number" "CRCW0603510KJNEA"
+		(property "Manufacturer Part Number" "CRCW0603510KJNEA"
 			(at 288.29 134.62 0)
 			(effects
@@
 			)
 		)
-		(property "Manufactaurer Part Number" "CC0603JRX7R9BB104"
+		(property "Manufacturer Part Number" "CC0603JRX7R9BB104"
 			(at 222.25 123.19 90)
 			(effects
@@
 			)
 		)
-		(property "Manufactaurer Part Number" "AC0603JR-07100KL"
+		(property "Manufacturer Part Number" "AC0603JR-07100KL"
 			(at 74.93 99.06 0)
 			(effects
@@
 			)
 		)
-		(property "Manufactaurer Part Number" "ERA-3AEB304V "
+		(property "Manufacturer Part Number" "ERA-3AEB304V "
 			(at 57.15 137.16 90)
 			(effects
@@
 			)
 		)
-		(property "Manufactaurer Part Number" "CRCW0603100RJNEA"
+		(property "Manufacturer Part Number" "CRCW0603100RJNEA"
 			(at 250.19 149.86 90)
 			(effects
@@
 			)
 		)
-		(property "Manufactaurer Part Number" "AC0603JR-07100KL"
+		(property "Manufacturer Part Number" "AC0603JR-07100KL"
 			(at 152.4 110.49 0)
 			(effects
@@
 			)
 		)
-		(property "Manufactaurer Part Number" "61200621621"
+		(property "Manufacturer Part Number" "61200621621"
 			(at 278.13 229.87 90)
 			(effects
@@
 			)
 		)
-		(property "Manufactaurer Part Number" "BQ78350DBT-R1A"
+		(property "Manufacturer Part Number" "BQ78350DBT-R1A"
 			(at 180.34 147.32 0)
 			(effects
@@
 			)
 		)
-		(property "Manufactaurer Part Number" "RT0603BRE0710KL"
+		(property "Manufacturer Part Number" "RT0603BRE0710KL"
 			(at 320.04 114.3 0)
 			(effects
@@
 			)
 		)
-		(property "Manufactaurer Part Number" " SML-D12M1WT86 "
+		(property "Manufacturer Part Number" " SML-D12M1WT86 "
 			(at 205.74 127 0)
 			(effects
@@
 			)
 		)
-		(property "Manufactaurer Part Number" "CC0603JRX7R9BB104"
+		(property "Manufacturer Part Number" "CC0603JRX7R9BB104"
 			(at 199.39 167.64 0)
 			(effects
@@
 			)
 		)
-		(property "Manufactaurer Part Number" " SML-D12M1WT86 "
+		(property "Manufacturer Part Number" " SML-D12M1WT86 "
 			(at 205.74 124.46 0)
 			(effects
@@
 			)
 		)
-		(property "Manufactaurer Part Number" "SKRPACE010"
+		(property "Manufacturer Part Number" "SKRPACE010"
 			(at 247.65 134.62 0)
 			(effects
@@
 			)
 		)
-		(property "Manufactaurer Part Number" "CRCW0603100RJNEA"
+		(property "Manufacturer Part Number" "CRCW0603100RJNEA"
 			(at 250.19 147.32 90)
 			(effects
@@
 			)
 		)
-		(property "Manufactaurer Part Number" "AC0603JR-07100KL"
+		(property "Manufacturer Part Number" "AC0603JR-07100KL"
 			(at 168.91 114.3 90)
 			(effects
@@
 			)
 		)
-		(property "Manufactaurer Part Number" "82306050029"
+		(property "Manufacturer Part Number" "82306050029"
 			(at 342.9 149.86 0)
 			(effects
@@
 			)
 		)
-		(property "Manufactaurer Part Number" " SML-D12M1WT86 "
+		(property "Manufacturer Part Number" " SML-D12M1WT86 "
 			(at 205.74 129.54 0)
 			(effects
@@
 			)
 		)
-		(property "Manufactaurer Part Number" "RT0603BRD0724K9L"
+		(property "Manufacturer Part Number" "RT0603BRD0724K9L"
 			(at 82.55 123.19 0)
 			(effects
@@
 			)
 		)
-		(property "Manufactaurer Part Number" "61200821621"
+		(property "Manufacturer Part Number" "61200821621"
 			(at 142.24 223.52 90)
 			(effects
@@
 			)
 		)
-		(property "Manufactaurer Part Number" "CRCW0603220KFKEA"
+		(property "Manufacturer Part Number" "CRCW0603220KFKEA"
 			(at 261.62 127 90)
 			(effects
@@
 			)
 		)
-		(property "Manufactaurer Part Number" "AC0603FR-071ML"
+		(property "Manufacturer Part Number" "AC0603FR-071ML"
 			(at 212.09 154.94 0)
 			(effects
@@
 			)
 		)
-		(property "Manufactaurer Part Number" "MMBT3904"
+		(property "Manufacturer Part Number" "MMBT3904"
 			(at 218.44 107.95 0)
 			(effects
