File: schematic/STAR_MCU.kicad_sch (KiCad schematic)
At the start: 159 parts, among them J1 EMU CFG, J10 Conn_01x04, J11 6120XX21621_61200621621, J12 Conn_01x04, J13 6120XX21621_61200821621, J14 6120XX21621_61200821621, J15 6120XX21621_61200821621, J16 6120XX21621_61200821621, J17 SSW-106-02-G-S-RA, J18 6120XX21621_61200621621, J19 6120XX21621_61200821621, J2 USB4216-03-A, J20 S5B-XH-A, J21 6120XX21621_61200621621, J22 SSW-106-02-G-S-RA, J23 Conn_02x20_Odd_Even, J24 HC-SR04, J25 HC-SR04, J26 HC-SR04, J27 HC-SR04, J28 HC-SR04, J29 HC-SR04, J3 UPSEL_CFG, J30 HC-SR04, J31 SSW-106-02-G-S-RA, J32 SSW-106-02-G-S-RA, J4 E1E2-Emulator-Interface, J5 SSW-106-02-G-S-RA, J6 SSW-106-02-G-D-RA, J7 USB4216-03-A, J8 Conn_02x20_Odd_Even, J9 Conn_01x09, SW1 OP_CFG, U1 R5F572NNHGFP-30, U2 CY7C65213A-28PVXI, U3 TVS2200DRV, U4 LDL1117S33R, U5 TPS2116DRLR, U6 TVS2200DRV, U7 DS18B20+, Y1 24MHz

Commit message: MCU ready for a look over
Parts:
- added J33, J34, J35, J36, J37, J38, J39: HC-SR04, Connector_PinSocket_2.54mm:PinSocket_1x04_P2.54mm_Vertical, symbol Connector:Conn_01x04_Socket
Connections:
- net HCSR04_ECHO1 is gone; now on net PMOD_JB_GPIO1: J24.3 (Pin_3)
- net HCSR04_ECHO2 is gone; now on net PMOD_JB_GPIO3: J25.3 (Pin_3)
- net HCSR04_ECHO3 is gone; now on net PMOD_JE_GPIO1: J26.3 (Pin_3)
- net HCSR04_ECHO4 is gone; now on net PMOD_JE_GPIO3: J27.3 (Pin_3)
- net HCSR04_ECHO5 is gone; now on net PMOD_JC_INT2: J28.3 (Pin_3)
- net HCSR04_ECHO6 is gone; now on net PMOD_JC_SDA: J29.3 (Pin_3)
- net HCSR04_ECHO7 is gone; now on net PMOD_JF_GPIO1: J30.3 (Pin_3)
- net HCSR04_TRIG1 is gone; now on net PMOD_JB_GPIO0: J24.2 (Pin_2)
- net HCSR04_TRIG2 is gone; now on net PMOD_JB_GPIO2: J25.2 (Pin_2)
- net HCSR04_TRIG3 is gone; now on net PMOD_JE_GPIO0: J26.2 (Pin_2)
- net HCSR04_TRIG4 is gone; now on net PMOD_JE_GPIO2: J27.2 (Pin_2)
- net HCSR04_TRIG5 is gone; now on net PMOD_JC_INT1: J28.2 (Pin_2)
- net HCSR04_TRIG6 is gone; now on net PMOD_JC_SCL: J29.2 (Pin_2)
- net HCSR04_TRIG7 is gone; now on net PMOD_JF_GPIO0: J30.2 (Pin_2)
- net GND: now also J33.4 (Pin_4), J34.4 (Pin_4), J35.4 (Pin_4), J36.4 (Pin_4), J37.4 (Pin_4), J38.4 (Pin_4), J39.4 (Pin_4)
- net P3V3_BUCK: now also J33.1 (Pin_1), J34.1 (Pin_1), J35.1 (Pin_1), J36.1 (Pin_1), J37.1 (Pin_1), J38.1 (Pin_1), J39.1 (Pin_1)
- net PMOD_JA_CIPO: now also J36.3 (Pin_3)
- net PMOD_JA_COPI: now also J37.2 (Pin_2)
- net PMOD_JA_CS0: now also J37.3 (Pin_3)
- net PMOD_JA_CS1: now also J38.2 (Pin_2)
- net PMOD_JA_DC: now also J39.3 (Pin_3)
- net PMOD_JA_GPIO: now also J38.3 (Pin_3)
- net PMOD_JA_RST: now also J39.2 (Pin_2)
- net PMOD_JA_SCK: now also J36.2 (Pin_2)
- net PMOD_JD_GPIO0: now also J34.2 (Pin_2)
- net PMOD_JD_GPIO1: now also J34.3 (Pin_3)
- net PMOD_JD_GPIO2: now also J35.2 (Pin_2)
- net PMOD_JD_GPIO3: now also J35.3 (Pin_3)
- net PMOD_JF_SCL: now also J33.2 (Pin_2)
- net PMOD_JF_SDA: now also J33.3 (Pin_3)
Other:
- note added: "RPi5"
- moved on the sheet: J24, J25, J26, J27, J28, J29, J30

Commit message: MCU is ready for review
Parts:
- removed J28, J29, J30, J33, J34, J35, J36, J37, J38, J39: HC-SR04, Connector_PinSocket_2.54mm:PinSocket_1x04_P2.54mm_Vertical, symbol Connector:Conn_01x04_Socket
- added D10, D11, D12, D13, D14, D15, D16, D17, D18, D19, D29, D30, D31, D32, D33, D34, D35, D36, D37, D9: RED, SML-D12Y1WT86:LEDC1608X55N, symbol PCM_SL_Devices:LED
- added J28, J29, J30, J33, J34, J35, J36, J37, J38, J39, J40, J41, J42, J43, J44, J45, J46, J47, J48, J49: Conn_01x02, Connector_PinHeader_2.54mm:PinHeader_1x02_P2.54mm_Vertical, symbol Connector_Generic:Conn_01x02
- added R35, R36, R38, R39, R40, R41, R42, R44, R45, R46, R47, R57, R58, R59, R60, R61, R62, R63, R64, R65: 68R, Resistor_SMD:R_0603_1608Metric_Pad0.98x0.95mm_HandSolder, symbol Device:R
Connections:
- net GND: now also D10.1, D11.1, D12.1, D13.1, D14.1, D15.1, D16.1, D17.1, D18.1, D19.1, D29.1, D30.1, D31.1, D32.1, D33.1, D34.1, D35.1, D36.1, D37.1, D9.1
- net PMOD_JA_CIPO: now also J43.1 (Pin_1)
- net PMOD_JA_COPI: now also J44.1 (Pin_1)
- net PMOD_JA_CS0: now also J45.1 (Pin_1)
- net PMOD_JA_CS1: now also J46.1 (Pin_1)
- net PMOD_JA_DC: now also J49.1 (Pin_1)
- net PMOD_JA_GPIO: now also J47.1 (Pin_1)
- net PMOD_JA_RST: now also J48.1 (Pin_1)
- net PMOD_JA_SCK: now also J42.1 (Pin_1)
- net PMOD_JC_INT1: now also J28.1 (Pin_1)
- net PMOD_JC_INT2: now also J29.1 (Pin_1)
- net PMOD_JC_SCL: now also J30.1 (Pin_1)
- net PMOD_JC_SDA: now also J33.1 (Pin_1)
- net PMOD_JD_GPIO0: now also J34.1 (Pin_1)
- net PMOD_JD_GPIO1: now also J35.1 (Pin_1)
- net PMOD_JD_GPIO2: now also J36.1 (Pin_1)
- net PMOD_JD_GPIO3: now also J37.1 (Pin_1)
- net PMOD_JF_GPIO0: now also J38.1 (Pin_1)
- net PMOD_JF_GPIO1: now also J39.1 (Pin_1)
- net PMOD_JF_SCL: now also J40.1 (Pin_1)
- net PMOD_JF_SDA: now also J41.1 (Pin_1)
- new net: J36.2 (Pin_2), R59.1
- new net: D31.2, R59.2
- new net: J43.2 (Pin_2), R65.1
- new net: D37.2, R65.2
- new net: J37.2 (Pin_2), R60.1
- new net: D32.2, R60.2
- new net: J44.2 (Pin_2), R41.1
- new net: D16.2, R44.2
- new net: J42.2 (Pin_2), R64.1
- new net: J29.2 (Pin_2), R36.1
- new net: D10.2, R36.2
- new net: D14.2, R41.2
- new net: D9.2, R35.2
- new net: J33.2 (Pin_2), R39.1
- new net: D12.2, R39.2
- new net: J30.2 (Pin_2), R38.1
- new net: J41.2 (Pin_2), R63.1
- new net: D35.2, R63.2
- new net: D18.2, R46.2
- new net: J47.2 (Pin_2), R45.1
- new net: J49.2 (Pin_2), R47.1
- new net: D19.2, R47.2
- new net: D36.2, R64.2
- new net: D15.2, R42.2
- new net: D11.2, R38.2
- new net: J40.2 (Pin_2), R62.1
- new net: J46.2 (Pin_2), R44.1
- new net: J48.2 (Pin_2), R46.1
- new net: D29.2, R57.2
- new net: D30.2, R58.2
- new net: J38.2 (Pin_2), R40.1
- new net: J45.2 (Pin_2), R42.1
- new net: J34.2 (Pin_2), R57.1
- new net: D13.2, R40.2
- new net: D33.2, R61.2
- new net: J39.2 (Pin_2), R61.1
- new net: J28.2 (Pin_2), R35.1
- new net: D34.2, R62.2
- new net: J35.2 (Pin_2), R58.1
- new net: D17.2, R45.2
Other:
- note added: "LEDs"
- moved on the sheet: J17, J22, J24, J25, J26, J27, J31, J32, J5, J6
