File: schematic/STAR_MOTOR_DRIVER.kicad_sch (KiCad schematic)
At the start: 46 parts, among them J1 6120XX21621_61200821621, J10 B6B-XH-A, J11 B6B-XH-A, J12 B6B-XH-A, J2 6120XX21621_61200621621, J3 B6B-XH-A, J4 6120XX21621_61200821621, J5 6120XX21621_61200821621, J6 6120XX21621_61200821621, J7 1017491, U1 DRV8243SQDGQRQ1 (S-Variant), U2 DRV8243SQDGQRQ1 (S-Variant), U3 DRV8243SQDGQRQ1 (S-Variant), U4 DRV8243SQDGQRQ1 (S-Variant)

Commit message: Fix typo: Manufactaurer → Manufacturer Part Number
- Corrected property name in all schematic, PCB, and project files
- Fixed 29 files across all board designs
Parts:
- C1, C2, C3, C4: Manufactaurer Part Number 865080343007 -> (none); Manufacturer Part Number (none) -> 865080343007
- C10, C11, C12, C9: Manufactaurer Part Number CC0603JRX7R9BB104 -> (none); Manufacturer Part Number (none) -> CC0603JRX7R9BB104
- C5, C6, C7, C8: Manufactaurer Part Number CL10B224KB8NNNC -> (none); Manufacturer Part Number (none) -> CL10B224KB8NNNC
- D1, D2, D3, D4: Manufactaurer Part Number 150060RS75000 -> (none); Manufacturer Part Number (none) -> 150060RS75000
- J1, J4, J5, J6: Manufactaurer Part Number 61200821621 -> (none); Manufacturer Part Number (none) -> 61200821621
- J10, J11, J12, J3: Manufactaurer Part Number B6B-XH-A -> (none); Manufacturer Part Number (none) -> B6B-XH-A
- J2: Manufactaurer Part Number 61200621621 -> (none); Manufacturer Part Number (none) -> 61200621621
- J7: Manufactaurer Part Number 1017491 -> (none); Manufacturer Part Number (none) -> 1017491
- R1, R2, R3, R4: Manufactaurer Part Number RT0603BRE0710KL -> (none); Manufacturer Part Number (none) -> RT0603BRE0710KL
- R10, R11, R12, R9: Manufactaurer Part Number ERA-3AEB3161V -> (none); Manufacturer Part Number (none) -> ERA-3AEB3161V
- R5, R6, R7, R8: Manufactaurer Part Number RT0603FRE0768RL -> (none); Manufacturer Part Number (none) -> RT0603FRE0768RL
- U1, U2, U3, U4: Manufactaurer Part Number DRV8243SQDGQRQ1 -> (none); Manufacturer Part Number (none) -> DRV8243SQDGQRQ1
Changed lines of the file:
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@@
 			)
 		)
-		(property "Manufactaurer Part Number" "RT0603BRE0710KL"
+		(property "Manufacturer Part Number" "RT0603BRE0710KL"
 			(at 153.67 101.6 0)
 			(effects
@@
 			)
 		)
-		(property "Manufactaurer Part Number" "  61200621621"
+		(property "Manufacturer Part Number" "  61200621621"
 			(at 270.51 175.26 90)
 			(effects
@@
 			)
 		)
-		(property "Manufactaurer Part Number" "CC0603JRX7R9BB104"
+		(property "Manufacturer Part Number" "CC0603JRX7R9BB104"
 			(at 35.56 52.07 0)
 			(effects
@@
 			)
 		)
-		(property "Manufactaurer Part Number" "CL10B224KB8NNNC"
+		(property "Manufacturer Part Number" "CL10B224KB8NNNC"
 			(at 29.21 179.07 0)
 			(effects
@@
 			)
 		)
-		(property "Manufactaurer Part Number" "865080343007 "
+		(property "Manufacturer Part Number" "865080343007 "
 			(at 22.86 179.07 0)
 			(effects
@@
 			)
 		)
-		(property "Manufactaurer Part Number" "ERA-3AEB3161V"
+		(property "Manufacturer Part Number" "ERA-3AEB3161V"
 			(at 168.91 245.11 0)
 			(effects
@@
 			)
 		)
-		(property "Manufactaurer Part Number" "B6B-XH-A"
+		(property "Manufacturer Part Number" "B6B-XH-A"
 			(at 297.18 102.87 0)
 			(effects
@@
 			)
 		)
-		(property "Manufactaurer Part Number" "RT0603BRE0710KL"
+		(property "Manufacturer Part Number" "RT0603BRE0710KL"
 			(at 152.4 33.02 0)
 			(effects
@@
 			)
 		)
-		(property "Manufactaurer Part Number" "CL10B224KB8NNNC"
+		(property "Manufacturer Part Number" "CL10B224KB8NNNC"
 			(at 29.21 52.07 0)
 			(effects
@@
 			)
 		)
-		(property "Manufactaurer Part Number" "865080343007 "
+		(property "Manufacturer Part Number" "865080343007 "
 			(at 22.86 52.07 0)
 			(effects
@@
 			)
 		)
-		(property "Manufactaurer Part Number" "61200821621"
+		(property "Manufacturer Part Number" "61200821621"
 			(at 339.09 191.77 90)
 			(effects
@@
 			)
 		)
-		(property "Manufactaurer Part Number" "CL10B224KB8NNNC"
+		(property "Manufacturer Part Number" "CL10B224KB8NNNC"
 			(at 29.21 247.65 0)
 			(effects
@@
 			)
 		)
-		(property "Manufactaurer Part Number" "DRV8243SQDGQRQ1"
+		(property "Manufacturer Part Number" "DRV8243SQDGQRQ1"
 			(at 66.04 30.48 0)
 			(effects
@@
 			)
 		)
-		(property "Manufactaurer Part Number" "865080343007 "
+		(property "Manufacturer Part Number" "865080343007 "
 			(at 22.86 120.65 0)
 			(effects
@@
 			)
 		)
-		(property "Manufactaurer Part Number" "CC0603JRX7R9BB104"
+		(property "Manufacturer Part Number" "CC0603JRX7R9BB104"
 			(at 35.56 247.65 0)
 			(effects
@@
 			)
 		)
-		(property "Manufactaurer Part Number" "DRV8243SQDGQRQ1"
+		(property "Manufacturer Part Number" "DRV8243SQDGQRQ1"
 			(at 66.04 226.06 0)
 			(effects
@@
 			)
 		)
-		(property "Manufactaurer Part Number" "B6B-XH-A"
+		(property "Manufacturer Part Number" "B6B-XH-A"
 			(at 377.19 101.6 0)
 			(effects
@@
 			)
 		)
-		(property "Manufactaurer Part Number" "B6B-XH-A"
+		(property "Manufacturer Part Number" "B6B-XH-A"
 			(at 297.18 52.07 0)
 			(effects
@@
 			)
 		)
-		(property "Manufactaurer Part Number" "1017491"
+		(property "Manufacturer Part Number" "1017491"
 			(at 251.46 207.01 0)
 			(effects
@@
 			)
 		)
-		(property "Manufactaurer Part Number" "DRV8243SQDGQRQ1"
+		(property "Manufacturer Part Number" "DRV8243SQDGQRQ1"
 			(at 66.04 99.06 0)
 			(effects
@@
 			)
 		)
-		(property "Manufactaurer Part Number" "ERA-3AEB3161V"
+		(property "Manufacturer Part Number" "ERA-3AEB3161V"
 			(at 168.91 49.53 0)
 			(effects
@@
 			)
 		)
-		(property "Manufactaurer Part Number" "61200821621"
+		(property "Manufacturer Part Number" "61200821621"
 			(at 340.36 233.68 90)
 			(effects
@@
 			)
 		)
-		(property "Manufactaurer Part Number" "150060RS75000 "
+		(property "Manufacturer Part Number" "150060RS75000 "
 			(at 177.8 27.94 0)
 			(effects
@@
 			)
 		)
-		(property "Manufactaurer Part Number" "61200821621"
+		(property "Manufacturer Part Number" "61200821621"
 			(at 339.09 217.17 90)
 			(effects
@@
 			)
 		)
-		(property "Manufactaurer Part Number" "CC0603JRX7R9BB104"
+		(property "Manufacturer Part Number" "CC0603JRX7R9BB104"
 			(at 35.56 120.65 0)
 			(effects
@@
 			)
 		)
-		(property "Manufactaurer Part Number" "865080343007 "
+		(property "Manufacturer Part Number" "865080343007 "
 			(at 22.86 247.65 0)
 			(effects
@@
 			)
 		)
-		(property "Manufactaurer Part Number" "RT0603BRE0710KL"
+		(property "Manufacturer Part Number" "RT0603BRE0710KL"
 			(at 153.67 228.6 0)
 			(effects
@@
 			)
 		)
-		(property "Manufactaurer Part Number" "RT0603FRE0768RL"
+		(property "Manufacturer Part Number" "RT0603FRE0768RL"
 			(at 163.83 223.52 90)
 			(effects
@@
 			)
 		)
-		(property "Manufactaurer Part Number" "CL10B224KB8NNNC"
+		(property "Manufacturer Part Number" "CL10B224KB8NNNC"
 			(at 29.21 120.65 0)
 			(effects
@@
 			)
 		)
-		(property "Manufactaurer Part Number" "150060RS75000 "
+		(property "Manufacturer Part Number" "150060RS75000 "
 			(at 177.8 96.52 0)
 			(effects
@@
 			)
 		)
-		(property "Manufactaurer Part Number" "150060RS75000 "
+		(property "Manufacturer Part Number" "150060RS75000 "
 			(at 177.8 223.52 0)
 			(effects
@@
 			)
 		)
-		(property "Manufactaurer Part Number" "RT0603FRE0768RL"
+		(property "Manufacturer Part Number" "RT0603FRE0768RL"
 			(at 163.83 96.52 90)
 			(effects
@@
 			)
 		)
-		(property "Manufactaurer Part Number" "RT0603FRE0768RL"
+		(property "Manufacturer Part Number" "RT0603FRE0768RL"
 			(at 163.83 27.94 90)
 			(effects
@@
 			)
 		)
-		(property "Manufactaurer Part Number" "RT0603BRE0710KL"
+		(property "Manufacturer Part Number" "RT0603BRE0710KL"
 			(at 152.4 160.02 0)
 			(effects
@@
 			)
 		)
-		(property "Manufactaurer Part Number" "CC0603JRX7R9BB104"
+		(property "Manufacturer Part Number" "CC0603JRX7R9BB104"
 			(at 35.56 179.07 0)
 			(effects
@@
 			)
 		)
-		(property "Manufactaurer Part Number" "ERA-3AEB3161V"
+		(property "Manufacturer Part Number" "ERA-3AEB3161V"
 			(at 168.91 118.11 0)
 			(effects
@@
 			)
 		)
-		(property "Manufactaurer Part Number" "ERA-3AEB3161V"
+		(property "Manufacturer Part Number" "ERA-3AEB3161V"
 			(at 168.91 176.53 0)
 			(effects
@@
 			)
 		)
-		(property "Manufactaurer Part Number" "61200821621"
+		(property "Manufacturer Part Number" "61200821621"
 			(at 340.36 172.72 90)
 			(effects
@@
 			)
 		)
-		(property "Manufactaurer Part Number" "150060RS75000 "
+		(property "Manufacturer Part Number" "150060RS75000 "
 			(at 177.8 154.94 0)
 			(effects
@@
 			)
 		)
-		(property "Manufactaurer Part Number" "RT0603FRE0768RL"
+		(property "Manufacturer Part Number" "RT0603FRE0768RL"
 			(at 163.83 154.94 90)
 			(effects
@@
 			)
 		)
-		(property "Manufactaurer Part Number" "DRV8243SQDGQRQ1"
+		(property "Manufacturer Part Number" "DRV8243SQDGQRQ1"
 			(at 66.04 157.48 0)
 			(effects
@@
 			)
 		)
-		(property "Manufactaurer Part Number" "B6B-XH-A"
+		(property "Manufacturer Part Number" "B6B-XH-A"
 			(at 377.19 53.34 0)
 			(effects
