File: schematic/STAR_POWER_BOARD.kicad_sch (KiCad schematic)
At the start: 72 parts, among them J1 1017491, J10 1017491, J11 1017491, J12 Conn_02x03_Counter_Clockwise, J2 USB4216-03-A, J3 1017491, J4 1017491, J5 1017491, J6 1017491, J9 1017491, Q1 CSD18540Q5B, Q2 CSD17577Q3A, Q3 CSD17577Q3A, Q4 CSD18540Q5B, Q5 SISS71DN-T1-GE3, U1 TPS566238PRQFR, U2 TPS566238PRQFR, U3 TPS40305DRCT

Commit message: added note
Parts:
- removed Q5: SISS71DN-T1-GE3, MOSFET_3DN-T1-GE3_VIS, symbol User_CADS:SISS71DN-T1-GE3
- added C34, C38, C41, C47, C48, C53, C60, C65, C75, C80, C84: 100n, Capacitor_SMD:C_0603_1608Metric_Pad1.08x0.95mm_HandSolder, symbol Device:C
- added C35: 1u, Capacitor_SMD:C_0603_1608Metric_Pad1.08x0.95mm_HandSolder, symbol Device:C
- added C36, C37, C39, C40, C42, C43, C44, C45, C46, C58, C61, C66, C67, C68, C69, C70, C71, C72, C73, C74, C77, C78, C79, C81, C82, C83: 10u, Capacitor_SMD:C_0805_2012Metric_Pad1.18x1.45mm_HandSolder, symbol Device:C
- added C49, C50, C62: 4u7, Capacitor_SMD:C_0805_2012Metric_Pad1.18x1.45mm_HandSolder, symbol Device:C
- added C51, C52: 330p, Capacitor_SMD:C_0603_1608Metric_Pad1.08x0.95mm_HandSolder, symbol Device:C
- added C54, C55, C56, C57: 10n, Capacitor_SMD:C_0603_1608Metric_Pad1.08x0.95mm_HandSolder, symbol Device:C
- added C59, C85, C86, C87: 22u, T527T226M025ATE100:CAPPM3528X120N, symbol Device:C_Polarized
- added C63, C64: 47n, Capacitor_SMD:C_0603_1608Metric_Pad1.08x0.95mm_HandSolder, symbol Device:C
- added C76: 1n, Capacitor_SMD:C_0603_1608Metric_Pad1.08x0.95mm_HandSolder, symbol Device:C
- added D1, D2: 82306050029, 82306050029:WESURGE_0603134, symbol 82306050029:82306050029
- added D3: RED, SML-D12Y1WT86:LEDC1608X55N, symbol PCM_SL_Devices:LED
- added FB1: 22R, Resistor_SMD:R_0603_1608Metric_Pad0.98x0.95mm_HandSolder, symbol Device:FerriteBead_Small
- added J13: PD_DBG, Connector_PinHeader_2.54mm:PinHeader_1x03_P2.54mm_Vertical, symbol Connector_Generic:Conn_01x03
- added J14: 1017491, 1017491, symbol 1017491:1017491
- added J16: PD_I2C, Connector_PinHeader_2.54mm:PinHeader_1x04_P2.54mm_Vertical, symbol Connector_Generic:Conn_01x04
- added J19: 6120XX21621_61200821621, 61200821621:61200821621, symbol 61200821621:6120XX21621_61200821621
- added J2, J21: 6120XX21621_61200621621, 61200621621:61200621621, symbol 61200621621:6120XX21621_61200621621
- added L4: VLS6045EX-1R0N, VLS6045EX-1R0N:VLS6045, symbol VLS6045EX-1R0N:VLS6045EX-1R0N
- added NT1: NetTie_2, NetTie:NetTie-2_SMD_Pad0.5mm, symbol Device:NetTie_2
- added R15, R16, R17, R18, R22: 10k, Resistor_SMD:R_0603_1608Metric_Pad0.98x0.95mm_HandSolder, symbol Device:R
- added R19, R20: 3k3, Resistor_SMD:R_0603_1608Metric_Pad0.98x0.95mm_HandSolder, symbol Device:R
- added R21: 100k, Resistor_SMD:R_0603_1608Metric_Pad0.98x0.95mm_HandSolder, symbol Device:R
- added R23: 68R, Resistor_SMD:R_0603_1608Metric_Pad0.98x0.95mm_HandSolder, symbol Device:R
- added R24: 10k5, Resistor_SMD:R_0603_1608Metric_Pad0.98x0.95mm_HandSolder, symbol Device:R
- added R25: 100R, Resistor_SMD:R_0603_1608Metric_Pad0.98x0.95mm_HandSolder, symbol Device:R
- added TH1: NTCGS163JX103DT7, NTCGS163JX103DT7:THRMC1608X90N, symbol NTCGS163JX103DT7:NTCGS163JX103DT7
- added U4: CAT24C512WI-GT3, CAT24C512WI-GT3:SOIC127P600X175-8N, symbol CAT24C512WI:CAT24C512WI-GT3
- added U5: TPS25751DREFR, TPS25751DREFR:TPS25751DREFR, symbol TPS25751DREFR:TPS25751DREFR
- added U6: TVS2200DRV, TVS2200DRVR:SON65P200X200X80-7N, symbol Power_Protection:TVS2200DRV
- added U7: BQ25798RQMR, BQ25798RQMR:BQ25798RQMR, symbol BQ25798RQMR:BQ25798RQMR
- C1, C2, C24, C25, C26, C27, C28, C3, C30, C5, C6, C9: value 22uF -> 22u
- C10, C4, C7: value 47uF -> 47u
- C11: value 3.3nF -> 3n3
- C12, C19, C20, C22, C29, C31, C8: value 100nF -> 100n
- C13, C14, C16: value 1uF -> 1u
- C15: value 10uF -> 10u
- C17: value 220pF -> 220p
- C18: value 5.1nF -> 5n1
- C21, C23: value 33pF -> 33p
- C33: value 100uF -> 100u
- J7: renamed from J2; Manufactaurer Part Number USB4216-03-A -> (none); Manufacturer Part Number (none) -> USB4216-03-A
- R10: value 1.1k -> 1k1
- R11: value 10k -> 5k3; DigiKey Link https://www.digikey.com/short/tv9hzj27 -> https://www.digikey.com/short/4ddtfdt4; DigiKey Part Number P10KDBCT-ND -> 541-4550-1-ND; DigiKey Price per Unit 0.10 -> 0.23; Manufactaurer Part Number CRCW0603220KFKEA -> (none); Manufacturer Part Number (none) -> TNPW06035K30BEEA; Manufacturer_Part_Number ERA-3AEB103V -> (none); Mouser Link https://mou.sr/4g4GMTT -> https://mou.sr/4nmPpgC; Mouser Part Number 667-ERA-3AEB103V -> 71-TNPW06035K30BEEA; Mouser Price per Unit 0.10 -> 0.23
- R12: value 10k -> 30k1; DigiKey Link https://www.digikey.com/short/tv9hzj27 -> https://www.digikey.com/short/w02rpcr5; DigiKey Part Number P10KDBCT-ND -> 13-AT0603FRE0730K1LCT-ND; Manufactaurer Part Number CRCW0603220KFKEA -> (none); Manufacturer Part Number (none) -> AT0603FRE0730K1L; Manufacturer_Part_Number ERA-3AEB103V -> (none); Mouser Link https://mou.sr/4g4GMTT -> https://mou.sr/4mTSEfI; Mouser Part Number 667-ERA-3AEB103V -> 603-AT0603FRE0730K1L
- R13: value 90k -> 137k; DigiKey Link https://www.digikey.com/short/8bphhvq7 -> https://www.digikey.com/short/8hf2ffh2; DigiKey Part Number YAG1747CT-ND -> 311-137KHRCT-ND; DigiKey Price per Unit 0.11 -> 0.10; Manufactaurer Part Number CRCW0603220KFKEA -> (none); Manufacturer Part Number (none) -> RC0603FR-07137KL; Manufacturer_Part_Number RT0603BRD0790K9L -> (none); Mouser Link https://mou.sr/3MG2Zid -> https://mou.sr/4ppspPZ; Mouser Part Number 603-RT0603BRD0790K9L -> 603-RC0603FR-07137KL; Mouser Price per Unit 0.11 -> 0.10
- R14: value 422 -> 100k; DigiKey Link https://www.digikey.com/short/h1d7mb49 -> https://www.digikey.com/short/fm0tww77; DigiKey Part Number P422DBCT-ND -> 311-100KLECT-ND; Manufactaurer Part Number CRCW0603220KFKEA -> (none); Manufacturer Part Number (none) -> AC0603JR-07100KL; Manufacturer_Part_Number ERA-3AEB4220V -> (none); Mouser Link https://mou.sr/3L0MRap -> https://mou.sr/42xldY2; Mouser Part Number 667-ERA-3AEB4220V -> 603-AC0603JR-07100KL
- R2: value 1.54k -> 1k54
- R3: value 7.15k -> 7k15
- R8: value 422 -> 422R
Connections:
- net AFE: no longer C10.1, C12.1, C13.1, C3.1, C4.1, C6.1, C7.1, C9.1, Q1.5 (D), Q1.6 (D), Q1.7 (D), Q1.8 (D), Q1.9 (D), Q4.5 (D), Q4.6 (D), Q4.7 (D), Q4.8 (D), Q4.9 (D), U2.5 (VIN_1), U2.6 (VIN_2), U3.1 (VDD)
- net GND: now also C11.1, C15.1, C34.2, C35.2, C36.2, C37.2, C38.2, C39.2, C40.2, C41.2, C42.2, C43.2, C44.2, C45.2, C46.2, C47.2, C48.2, C49.2, C50.2, C51.2, C52.2, C53.2, C54.1, C55.1, C56.1, C57.1, C58.2, C59.2, C60.2, C61.2, C62.1, C65.2, C66.2, C67.2, C68.2, C69.2, C70.2, C71.2, C72.2, C73.2, C74.2, C75.2, C77.2, C78.2, C79.2, C80.2, C81.2, C82.2, C83.2, C84.2, C85.2, C86.2, C87.2, D1.2 (A2), D2.2 (A2), J13.1 (Pin_1), J14.2 (1.2), J14.4 (2.2), J16.1 (Pin_1), J19.2, J19.4, J19.6, J19.8, J2.2, J2.4, J2.6, J21.2, J21.4, J21.6, NT1.1, R15.1, R16.1, R17.1, R18.1, U4.4 (VSS), U5.10 (~{I2CT_IRQ}), U5.11 (GND_1), U5.12 (GND_2), U5.13 (GPIO11), U5.14 (GND_3), U5.18 (~{I2CC_IRQ}), U5.19 (GPIO3), U5.3 (ADCIN2), U5.31 (GND_4), U5.36 (GPIO7), U5.37 (GPIO6), U5.39 (GND_5), U5.5 (GPIO0), U5.6 (GPIO1), U5.7 (GPIO2), U6.1 (GND), U6.2 (GND), U6.3 (GND), U6.7 (GND), U7.27 (GND); no longer C11.2, C15.2, R13.2
- net P3V3_BUCK: now also C60.1, C61.1, J19.1, J19.3, J19.5, J19.7, J2.1, J2.3, J2.5, U5.38 (VIN_3V3)
- net P5V0_BUCK: now also C53.1, C58.1, C59.1, J21.1, J21.3, J21.5, U5.34 (PP5V), U5.35 (PP5V)
- net SYSTEM_VOLTAGE: no longer C1.1, C2.1, C5.1, C8.1, U1.5 (VIN_1), U1.6 (VIN_2)
- net 5V0_FB: now reaches C23.2, R6.2, R7.1, U2.2 (FB)
- net at R11.1: now also R13.1, C62.2, U7.5 (REGN); no longer J7.A5 (CC1)
- net 6V0_LDRV: now reaches Q2.4 (G), Q3.4 (G), R3.1, U3.9 (LDRV/_OC)
- net 6V0_FB: now reaches C17.2, C32.2, R10.1, R2.2, R9.2, U3.5 (FB)
- net 3V3_FB: now reaches C21.2, R4.2, R5.1, U1.2 (FB)
- net at R14.1: now also R13.2, U7.17 (ILIM_HIZ); no longer R13.1
- net BB_TS: now reaches R12.1
- net BB_TS: now also R11.2, TH1.2, U7.16 (TS_1), U7.32 (TS_2); no longer J7.B5 (CC2)
- net at R1.1: now also C15.2, U3.10 (BP); no longer U3.3 (PGOOD)
- net at U3.2 (EN/SS): now also C11.2; no longer C11.1
- net 6V0_HDRV: now reaches Q1.4 (G), Q4.4 (G), U3.7 (HDRV)
- net USBC_P: now reaches J7.A6 (DP1)
- net USBC_P: now also J7.B6 (DP2), D1.1 (A1), U5.26 (GPIO4/USB_P/LD1)
- net USBC_N: now reaches J7.A7 (DN1)
- net USBC_N: now also J7.B7 (DN2), D2.1 (A1), U5.27 (GPIO5/USB_N/LD2)
- net 3V3 BST renamed 3V3_BST
- net 3V3 SW renamed 3V3_SW
- net 5V0 BST renamed 5V0_BST
- net 5V0 SW renamed 5V0_SW
- net 6V0 SW renamed 6V0_SW
- removed net USBC VBUS: J7.A4 (VBUS_1), J7.B4 (VBUS_2), R11.2, R12.2, R14.2
- new net: C54.2, C55.2, C56.2, C57.2, FB1.1, J7.A4 (VBUS_1), J7.B4 (VBUS_2), U6.4 (IN), U6.5 (IN), U6.6 (IN)
- new net: R18.2, U4.7 (WP)
- new net: C39.1, C40.1, C41.1, U5.4 (LDO_1V5)
- new net: D3.2, R23.2
- new net: C65.1, C66.1, C67.1, C68.1, C69.1, U7.29 (PMID)
- new net: R25.1, U7.18 (BATP)
- new net: R24.1, U7.20 (PROG)
- new net: R17.2, U4.3 (A2)
- new net: R1.2, U3.3 (PGOOD)
- new net: R16.2, U4.2 (A1)
- new net: R21.2, U5.2 (ADCIN1)
- new net: J16.3 (Pin_3), U5.8 (I2CT_SDA)
- new net: J16.2 (Pin_2), U5.9 (I2CT_SCL)
- new net: R15.2, U4.1 (A0)
- new net BB_BTST1: C63.2, U7.4 (BTST1)
- new net BB_BTST2: C64.2, U7.19 (BTST2)
- new net BB_SDRV: C76.1, U7.24 (SDRV_1), U7.33 (SDRV_2)
- new net BB_STAT: D3.1, R22.1, U7.1 (STAT_1), U7.30 (STAT_2)
- new net BB_SW1: C63.1, L4.1, U7.28 (SW1)
- new net BB_SW2: C64.1, L4.2, U7.26 (SW2)
- new net BQ25798_GNDA: C76.2, NT1.2, R12.2, R14.2, R24.2, TH1.1, U7.10 (ACDRV2), U7.11 (ACDRV1), U7.13 (~{CE})
- new net C_CC1: C51.1, J7.A5 (CC1), U5.28 (CC1)
- new net C_CC2: C52.1, J7.B5 (CC2), U5.29 (CC2)
- new net PACK+: C77.1, C78.1, C79.1, C80.1, J14.1 (1.1), J14.3 (2.1), R25.2, U7.22 (BAT_1), U7.23 (BAT_2)
- new net SYS_VOLTAGE: C1.1, C10.1, C12.1, C13.1, C2.1, C3.1, C4.1, C5.1, C6.1, C7.1, C8.1, C81.1, C82.1, C83.1, C84.1, C85.1, C86.1, C87.1, C9.1, Q1.5 (D), Q1.6 (D), Q1.7 (D), Q1.8 (D), Q1.9 (D), Q4.5 (D), Q4.6 (D), Q4.7 (D), Q4.8 (D), Q4.9 (D), U1.5 (VIN_1), U1.6 (VIN_2), U2.5 (VIN_1), U2.6 (VIN_2), U3.1 (VDD), U7.25 (SYS)
- new net USBC_DRAIN: U5.15 (DRAIN_1), U5.30 (DRAIN_2), U5.40 (DRAIN_3)
- new net USBC_LDO_3V3: C34.1, C35.1, C36.1, C37.1, C38.1, J16.4 (Pin_4), R19.2, R20.2, R21.1, R22.2, R23.1, U4.8 (VCC), U5.1 (LDO_3V3)
- new net USBC_PPHV: C42.1, C43.1, C44.1, C45.1, C46.1, C47.1, C70.1, C71.1, C72.1, C73.1, C74.1, C75.1, U5.20 (PPHV), U5.21 (PPHV), U5.22 (PPHV), U7.2 (VBUS_1), U7.3 (VBUS_2), U7.31 (VAC1_2), U7.8 (VAC2), U7.9 (VAC1_1)
- new net USBC_SCL: J13.2 (Pin_2), R20.1, U4.6 (SCL), U5.17 (I2CC_SCL), U7.14 (SCL)
- new net USBC_SDA: J13.3 (Pin_3), R19.1, U4.5 (SDA), U5.16 (I2CC_SDA), U7.15 (SDA)
- new net USBC_VBUS: C48.1, C49.1, C50.1, FB1.2, U5.23 (VBUS_IN), U5.24 (VBUS_IN), U5.25 (VBUS_IN), U5.32 (VBUS), U5.33 (VBUS)
- no-connect marks 4 -> 10
Other:
- note added: ""can be used to directly program the TPS25751, and program the BQ25798 through the host microcontroller " ^^^^ for the I2Ct lines (pins 8, 9)"
- note added: "*** THIS IS 5 to 20V output of this ***"
- note added: "1010 ???? GND=0 so this: 1010 0000 -> 0x50 which is what we need for our PD controller"
- note added: "3V3 Buck"
- note added: "512Kb"
- note added: "5V0 Buck"
- note added: "6V0 Buck"
- note added: "ADCIN1 & ADCIN2 configured for "SafeMode" I2C Target is 0x20"
- note added: "Buck-Boost Battery Charger"
- note added: "D+/- Handled on TPS25751DREFR"
- note added: "EEPROM"
- note added: "Flash this with the bin taken from TI's website. Use I2C to USB adapter. Flash this when the system is off (not powered), only flash/power this."
- note added: "Max Power Sourced = 45W, Sink Power = 60W"
- note added: "PACK+"
- note added: "R = (3.3-2)/20ma = 65 Ohms"
- note added: "TPS25751DREFR will load from EEPROM"
- note added: "To MCU (3V3 Buck)"
- note added: "To MCU (5V0 Buck)"
- note added: "To Motor Driver (3V3 Buck)"
- note added: "USB-C"
- note added: "USB-C PD Controller"
- note added: "VSYS caps need 2A ripple support"
- note added: "internal debugging"
- note added: "pins 15&30 tie to exposed pad 40 for internal fet"
- note removed: "3.3V Buck"
- note removed: "5V Buck"
- note removed: "5V/5A Fsw=600kHz L=2u2H Ic(RMS1) = 2A D = Vout/Vin = 5/12.6 = 0.397 D = Vout/Vin = 5/9.6 = 0.521 Using 9.6V since its closer to 50% duty I_Ripple = (Vout(1 - Vout/Vin))/(L*f) ; use larger Vin I_In = Iout * (Vout/Vin) Ic(RMS) = Iout * SQRT[(Vout/Vin)(1-(Vout/Vin))] Ic(RMS)tot = SQRT[Ic(RMS1)^2 + Ic(RMS2)^2] I_Ripple = 2.285A I_In = 2.6A Ic(RMS2) = 2.497A Ic(RMS)tot = 3.2A -> 3.8A 1, find cap bank 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"
- note removed: "6V 24A"
- note removed: "6V Buck"
- note removed: "6V/20A L=440nH f=1.2MHz Vin=[9.6,12.6] D = Vout/Vin = 6/12.6 = 0.476 ; use for worst-case input ripple I_Ripple = (Vout(1 - Vout/Vin))/(L*f) ; use larger Vin I_In = Iout * (Vout/Vin) ; use smaller Vin for max current Ic(RMS,in) = Iout * SQRT[D*(1-D)] Ic(RMS,out) = I_Ripple / (2*sqrt(3)) I_Ripple = 5.95A I_In = 12.5A Ic(RMS,in) = 9.99A -> 12A Ic(RMS,out) = 1.72A -> 2.1A 1, Input cap bank > 12A rms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"
- note removed: "For Voltage: R5= (.6V * R4) / (6 - .6V)"
- note removed: "For a triangular wave from the inductor, the formula is Ic(RMS) = I_Ripple / (2*sqrt(3)). Ic(RMS,out) = 2.285A / 3.464 = 0.66A -> 0.8A"
- note removed: "Iin = Vout * Iout / Vin * n"
- note removed: "Might need to double the fets, that is what we bench says"
- note removed: "ROCSET = ( (IOUT_max - (IP_P / 2)) * RDS_on - VOCLOS ) / ( 2 * IOCSET ) Iout max target current IP induct ripple current rds on res low side mosfet voclos offset voltage = -8mv iocset internal current = 9.5microamps"
- note removed: "V_OC = (R_OCSET * 2 * I_OCSET_min) + V_OCLOS_min V_OC = (7.68 kΩ * 2 * 9.5 µA) + (-8 mV) V_OC = 137.9 mV I_valley = V_OC / R_DS(on) I_valley = 137.9 mV / 7.8 mΩ I_valley = 17.68 A I_SCP = I_valley + (I_RIPPLE / 2) I_SCP = 17.68 A + (5.95 A / 2) I_SCP = 20.66 A"
- note removed: "inductor = (vinmax -vout)/(.3*Iout) * (Vout/Vinmax) * (1/Fsw)"
- note removed: "might need to change inductor"
- moved on the sheet: C1, C10, C11, C12, C13, C14, C15, C16, C17, C18, C19, C2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

Commit message: Rename STAR_BUS to STAR_BMS (Battery Management System)
File Renames:
- STAR_BUS.kicad_sch → STAR_BMS.kicad_sch
- STAR_BUS.kicad_pro → STAR_BMS.kicad_pro
- STAR_BUS.kicad_pcb → STAR_BMS.kicad_pcb
- STAR_BUS.kicad_prl → STAR_BMS.kicad_prl (not tracked)
- STAR_BUS-backups/ → STAR_BMS-backups/

Internal Reference Updates:
- Updated all "STAR_BUS" references to "STAR_BMS" in project files
- Updated cross-references in STAR_MOTOR_DRIVER and STAR_POWER_BOARD

Corrects naming to properly reflect Battery Management System (BMS)
instead of BUS.
Parts:
- removed J10, J11, J3, J4, J5, J6, J9: 1017491, 1017491, symbol 1017491:1017491
- removed J12: Conn_02x03_Counter_Clockwise, Connector_PinHeader_2.54mm:PinHeader_2x03_P2.54mm_Vertical, symbol Connector_Generic:Conn_02x03_Counter_Clockwise
- J1: DigiKey Link https://www.digikey.com/short/nbbz5wdw -> https://www.digikey.com/short/297znmhj; DigiKey Part Number 277-17493-ND -> 277-17493-ND; Manufacturer Part Number (none) -> 1017491; Mouser Link https://mou.sr/44CGuAW -> https://mou.sr/4pNdQFk
Connections:
- net SYSTEM_VOLTAGE is gone; now on net GND: J1.3 (2.1), J1.4 (2.2)
- net GND: now also J14.1 (1.1); no longer J1.1 (1.1), J1.2 (1.2), J14.4 (2.2)
- net P6V0_BUCK: now also J1.1 (1.1), J1.2 (1.2)
- net PACK+: now also J14.4 (2.2); no longer J14.1 (1.1)
Other:
- note added: "To Motor Driver (6V0 Buck)"
- note removed: "Microcontroller"
- note removed: "Motor Driver"
- note removed: "USBC"
- moved on the sheet: J14, J19, J2, J21

Commit message: Add CAPC7866X950N footprint library and fix schematic reference
- Register CAPC7866X950N footprint library in fp-lib-table
- Update STAR_POWER_BOARD schematic to use library-prefixed footprint reference
- Fixes missing footprint issue for 100uF capacitor in power board design
Parts:
- removed C34, C38, C41, C47, C48, C53, C60, C65, C75, C80, C84: 100n, Capacitor_SMD:C_0603_1608Metric_Pad1.08x0.95mm_HandSolder, symbol Device:C
- removed C35: 1u, Capacitor_SMD:C_0603_1608Metric_Pad1.08x0.95mm_HandSolder, symbol Device:C
- removed C36, C37, C39, C40, C42, C43, C44, C45, C46, C58, C61, C66, C67, C68, C69, C70, C71, C72, C73, C74, C77, C78, C79, C81, C82, C83: 10u, Capacitor_SMD:C_0805_2012Metric_Pad1.18x1.45mm_HandSolder, symbol Device:C
- removed C49, C50, C62: 4u7, Capacitor_SMD:C_0805_2012Metric_Pad1.18x1.45mm_HandSolder, symbol Device:C
- removed C51, C52: 330p, Capacitor_SMD:C_0603_1608Metric_Pad1.08x0.95mm_HandSolder, symbol Device:C
- removed C54, C55, C56, C57: 10n, Capacitor_SMD:C_0603_1608Metric_Pad1.08x0.95mm_HandSolder, symbol Device:C
- removed C59, C85, C86, C87: 22u, T527T226M025ATE100:CAPPM3528X120N, symbol Device:C_Polarized
- removed C63, C64: 47n, Capacitor_SMD:C_0603_1608Metric_Pad1.08x0.95mm_HandSolder, symbol Device:C
- removed C76: 1n, Capacitor_SMD:C_0603_1608Metric_Pad1.08x0.95mm_HandSolder, symbol Device:C
- removed D1, D2: 82306050029, 82306050029:WESURGE_0603134, symbol 82306050029:82306050029
- removed D3: RED, SML-D12Y1WT86:LEDC1608X55N, symbol PCM_SL_Devices:LED
- removed FB1: 22R, Resistor_SMD:R_0603_1608Metric_Pad0.98x0.95mm_HandSolder, symbol Device:FerriteBead_Small
- removed J13: PD_DBG, Connector_PinHeader_2.54mm:PinHeader_1x03_P2.54mm_Vertical, symbol Connector_Generic:Conn_01x03
- removed J16: PD_I2C, Connector_PinHeader_2.54mm:PinHeader_1x04_P2.54mm_Vertical, symbol Connector_Generic:Conn_01x04
- removed J7: USB4216-03-A, USB421603A, symbol USB4216-03-A:USB4216-03-A
- removed L4: VLS6045EX-1R0N, VLS6045EX-1R0N:VLS6045, symbol VLS6045EX-1R0N:VLS6045EX-1R0N
- removed NT1: NetTie_2, NetTie:NetTie-2_SMD_Pad0.5mm, symbol Device:NetTie_2
- removed R11: 5k3, Resistor_SMD:R_0603_1608Metric_Pad0.98x0.95mm_HandSolder, symbol Device:R
- removed R12: 30k1, Resistor_SMD:R_0603_1608Metric_Pad0.98x0.95mm_HandSolder, symbol Device:R
- removed R13: 137k, Resistor_SMD:R_0603_1608Metric_Pad0.98x0.95mm_HandSolder, symbol Device:R
- removed R14, R21: 100k, Resistor_SMD:R_0603_1608Metric_Pad0.98x0.95mm_HandSolder, symbol Device:R
- removed R15, R16, R17, R18, R22: 10k, Resistor_SMD:R_0603_1608Metric_Pad0.98x0.95mm_HandSolder, symbol Device:R
- removed R19, R20: 3k3, Resistor_SMD:R_0603_1608Metric_Pad0.98x0.95mm_HandSolder, symbol Device:R
- removed R23: 68R, Resistor_SMD:R_0603_1608Metric_Pad0.98x0.95mm_HandSolder, symbol Device:R
- removed R24: 10k5, Resistor_SMD:R_0603_1608Metric_Pad0.98x0.95mm_HandSolder, symbol Device:R
- removed R25: 100R, Resistor_SMD:R_0603_1608Metric_Pad0.98x0.95mm_HandSolder, symbol Device:R
- removed TH1: NTCGS163JX103DT7, NTCGS163JX103DT7:THRMC1608X90N, symbol NTCGS163JX103DT7:NTCGS163JX103DT7
- removed U4: CAT24C512WI-GT3, CAT24C512WI-GT3:SOIC127P600X175-8N, symbol CAT24C512WI:CAT24C512WI-GT3
- removed U5: TPS25751DREFR, TPS25751DREFR:TPS25751DREFR, symbol TPS25751DREFR:TPS25751DREFR
- removed U6: TVS2200DRV, TVS2200DRVR:SON65P200X200X80-7N, symbol Power_Protection:TVS2200DRV
- removed U7: BQ25798RQMR, BQ25798RQMR:BQ25798RQMR, symbol BQ25798RQMR:BQ25798RQMR
- C33: footprint CAPC7866X950N -> CAPC7866X950N:CAPC7866X950N
Connections:
- net PACK+ is gone; now on net SYS_VOLTAGE: J14.3 (2.1), J14.4 (2.2)
- no-connect marks 10 -> 4
Other:
- note added: "SYS"
- note removed: ""can be used to directly program the TPS25751, and program the BQ25798 through the host microcontroller " ^^^^ for the I2Ct lines (pins 8, 9)"
- note removed: "*** THIS IS 5 to 20V output of this ***"
- note removed: "1010 ???? GND=0 so this: 1010 0000 -> 0x50 which is what we need for our PD controller"
- note removed: "512Kb"
- note removed: "ADCIN1 & ADCIN2 configured for "SafeMode" I2C Target is 0x20"
- note removed: "Buck-Boost Battery Charger"
- note removed: "D+/- Handled on TPS25751DREFR"
- note removed: "EEPROM"
- note removed: "Flash this with the bin taken from TI's website. Use I2C to USB adapter. Flash this when the system is off (not powered), only flash/power this."
- note removed: "Max Power Sourced = 45W, Sink Power = 60W"
- note removed: "PACK+"
- note removed: "R = (3.3-2)/20ma = 65 Ohms"
- note removed: "TPS25751DREFR will load from EEPROM"
- note removed: "USB-C"
- note removed: "USB-C PD Controller"
- note removed: "VSYS caps need 2A ripple support"
- note removed: "internal debugging"
- note removed: "pins 15&30 tie to exposed pad 40 for internal fet"
- moved on the sheet: C1, C10, C11, C12, C13, C14, C15, C16, C17, C18, C19, C2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
