File: schematic/EV2300_Replacement.kicad_pcb (KiCad board)
At the start: 2 copper layers, 133 parts, among them J1 USB4216-03-A, J2 22053041, J3 22053041, J4 USB4216-03-A, J5 E1E2-Emulator-Interface, J6 EMU CFG, J7 UPSEL_CFG, SW1 OP_CFG, U1 TVS2200DRV, U2 TVS2200DRV, U3 LDL1117S33R, U4 CY7C65213A-28PVXI, U5 TPS2116DRLR, U6 R5F572NNHGFP-30, Y1 ECS-240-8-30B-CKM-TR

Commit message: EV2300
Parts:
- added J10: Conn_01x02, Connector_PinHeader_2.54mm:PinHeader_1x02_P2.54mm_Vertical, F.Cu at (155.1, 107.3)
- added J11: Conn_01x02, Connector_PinHeader_2.54mm:PinHeader_1x02_P2.54mm_Vertical, F.Cu at (159.7, 107.3)
- added J8: Conn_01x02, Connector_PinHeader_2.54mm:PinHeader_1x02_P2.54mm_Vertical, F.Cu at (145.9, 107.3)
- added J9: Conn_01x02, Connector_PinHeader_2.54mm:PinHeader_1x02_P2.54mm_Vertical, F.Cu at (150.5, 107.3)
- added R38: 4k7, Resistor_SMD:R_0603_1608Metric_Pad0.98x0.95mm_HandSolder, F.Cu at (141.5, 71.8)
- added R39: 4k7, Resistor_SMD:R_0603_1608Metric_Pad0.98x0.95mm_HandSolder, F.Cu at (141.5, 74.3)
- moved SW1 70.5 mm to (161.8, 76.1)
- moved Y1 63.8 mm to (171.9, 81.6)
- moved D1 59.8 mm to (170.5, 67.4)
- moved D4 59.8 mm to (170.5, 76.7)
- moved D2 59.8 mm to (170.5, 70.5)
- moved D3 59.8 mm to (170.5, 73.6)
- moved U5 53.0 mm to (161.1, 81.4)
- moved D5 46.9 mm to (169.3, 106.2)
- moved D6 46.9 mm to (169.3, 109.6)
- moved J6 39.8 mm to (125.9, 103.7)
- moved J7 39.8 mm to (130.5, 103.7)
- moved U4 35.0 mm to (118.4, 107.4)
- moved D7 30.8 mm to (174.4, 106.0)
- moved D8 30.8 mm to (174.4, 108.9)
- moved J1 27.6 mm to (151.1, 71.3)
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Connections:
- R30 pad 1: /RX72N_PIN_34 -> Net-(J8-Pin_1)
- R31 pad 1: /RX72N_PIN_33 -> Net-(J9-Pin_1)
- R33 pad 1: /RX72N_PIN_33 -> /BMS_SMBUS_DATA
- R33 pad 2: /BMS_SMBUS_DATA -> Net-(U6-P13/TXD2)
- R34 pad 1: /RX72N_PIN_34 -> /BMS_SMBUS_CLK
- R34 pad 2: /BMS_SMBUS_CLK -> Net-(U6-P12/RXD2)
- U6 pad 33: /BMS_SMBUS_DATA -> Net-(U6-P13/TXD2)
- U6 pad 34: /BMS_SMBUS_CLK -> Net-(U6-P12/RXD2)
