File: schematic/EV2300_Replacement.kicad_sch (KiCad schematic)
At the start: 139 parts, among them J1 USB4216-03-A, J10 Conn_01x02, J11 Conn_01x02, J2 22053041, J3 22053041, J4 USB4216-03-A, J5 E1E2-Emulator-Interface, J6 EMU CFG, J7 UPSEL_CFG, J8 Conn_01x02, J9 Conn_01x02, SW1 OP_CFG, U1 TVS2200DRV, U2 TVS2200DRV, U3 LDL1117S33R, U4 CY7C65213A-28PVXI, U5 TPS2116DRLR, U6 R5F572NNHGFP-30, Y1 ECS-240-8-30B-CKM-TR

Commit message: publish branch
Parts:
- added TP1, TP10, TP11, TP12, TP13, TP14, TP15, TP16, TP17, TP18, TP19, TP2, TP20, TP21, TP22, TP23, TP24, TP25, TP26, TP27, TP28, TP29, TP3, TP30, TP31, TP32, TP33, TP34, TP35, TP36, TP37, TP38, TP39, TP4, TP40, TP41, TP42, TP43, TP44, TP45, TP46, TP47, TP48, TP49, TP5, TP50, TP51, TP52, TP53, TP54, TP55, TP56, TP57, TP58, TP59, TP6, TP60, TP61, TP62, TP63, TP64, TP65, TP66, TP67, TP68, TP69, TP7, TP70, TP71, TP72, TP73, TP74, TP8, TP9: 3825, 3825, symbol 3825:3825
Connections:
- net BOARD_3V3: now also TP1.1, TP2.1
- net EMU_TDI_RXD: now also TP4.1
- net EMU_TDO_TXD: now also TP5.1
- net GND: now also TP72.1, TP73.1, TP74.1
- net PMOD_JC_SCL: now also TP27.1
- net PMOD_JC_SDA: now also TP26.1
- net RX72N_PIN_100: now reaches U6.100 (P05)
- net RX72N_PIN_100: now also TP71.1
- net RX72N_PIN_18: now reaches U6.18 (P32)
- net RX72N_PIN_18: now also TP3.1
- net RX72N_PIN_23: now reaches U6.23 (P25)
- net RX72N_PIN_23: now also TP6.1
- net RX72N_PIN_24: now reaches U6.24 (P24)
- net RX72N_PIN_24: now also TP7.1
- net RX72N_PIN_25: now reaches U6.25 (P23)
- net RX72N_PIN_25: now also TP8.1
- net RX72N_PIN_26: now reaches U6.26 (P22)
- net RX72N_PIN_26: now also TP9.1
- net RX72N_PIN_27: now reaches U6.27 (P21)
- net RX72N_PIN_27: now also TP10.1
- net RX72N_PIN_28: now reaches U6.28 (P20)
- net RX72N_PIN_28: now also TP11.1
- net RX72N_PIN_29: now reaches U6.29 (P17)
- net RX72N_PIN_29: now also TP12.1
- net RX72N_PIN_31: now reaches U6.31 (P15/RXD1)
- net RX72N_PIN_31: now also TP13.1
- net RX72N_PIN_32: now reaches U6.32 (P14)
- net RX72N_PIN_32: now also TP14.1
- net RX72N_PIN_39: now reaches U6.39 (P55)
- net RX72N_PIN_39: now also TP17.1
- net RX72N_PIN_40: now reaches U6.40 (P54)
- net RX72N_PIN_40: now also TP18.1
- net RX72N_PIN_41: now reaches U6.41 (P53)
- net RX72N_PIN_41: now also TP19.1
- net RX72N_PIN_42: now reaches U6.42 (P52)
- net RX72N_PIN_42: now also TP20.1
- net RX72N_PIN_43: now reaches U6.43 (P51)
- net RX72N_PIN_43: now also TP21.1
- net RX72N_PIN_44: now reaches U6.44 (P50)
- net RX72N_PIN_44: now also TP22.1
- net RX72N_PIN_46: now reaches U6.46 (PC6)
- net RX72N_PIN_46: now also TP23.1
- net RX72N_PIN_47: now reaches U6.47 (PC5)
- net RX72N_PIN_47: now also TP24.1
- net RX72N_PIN_48: now reaches U6.48 (PC4)
- net RX72N_PIN_48: now also TP25.1
- net RX72N_PIN_51: now reaches U6.51 (PC1)
- net RX72N_PIN_51: now also TP28.1
- net RX72N_PIN_52: now reaches U6.52 (PC0)
- net RX72N_PIN_52: now also TP29.1
- net RX72N_PIN_55: now reaches U6.55 (PB5)
- net RX72N_PIN_55: now also TP32.1
- net RX72N_PIN_56: now reaches U6.56 (PB4)
- net RX72N_PIN_56: now also TP33.1
- net RX72N_PIN_57: now reaches U6.57 (PB3)
- net RX72N_PIN_57: now also TP34.1
- net RX72N_PIN_58: now reaches U6.58 (PB2)
- net RX72N_PIN_58: now also TP35.1
- net RX72N_PIN_59: now reaches U6.59 (PB1)
- net RX72N_PIN_59: now also TP36.1
- net RX72N_PIN_61: now reaches U6.61 (PB0)
- net RX72N_PIN_61: now also TP37.1
- net RX72N_PIN_63: now reaches U6.63 (PA7)
- net RX72N_PIN_63: now also TP38.1
- net RX72N_PIN_64: now reaches U6.64 (PA6)
- net RX72N_PIN_64: now also TP39.1
- net RX72N_PIN_65: now reaches U6.65 (PA5)
- net RX72N_PIN_65: now also TP40.1
- net RX72N_PIN_66: now reaches U6.66 (PA4)
- net RX72N_PIN_66: now also TP41.1
- net RX72N_PIN_67: now reaches U6.67 (PA3)
- net RX72N_PIN_67: now also TP42.1
- net RX72N_PIN_68: now reaches U6.68 (PA2)
- net RX72N_PIN_68: now also TP43.1
- net RX72N_PIN_69: now reaches U6.69 (PA1)
- net RX72N_PIN_69: now also TP44.1
- net RX72N_PIN_70: now reaches U6.70 (PA0)
- net RX72N_PIN_70: now also TP45.1
- net RX72N_PIN_71: now reaches U6.71 (PE7)
- net RX72N_PIN_71: now also TP46.1
- net RX72N_PIN_72: now reaches U6.72 (PE6)
- net RX72N_PIN_72: now also TP47.1
- net RX72N_PIN_73: now reaches U6.73 (PE5)
- net RX72N_PIN_73: now also TP48.1
- net RX72N_PIN_74: now reaches U6.74 (PE4)
- net RX72N_PIN_74: now also TP49.1
- net RX72N_PIN_75: now reaches U6.75 (PE3)
- net RX72N_PIN_75: now also TP50.1
- net RX72N_PIN_76: now reaches U6.76 (PE2)
- net RX72N_PIN_76: now also TP51.1
- net RX72N_PIN_77: now reaches U6.77 (PE1)
- net RX72N_PIN_77: now also TP52.1
- net RX72N_PIN_78: now reaches U6.78 (PE0)
- net RX72N_PIN_78: now also TP53.1
- net RX72N_PIN_79: now reaches U6.79 (PD7)
- net RX72N_PIN_79: now also TP54.1
- net RX72N_PIN_80: now reaches U6.80 (PD6)
- net RX72N_PIN_80: now also TP55.1
- net RX72N_PIN_81: now reaches U6.81 (PD5)
- net RX72N_PIN_81: now also TP56.1
- net RX72N_PIN_82: now reaches U6.82 (PD4)
- net RX72N_PIN_82: now also TP57.1
- net RX72N_PIN_83: now reaches U6.83 (PD3)
- net RX72N_PIN_83: now also TP58.1
- net RX72N_PIN_84: now reaches U6.84 (PD2)
- net RX72N_PIN_84: now also TP59.1
- net RX72N_PIN_85: now reaches U6.85 (PD1)
- net RX72N_PIN_85: now also TP60.1
- net RX72N_PIN_86: now reaches U6.86 (PD0)
- net RX72N_PIN_86: now also TP61.1
- net RX72N_PIN_87: now reaches U6.87 (P47)
- net RX72N_PIN_87: now also TP62.1
- net RX72N_PIN_88: now reaches U6.88 (P46)
- net RX72N_PIN_88: now also TP63.1
- net RX72N_PIN_89: now reaches U6.89 (P45)
- net RX72N_PIN_89: now also TP64.1
- net RX72N_PIN_90: now reaches U6.90 (P44)
- net RX72N_PIN_90: now also TP65.1
- net RX72N_PIN_91: now reaches U6.91 (P43)
- net RX72N_PIN_91: now also TP66.1
- net RX72N_PIN_92: now reaches U6.92 (P42)
- net RX72N_PIN_92: now also TP67.1
- net RX72N_PIN_93: now reaches U6.93 (P41)
- net RX72N_PIN_93: now also TP68.1
- net RX72N_PIN_95: now reaches U6.95 (P40)
- net RX72N_PIN_95: now also TP69.1
- net RX72N_PIN_98: now reaches U6.98 (P07)
- net RX72N_PIN_98: now also TP70.1
- net SCI9_RXD9 renamed RX72N_PIN_54
- net RX72N_PIN_54: now also TP31.1
- net SCI9_TXD9 renamed RX72N_PIN_53
- net RX72N_PIN_53: now also TP30.1
- new net RX72N_PIN_33: TP15.1
- new net RX72N_PIN_34: TP16.1
- no-connect marks 78 -> 16
Other:
- note added: "Test Points"
- moved on the sheet: C1, C10, C11, C12, C13, C14, C15, C16, C17, C18, C19, C2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
