File: schematic/STAR_POWER_BOARD.kicad_pcb (KiCad board)
At the start: 4 copper layers, 96.2 x 92.9 mm, 67 parts, among them J1 Screw_Terminal_01x02, J2 1017491, J3 USB4216-03-A, J4 Screw_Terminal_01x02, J5 Screw_Terminal_01x02, J6 1017491, J7 1017491, Q1 CSD18540Q5B, Q2 CSD17577Q3A, Q3 CSD17577Q3A, Q4 CSD18540Q5B, Q5 SSM6J507NU-LF, U1 TPS566238PRQFR, U2 TPS566238PRQFR, U3 TPS40305DRCT

Commit message: initial push
initial push
Parts:
- removed C1, C4, C7: 47u, Capacitor_SMD:C_1210_3225Metric_Pad1.33x2.70mm_HandSolder
- removed C10: 1u, Capacitor_SMD:C_0603_1608Metric_Pad1.08x0.95mm_HandSolder
- removed C13: 10u, Capacitor_SMD:C_0603_1608Metric_Pad1.08x0.95mm_HandSolder
- removed C15: 220p, Capacitor_SMD:C_0603_1608Metric_Pad1.08x0.95mm_HandSolder
- removed C17: 5n1, Capacitor_SMD:C_0603_1608Metric_Pad1.08x0.95mm_HandSolder
- removed C18: 3n3, Capacitor_SMD:C_0603_1608Metric_Pad1.08x0.95mm_HandSolder
- removed C21: 100n, Capacitor_SMD:C_0603_1608Metric_Pad1.08x0.95mm_HandSolder
- removed C28: 820p, Capacitor_SMD:C_0603_1608Metric_Pad1.08x0.95mm_HandSolder
- removed C33: 100u, CAPC7866X950N:CAPC7866X950N
- removed J1: Screw_Terminal_01x02, 282837_2:TE_282837-2
- removed J2, J6, J7: 1017491, 1017491:1017491
- removed L3: SRP1038A-R36M, INDPM110100X400N:INDPM110100X400N
- removed Q1, Q4: CSD18540Q5B, DNK0008A:DNK0008A
- removed Q2, Q3: CSD17577Q3A, Q3A:Q3A
- removed R1: 100k, Resistor_SMD:R_0603_1608Metric_Pad0.98x0.95mm_HandSolder
- removed R10: 1k1, Resistor_SMD:R_0603_1608Metric_Pad0.98x0.95mm_HandSolder
- removed R2: 1k54, Resistor_SMD:R_0603_1608Metric_Pad0.98x0.95mm_HandSolder
- removed R3: 7k15, Resistor_SMD:R_0603_1608Metric_Pad0.98x0.95mm_HandSolder
- removed R8: 422R, Resistor_SMD:R_0603_1608Metric_Pad0.98x0.95mm_HandSolder
- removed R9: 10k, Resistor_SMD:R_0603_1608Metric_Pad0.98x0.95mm_HandSolder
- removed U3: TPS40305DRCT, TPS40305DRCT:TPS40305DRCT
Routing:
- net /6V0_FB: track 15.3 -> 0.00 mm
- net Net-(U3-BP): track 8.85 -> 0.00 mm
- net /6V0_LDRV: track 43.2 -> 36.6 mm, vias 3 -> 0
- net Net-(U3-COMP): track 6.07 -> 0.00 mm
- net /6V0_SW: track 18.1 -> 13.7 mm, vias 40 -> 0
- net GND: track 22.9 -> 18.7 mm, vias 152 -> 112
- net /FUSE+: track 7.12 -> 2.97 mm, vias 101 -> 46
- net Net-(U3-PGOOD): track 17.8 -> 13.7 mm, vias 2 -> 0
- net /6V0_HDRV: track 39.1 -> 35.5 mm, vias 3 -> 0
- net Net-(U3-EN/SS): track 3.60 -> 0.00 mm
- net Net-(U3-BOOT): track 3.25 -> 0.00 mm
- net Net-(C28-Pad1): track 2.88 -> 0.00 mm
- net Net-(C17-Pad2): track 2.46 -> 0.00 mm
- net /P6V0_BUCK: track 0.51 -> 0.00 mm, vias 72 -> 0
- net /SWITCH_OUT: vias 16 -> 0
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- removed copper zone on F.Cu, net /6V0_SW
- removed copper zone on In2.Cu, net /6V0_SW
- removed copper zone on F.Cu, net /P6V0_BUCK
- removed copper zone on In2.Cu, net /P6V0_BUCK
- removed copper zone on F.Cu, net /PACK+
- removed copper zone on In2.Cu, net /PACK+
- removed copper zone on F.Cu, net /SWITCH_OUT
- removed copper zone on In2.Cu, net /SWITCH_OUT
- removed copper zone on In2.Cu, net GND
Other:
- board size 96.2 x 92.9 mm -> 96.2 x 61.1 mm
- board text removed: "6V"
- board text removed: "6V ↑"
- board text removed: "FUSE"
- board text removed: "PACK+"
- board text removed: "SWITCH"
