Commit message: fix(geometry): update wheel radius for goBILDA Wasteland 144mm wheels
The chassis is being rebuilt with goBILDA Wasteland wheels (part
3616-0014-0144, 144 mm diameter) per the current PO. New radius is
0.072 m, replacing the old 0.0325 m DFRobot 65 mm wheel constant.

Updated everywhere it was hardcoded so producers and consumers agree:

- star-beaglebone-blue/src/inc/hardware_config.h: BBB telemetry
  velocity computation constant.
- star-ros2/.../star_gateway_bridge_node.{cpp,hpp}: ROS2 parameter
  default + doc comment.
- star-ros2/.../message_converter.hpp: BbbParams struct example
  comments and the in-class default initializer used as a fallback
  before init_bbb_params() runs.
- star-ros2/.../star_simulation/urdf/star_gazebo.xacro: Gazebo
  DiffDrive plugin wheel_radius.
- star-ros2/.../star_simulation/urdf/star_sim.urdf.xacro: xacro
  property + spec comment.
- star-ros2/.../star_bringup/launch/slam.launch.py: SLAM bringup
  parameter override.
- star-ros2/.../star_spi_bridge/src/star_spi_driver_node.cpp: SPI
  bridge parameter default.
- star-ros2/.../star_spi_bridge/launch/star_spi_bridge.launch.py:
  SPI bridge launch parameter override.
- star-ros2/.../star_spi_bridge/test/test_spi_message_converter.cpp:
  test fixture parameters AND the literal expected values in the
  assertions (one revolution distance, angular = linear/radius).

Miter gears in the new gear stage (goBILDA 2320-1006-0024 +
2320-4008-0024) are 24-tooth 1:1, so ticks_per_rev (11599 = 341 PPR
* 34.02:1 motor gearbox) is unchanged.

Not touched, but flagged TODO in star_sim.urdf.xacro: chassis
dimensions (0.20 x 0.15 x 0.08 m), track width (0.150 m), and
wheelbase (0.120 m) are still sized for the DFRobot platform. The
new build uses 312 mm U-channels and the geometry needs measuring
on the assembled chassis -- not changed here because the right
values aren't known yet.

File: star-ros2/src/star_simulation/urdf/star_gazebo.xacro (robot description, xacro)
@@ -18,5 +18,5 @@
       <right_joint>back_right_wheel_joint</right_joint>
       <wheel_separation>0.150</wheel_separation>
-      <wheel_radius>0.0325</wheel_radius>
+      <wheel_radius>0.072</wheel_radius>
       <max_linear_acceleration>1.0</max_linear_acceleration>
       <min_linear_acceleration>-1.0</min_linear_acceleration>

File: star-ros2/src/star_simulation/urdf/star_sim.urdf.xacro (robot description, xacro)
@@ -9,8 +9,8 @@
     - Gazebo plugin declarations (via star_gazebo.xacro include)
   Robot specs (DFRobot FIT0520 motors, MPU-9250 IMU, RPLiDAR C1):
-    - Wheel radius: 0.0325 m
-    - Track width (wheel separation): 0.150 m
-    - Wheelbase (front-to-back): 0.120 m
-    - Chassis: 0.20 x 0.15 x 0.08 m (L x W x H)
+    - Wheel radius: 0.072 m (goBILDA Wasteland 144mm, part 3616-0014-0144)
+    - Track width (wheel separation): 0.150 m  -- TODO: update for 312mm U-channel chassis
+    - Wheelbase (front-to-back): 0.120 m       -- TODO: update for 312mm U-channel chassis
+    - Chassis: 0.20 x 0.15 x 0.08 m (L x W x H) -- TODO: update for new chassis
     - Total mass: ~2.4 kg (2.0 kg chassis + 4 x 0.1 kg wheels)
 -->
@@ -23,5 +23,5 @@
   <xacro:property name="chassis_height" value="0.08"/>
   <xacro:property name="chassis_mass" value="2.0"/>
-  <xacro:property name="wheel_radius" value="0.0325"/>
+  <xacro:property name="wheel_radius" value="0.072"/>
   <xacro:property name="wheel_width" value="0.030"/>
   <xacro:property name="wheel_mass" value="0.1"/>

Commit message: fix(geometry): set track width to 356mm and update URDF for new chassis
CAD-confirmed values from the new goBILDA Wasteland chassis build:
- Track width (axle-to-axle, left-right): 356 mm
  (304 mm inside-wheel-to-inside-wheel + 52 mm wheel width)
- Wheel base (axle-to-axle, front-to-back): 264 mm
- Chassis bounding box: 0.346 x 0.292 x 0.118 m

The ROS2 parameter named `wheel_base` in code is actually the
*track width* (used for differential-drive twist-to-wheel-velocity
conversion) -- the existing 0.150 m default was a track width from
the old DFRobot platform, not a wheelbase. Updated to 0.356 m
everywhere it is hardcoded:

- star_gateway_bridge_node.cpp: parameter default + comment.
- star_gateway_bridge_node.hpp: doc comment now correctly labels
  the parameter as track width rather than "distance between
  wheels."
- message_converter.hpp: BbbParams default initializer.
- slam.launch.py, star_spi_driver_node.cpp,
  star_spi_bridge.launch.py: launch/param defaults.
- test_spi_message_converter.cpp: test fixture.

For the Gazebo simulation URDF (star_gazebo.xacro,
star_sim.urdf.xacro), updated chassis dimensions and wheel offsets
to match the real chassis:

- chassis_length 0.20 -> 0.346, chassis_width 0.15 -> 0.292,
  chassis_height 0.08 -> 0.118 (from STAR.stl bounding box).
- wheel_width 0.030 -> 0.052 (goBILDA Wasteland spec).
- track_half 0.075 -> 0.178 (= track_width / 2).
- wheel_y_offset 0.090 -> 0.204 (= track_half + half wheel width,
  preserving the convention used by the existing URDF).
- wheel_x_offset 0.060 -> 0.132 (= 264 mm wheelbase / 2). The
  front-back offset is geometric only -- skid-steer kinematics
  do not use it.
- gazebo DiffDrive plugin wheel_separation 0.150 -> 0.356.

Updated the spec block at the top of star_sim.urdf.xacro to drop
the obsolete DFRobot/MPU-9250 reference and document the new
geometry source.

File: star-ros2/src/star_simulation/urdf/star_gazebo.xacro (robot description, xacro)
@@ -17,5 +17,5 @@
       <right_joint>front_right_wheel_joint</right_joint>
       <right_joint>back_right_wheel_joint</right_joint>
-      <wheel_separation>0.150</wheel_separation>
+      <wheel_separation>0.356</wheel_separation>
       <wheel_radius>0.072</wheel_radius>
       <max_linear_acceleration>1.0</max_linear_acceleration>

File: star-ros2/src/star_simulation/urdf/star_sim.urdf.xacro (robot description, xacro)
@@ -8,10 +8,11 @@
     - LiDAR and IMU visual geometry
     - Gazebo plugin declarations (via star_gazebo.xacro include)
-  Robot specs (DFRobot FIT0520 motors, MPU-9250 IMU, RPLiDAR C1):
+  Robot specs (goBILDA Wasteland chassis, 312mm U-channels, miter-gear drive):
     - Wheel radius: 0.072 m (goBILDA Wasteland 144mm, part 3616-0014-0144)
-    - Track width (wheel separation): 0.150 m  -- TODO: update for 312mm U-channel chassis
-    - Wheelbase (front-to-back): 0.120 m       -- TODO: update for 312mm U-channel chassis
-    - Chassis: 0.20 x 0.15 x 0.08 m (L x W x H) -- TODO: update for new chassis
-    - Total mass: ~2.4 kg (2.0 kg chassis + 4 x 0.1 kg wheels)
+    - Wheel width: 0.052 m
+    - Track width (wheel center-to-center, left-right): 0.356 m (304 mm inner + 52 mm wheel)
+    - Wheelbase (front-to-back, axle-to-axle): 0.264 m (per CAD)
+    - Chassis bounding (from STAR.stl): 0.346 x 0.292 x 0.118 m (L x W x H)
+    - Total mass: TBD
 -->
 <robot name="star" xmlns:xacro="http://www.ros.org/wiki/xacro">
@@ -19,17 +20,17 @@
   <!-- Properties                                                          -->
   <!-- ================================================================== -->
-  <xacro:property name="chassis_length" value="0.20"/>
-  <xacro:property name="chassis_width" value="0.15"/>
-  <xacro:property name="chassis_height" value="0.08"/>
+  <xacro:property name="chassis_length" value="0.346"/>
+  <xacro:property name="chassis_width" value="0.292"/>
+  <xacro:property name="chassis_height" value="0.118"/>
   <xacro:property name="chassis_mass" value="2.0"/>
   <xacro:property name="wheel_radius" value="0.072"/>
-  <xacro:property name="wheel_width" value="0.030"/>
+  <xacro:property name="wheel_width" value="0.052"/>
   <xacro:property name="wheel_mass" value="0.1"/>
   <!-- Half track width: center of left wheel to center of right wheel -->
-  <xacro:property name="track_half" value="0.075"/>
+  <xacro:property name="track_half" value="0.178"/>
   <!-- Wheel Y offset: half track + half wheel width (wheel outside chassis) -->
-  <xacro:property name="wheel_y_offset" value="0.090"/>
-  <!-- Front/back wheel X offset from base_link center -->
-  <xacro:property name="wheel_x_offset" value="0.060"/>
+  <xacro:property name="wheel_y_offset" value="0.204"/>
+  <!-- Front/back wheel X offset from base_link center (half of 264mm wheelbase) -->
+  <xacro:property name="wheel_x_offset" value="0.132"/>
   <!-- base_link sits at wheel axle height. Chassis center is above axle. -->
   <xacro:property name="chassis_z_offset" value="${chassis_height / 2}"/>
