Commit message: fix(sim): set chassis/wheel mass from actual BOM (aluminum build)
Gazebo sim only -- masses are not consulted by any real-hardware code
path (motor control, odometry, EKF, nav2). Previous values (2.0 kg
chassis, 0.1 kg wheels) were DFRobot holdovers and made sim dynamics
diverge from reality.

chassis_mass = 3.6 kg:
  0.412 kg  2x 312 mm U-channel @ 206 g           (measured)
  1.430 kg  18"x18"x1/8" aluminum sheet, 80% used (calculated from
            density: 0.209 m^2 * 0.80 * 3.175 mm * 2700 kg/m^3)
  0.384 kg  4x 6V 210RPM metal gearmotors @ 96 g  (datasheet)
  0.900 kg  drivetrain (miter gears, shafts, hubs, bearings, collars)
  0.500 kg  electronics (BeagleBone Blue + battery + sensors + cable)

wheel_mass = 0.348 kg each (goBILDA Wasteland 144mm, measured).

The 0.9 kg drivetrain and 0.5 kg electronics figures are estimates;
refine as hardware components are weighed. The breakdown is kept in
the xacro header comment so the assumption is visible.

File: star-ros2/src/star_simulation/urdf/star_sim.urdf.xacro (robot description, xacro)
@@ -14,5 +14,16 @@
     - Wheelbase (front-to-back, axle-to-axle): 0.264 m (per CAD)
     - Chassis bounding (from STAR.stl): 0.346 x 0.292 x 0.118 m (L x W x H)
-    - Total mass: TBD
+    - Masses (Gazebo sim only, not used on real hardware):
+        * wheel_mass:   0.348 kg each (goBILDA Wasteland, measured)
+        * chassis_mass: 3.6 kg lumped, breakdown:
+            - 2x 312mm U-channel  @ 206 g =  0.412 kg  (measured)
+            - 18" x 18" x 1/8" aluminum sheet, 80% used = 1.430 kg
+              (0.209 m^2 * 0.80 * 0.003175 m * 2700 kg/m^3)
+            - 4x DC gearmotor     @  96 g =  0.384 kg  (datasheet)
+            - Drivetrain (4 miter gear pairs, shafts, hubs,
+              bearings, collars)         ~= 0.9 kg    (estimate)
+            - Electronics (BBB + battery + sensors + cabling)
+                                          ~= 0.5 kg    (estimate)
+          Refine the 0.9 and 0.5 estimates as hardware is weighed.
 -->
 <robot name="star" xmlns:xacro="http://www.ros.org/wiki/xacro">
@@ -23,8 +34,8 @@
   <xacro:property name="chassis_width" value="0.292"/>
   <xacro:property name="chassis_height" value="0.118"/>
-  <xacro:property name="chassis_mass" value="2.0"/>
+  <xacro:property name="chassis_mass" value="3.6"/>
   <xacro:property name="wheel_radius" value="0.072"/>
   <xacro:property name="wheel_width" value="0.052"/>
-  <xacro:property name="wheel_mass" value="0.1"/>
+  <xacro:property name="wheel_mass" value="0.348"/>
   <!-- Half track width: center of left wheel to center of right wheel -->
   <xacro:property name="track_half" value="0.178"/>

Commit message: fix(sim): add Milwaukee M18 drill battery to chassis mass (4.2 kg)
The STAR build is powered by a Milwaukee M18 XC 5.0Ah pack
(48-11-1850), not a small hobby LiPo. Per the Home Depot listing
the pack alone is 1.54 lb (0.699 kg) with an envelope of
~114x79x73 mm. That is heavier than the entire previous 0.5 kg
"electronics" lump in the chassis breakdown, so split the battery
out as its own line item and reduce the remaining electronics
estimate to 0.4 kg (BBB + battery mount/receiver + sensors +
cabling).

New chassis_mass = 4.2 kg (was 3.6 kg):
  0.412 kg  2x 312 mm U-channel
  1.430 kg  18"x18"x1/8" aluminum sheet (80% used)
  0.384 kg  4x gearmotors
  0.900 kg  drivetrain (estimate)
  0.699 kg  Milwaukee M18 XC 5.0Ah battery (datasheet)
  0.400 kg  electronics (estimate)

Gazebo sim only -- no hardware code path consults chassis_mass.

File: star-ros2/src/star_simulation/urdf/star_sim.urdf.xacro (robot description, xacro)
@@ -16,5 +16,5 @@
     - Masses (Gazebo sim only, not used on real hardware):
         * wheel_mass:   0.348 kg each (goBILDA Wasteland, measured)
-        * chassis_mass: 3.6 kg lumped, breakdown:
+        * chassis_mass: 4.2 kg lumped, breakdown:
             - 2x 312mm U-channel  @ 206 g =  0.412 kg  (measured)
             - 18" x 18" x 1/8" aluminum sheet, 80% used = 1.430 kg
@@ -22,8 +22,11 @@
             - 4x DC gearmotor     @  96 g =  0.384 kg  (datasheet)
             - Drivetrain (4 miter gear pairs, shafts, hubs,
-              bearings, collars)         ~= 0.9 kg    (estimate)
-            - Electronics (BBB + battery + sensors + cabling)
-                                          ~= 0.5 kg    (estimate)
-          Refine the 0.9 and 0.5 estimates as hardware is weighed.
+              bearings, collars)         ~= 0.900 kg  (estimate)
+            - Milwaukee M18 XC 5.0Ah battery (48-11-1850)
+                                           = 0.699 kg  (1.54 lb
+              per Home Depot listing; envelope 114x79x73 mm)
+            - Electronics (BBB + battery mount + sensors +
+              cabling)                   ~= 0.400 kg  (estimate)
+          Refine the 0.9 and 0.4 estimates as hardware is weighed.
 -->
 <robot name="star" xmlns:xacro="http://www.ros.org/wiki/xacro">
@@ -34,5 +37,5 @@
   <xacro:property name="chassis_width" value="0.292"/>
   <xacro:property name="chassis_height" value="0.118"/>
-  <xacro:property name="chassis_mass" value="3.6"/>
+  <xacro:property name="chassis_mass" value="4.2"/>
   <xacro:property name="wheel_radius" value="0.072"/>
   <xacro:property name="wheel_width" value="0.052"/>

Commit message: fix: address second CodeRabbit review round + unbreak SPI bridge test
CI surfaced a real test regression caused by the wheel_base bump
in the earlier wheel-radius commit, plus 6 new CodeRabbit findings
on the closed-loop PID wiring. Fixed all 6, pushed back on 1
(SCREAMING_SNAKE_CASE rename for typed enum constants).

CI test failure (test_spi_message_converter):

The wheel-radius commit bumped the SpiMessageConverter::Parameters
fixture from {0.150, 0.0325, 11599} to {0.356, 0.072, 11599}, but
two tests had hardcoded *expected* values (0.15, 0.515, 0.485)
computed against the old wheel_base=0.150. Replace the hardcoded
literals with kTestTrackWidthM-derived expressions:

  TwistToVelocity_RotateLeft (line 56-57):
    expected_right = angular.z * (kTestTrackWidthM / 2.0)
    expected_left  = -expected_right

  RoundTrip_TwistToVelocityToJointState (line 230-234):
    half_track = kTestTrackWidthM / 2.0
    expected_right = linear.x + angular.z * half_track
    expected_left  = linear.x - angular.z * half_track

Both expected values now scale automatically if kTestTrackWidthM
ever changes again, so this class of regression cannot happen.

CodeRabbit fixes:

1. motor_control_task.c rear-right PID setpoint mismatch (Major):
   The encoder feedback for k_bb_motor_idx_rr is mirrored from
   front-right (PRU encoder ch4 broken on 5.10-ti), but the PID
   was still consuming cmd.velocity_setpoint_mps[rr] independently.
   For symmetric skid-steer commands this is fine, but if the
   gateway ever sends asymmetric right-side velocities (FR != RR),
   the rear-right PID would chase its own target while its
   feedback reports what FR is doing -- the integral term would
   diverge and drive the right side against itself. Mirror the
   setpoint too: when i == k_bb_motor_idx_rr, use
   cmd.velocity_setpoint_mps[k_bb_motor_idx_fr] instead. The two
   right-side PIDs now receive identical input and feedback, so
   they track exactly without any chance of divergence.

2. motor_control_task.c fail-closed dispatch (Major): The previous
   if/else dispatch treated every non-velocity mode as direct duty.
   A corrupted enum value (memory smash, future enum addition that
   forgets to update this dispatch) would silently bypass the PID
   and drive duty_percent[]. Restructure to:
       if (estop)              { ... reset PIDs, duty=0 ... }
       else if (mode==velocity)  { ... PID ... }
       else if (mode==direct)    { ... pass-through ... }
       else                      { reset PIDs, duty=0 (fail closed) }
   The unknown-mode branch resets the PID integrators so the next
   valid command starts from a clean slate.

3. bb_pid_config.h derive loop rate from hardware (Trivial):
   k_bb_pid_loop_hz was hardcoded to 100U, duplicating
   k_bb_motor_period_ns from hardware_config.h. If someone changes
   the motor task rate, the documented PID rate would silently
   drift away from the real loop. Include hardware_config.h and
   compute k_bb_pid_loop_hz from k_bb_ns_per_sec / k_bb_motor_period_ns
   so it's mechanically impossible for the two to disagree.

4. hardware_config.h Doxygen contract on bb_wheel_geometry_t (Major):
   Added the project-required @invariant (sync requirement with
   star_gateway_bridge_node.cpp / star_spi_driver_node.cpp), @code
   (showing rad_per_tick computation), @see (cross-references), and
   inline /**< member documentation on k_bb_ticks_per_rev. Also
   expanded the s_bb_wheel_radius_m doc to explain the meters/float
   choice and the cross-reference to the gateway parameters.

5. message_converter.hpp DEFAULT_WHEEL_BASE_M (Minor): Bumped from
   0.150 (DFRobot legacy default) to 0.356 (goBILDA Wasteland
   chassis) so any caller that omits the explicit wheel_base
   argument gets the current platform value. Updated the matching
   doc comments on twist_to_velocity_command() and
   velocity_command_to_twist() to reference 0.356m. Verified all
   production callers (star_gateway_bridge_node.cpp lines 607, 770)
   pass wheel_base_ explicitly and existing tests in
   test_message_converter.cpp use a local WHEEL_BASE_M=0.150
   constant they pass explicitly, so this is a no-op for them.

6. star_sim.urdf.xacro mesh scale (Minor): The wheel/chassis STL
   files in star-ros2/src/star_simulation/meshes/ are exported in
   millimeters (verified: wheel bbox 144x181x124 mm, chassis bbox
   292x346x117 mm), but URDF distances are meters by default and
   the mesh elements had no scale attribute. Without the scale,
   Gazebo would render the wheels as 144 m diameter and the
   chassis as 346 m long while the inertia parameters still used
   the correct 0.072 m / 0.356 m metric values -- a visual/physics
   mismatch that would make the sim useless. Added
   scale="0.001 0.001 0.001" to all 4 mesh references (wheel
   visual + collision, chassis visual + collision).

PUSHED BACK on hardware_config.h:265 SCREAMING_SNAKE_CASE rename.
CodeRabbit cited the project rule "Macro and constant names use
SCREAMING_SNAKE_CASE" but applied it to typed enum values
(k_bb_ticks_per_rev) and static const variables (s_bb_wheel_radius_m).
Per CLAUDE.md the SCREAMING_SNAKE_CASE rule is for #define macros
specifically, while typed enum constants use the k_ lowercase prefix
and static variables use the s_ lowercase prefix. Every other typed
enum and static const in hardware_config.h follows the same k_/s_
convention -- renaming just the new ones would create inconsistency.
The project convention is correct as-is; CodeRabbit applied the
wrong rule.

Build: all 6 host ctest targets still pass under -Werror, including
the 12 motor_control unit tests. CI's test_spi_message_converter
gtest expected values now scale from kTestTrackWidthM so the
RotateLeft and RoundTrip failures are fixed. The cross-compile and
ROS2 colcon paths are still validated by CI (no toolchain locally).

File: star-ros2/src/star_simulation/urdf/star_sim.urdf.xacro (robot description, xacro)
@@ -83,5 +83,7 @@
       <visual>
         <geometry>
-          <mesh filename="package://star_simulation/meshes/wheel_visual.stl"/>
+          <!-- STL exports are in millimeters; URDF distances are in meters. -->
+          <mesh filename="package://star_simulation/meshes/wheel_visual.stl"
+                scale="0.001 0.001 0.001"/>
         </geometry>
         <material name="wheel_black">
@@ -91,5 +93,6 @@
       <collision>
         <geometry>
-          <mesh filename="package://star_simulation/meshes/wheel_collision.stl"/>
+          <mesh filename="package://star_simulation/meshes/wheel_collision.stl"
+                scale="0.001 0.001 0.001"/>
         </geometry>
       </collision>
@@ -106,5 +109,7 @@
     <visual>
       <geometry>
-        <mesh filename="package://star_simulation/meshes/chassis_visual.stl"/>
+        <!-- STL exports are in millimeters; URDF distances are in meters. -->
+        <mesh filename="package://star_simulation/meshes/chassis_visual.stl"
+              scale="0.001 0.001 0.001"/>
       </geometry>
       <material name="chassis_blue">
@@ -114,5 +119,6 @@
     <collision>
       <geometry>
-        <mesh filename="package://star_simulation/meshes/chassis_collision.stl"/>
+        <mesh filename="package://star_simulation/meshes/chassis_collision.stl"
+              scale="0.001 0.001 0.001"/>
       </geometry>
     </collision>
